File: BUS_BOARD/bus-board.sch (KiCad schematic (older format))
At the start: 42 parts, among them J1 Conn_01x08, J10 Conn_01x08, J11 Conn_01x01, J12 Conn_01x08, J13 Conn_01x08, J14 Conn_01x08, J15 Conn_01x08, J16 Conn_01x08, J2 Conn_01x08, J3 Conn_01x08, J4 Conn_01x08, J5 Conn_01x08, J6 Conn_01x08, J7 Conn_01x08, J8 Conn_01x08, J9 Conn_01x08

Commit message: Bus Board work
Parts:
- gave numbers to parts that had none: 2
Other:
- moved on the sheet: J1, J10, J11, J12, J13, J14, J15, J16, J17, J18, J2, J3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
