File: ALU/ALU.kicad_pcb (KiCad board)
At the start: 4 copper layers, 177.5 x 141.3 mm, 53 parts, among them J1 Conn_01x08, J2 Conn_01x08, J3 Conn_01x08, J4 Conn_01x03, J5 Conn_01x02, J6 Conn_01x04, U1 74LS08, U10 74LS86, U11 74LS08, U12 74LS04, U13 74LS245, U14 74LS245, U15 74LS283, U16 74LS157, U17 74LS283, U18 74LS194, U19 74LS04, U2 74LS86, U20 74LS157, U21 74LS86, U22 74LS194, U23 74LS86, U24 74LS245, U25 74LS08, U26 74LS138, U27 74LS08, U3 74LS32, U4 74LS02, U5 74LS245, U6 74LS245, U7 74LS08, U8 74LS245, U9 74LS32

Commit message: Update README
Parts:
- added U28: 74LS245, Package_DIP:DIP-20_W7.62mm, F.Cu at (120.7, 173.4)
- J6: value Conn_01x04 -> Conn_01x05; footprint Connector_PinHeader_2.54mm:PinHeader_1x04_P2.54mm_Vertical -> Connector_PinHeader_2.54mm:PinHeader_1x05_P2.54mm_Vertical
- moved J6 2.11 mm to (162.1, 149.0)
Connections:
- J6 pad 4: /F3 -> /INVERT
- U16 pad 1: /NOT_OUT -> /INVERT
- U16 pad 12: /ALU_OUT8 -> Net-(U16-Pad12)
- U16 pad 4: /ALU_OUT5 -> Net-(U16-Pad4)
- U16 pad 7: /ALU_OUT6 -> Net-(U16-Pad7)
- U16 pad 9: /ALU_OUT7 -> Net-(U16-Pad9)
- U20 pad 1: /NOT_OUT -> /INVERT
- U20 pad 12: /ALU_OUT4 -> Net-(U20-Pad12)
- U20 pad 4: /ALU_OUT1 -> Net-(U20-Pad4)
- U20 pad 7: /ALU_OUT2 -> Net-(U20-Pad7)
- U20 pad 9: /ALU_OUT3 -> Net-(U20-Pad9)
- U26 pad 10: Net-(U26-Pad10) -> /SHL
- U26 pad 11: Net-(U26-Pad11) -> /XOR_OUT
- U26 pad 12: Net-(U26-Pad12) -> /OR_OUT
- U26 pad 13: Net-(U26-Pad13) -> /AND_OUT
- U26 pad 6: /F3 -> VCC
- U26 pad 7: Net-(U26-Pad7) -> /PASS
- U26 pad 9: Net-(U26-Pad9) -> /SHR
- U27 pad 4: Net-(U26-Pad9) -> /SHR
- U27 pad 5: Net-(U26-Pad10) -> /SHL
Routing:
- net /F3: track 87.6 -> 0.00 mm
- net /INVERT: track 0.00 -> 31.7 mm
- net /ALU_EN: track 0.00 -> 26.2 mm
- net /NOT_OUT: track 25.5 -> 0.00 mm
- net Net-(U26-Pad10): track 19.5 -> 0.00 mm
- net /SHL: track 26.7 -> 46.2 mm
- net Net-(U26-Pad9): track 12.8 -> 0.00 mm
- net /SHR: track 25.7 -> 38.5 mm
- removed copper zone on B.Cu, net GND
