File: ALU/ALU.sch (KiCad schematic (older format))
At the start: 49 parts, among them J1 Conn_01x08, J2 Conn_01x08, J3 Conn_01x08, J4 Conn_01x03, J5 Conn_01x02, J6 Conn_01x04, U1 74LS08, U10 74LS86, U11 74LS08, U12 74LS04, U13 74LS245, U14 74LS245, U15 74LS283, U16 74LS157, U17 74LS283, U18 74LS194, U19 74LS04, U2 74LS86, U20 74LS157, U21 74LS86, U22 74LS194, U23 74LS86, U24 74LS245, U25 74LS08, U26 74LS138, U27 74LS08, U3 74LS32, U4 74LS02, U5 74LS245, U6 74LS245, U7 74LS08, U8 74LS245, U9 74LS32

Commit message: Update README
Parts:
- added U28: 74LS245, Package_DIP:DIP-20_W7.62mm, symbol 74xx:74LS245
- J6: value Conn_01x04 -> Conn_01x05; footprint Connector_PinHeader_2.54mm:PinHeader_1x04_P2.54mm_Vertical -> Connector_PinHeader_2.54mm:PinHeader_1x05_P2.54mm_Vertical; symbol Connector_Generic:Conn_01x04 -> Connector_Generic:Conn_01x05
Connections:
- net NOT_OUT is gone; now on net INVERT: U16.1 (S), U20.1 (S)
- net ALU_OUT1: now also U28.9 (A7); no longer U20.4 (Za)
- net ALU_OUT2: now also U28.8 (A6); no longer U20.7 (Zb)
- net ALU_OUT3: now also U28.7 (A5); no longer U20.9 (Zc)
- net ALU_OUT4: now also U28.6 (A4); no longer U20.12 (Zd)
- net ALU_OUT5: now also U28.5 (A3); no longer U16.4 (Za)
- net ALU_OUT6: now also U28.4 (A2); no longer U16.7 (Zb)
- net ALU_OUT7: now also U28.3 (A1); no longer U16.9 (Zc)
- net ALU_OUT8: now also U28.2 (A0); no longer U16.12 (Zd)
- net AND_OUT: now also U26.13 (O2)
- net GND: now also U28.1 (A->B), U28.10 (GND)
- net OR_OUT: now also U26.12 (O3)
- net PASS: now also U26.7 (O7)
- net SHL: now also U26.10 (O5), U27.5
- net SHR: now also U26.9 (O6), U27.4
- net VCC: now also U26.6 (E3), U28.20 (VCC)
- net XOR_OUT: now also U26.11 (O4)
- net F3 renamed INVERT
- net INVERT: no longer U26.6 (E3)
- new net: U16.12 (Zd), U28.18 (B0)
- new net: U16.4 (Za), U28.15 (B3)
- new net: U16.7 (Zb), U28.16 (B2)
- new net: U16.9 (Zc), U28.17 (B1)
- new net: U20.12 (Zd), U28.14 (B4)
- new net: U20.4 (Za), U28.11 (B7)
- new net: U20.7 (Zb), U28.12 (B6)
- new net: U20.9 (Zc), U28.13 (B5)
- new net ALU_EN: J6.5 (Pin_5), U28.19 (CE)
Changed lines of the file:
@@
 	1    0    0    -1
 $EndComp
-Text HLabel 10050 14450 3    59   Output ~ 0
+Text HLabel 11100 16450 3    59   Output ~ 0
 ALU_OUT8
 $Comp
@@
 	1    0    0    -1
 $EndComp
-Text HLabel 12200 14450 3    59   Output ~ 0
+Text HLabel 11500 16450 3    59   Output ~ 0
 ALU_OUT4
 $Comp
@@
 Text Notes 11200 14500 0    79   ~ 0
 Multiplexer
-Text HLabel 10350 14450 3    59   Output ~ 0
+Text HLabel 11200 16450 3    59   Output ~ 0
 ALU_OUT7
-Text HLabel 10650 14450 3    59   Output ~ 0
+Text HLabel 11300 16450 3    59   Output ~ 0
 ALU_OUT6
-Text HLabel 10950 14450 3    59   Output ~ 0
+Text HLabel 11400 16450 3    59   Output ~ 0
 ALU_OUT5
-Text HLabel 12500 14450 3    59   Output ~ 0
+Text HLabel 11600 16450 3    59   Output ~ 0
 ALU_OUT3
-Text HLabel 12800 14450 3    59   Output ~ 0
+Text HLabel 11700 16450 3    59   Output ~ 0
 ALU_OUT2
-Text HLabel 13100 14450 3    59   Output ~ 0
+Text HLabel 11800 16450 3    59   Output ~ 0
 ALU_OUT1
 Wire Wire Line
@@
 	0    -1   -1   0
 $EndComp
-Text HLabel 21000 3000 2    50   Input ~ 0
-PASS
 $Comp
 L power:GND #PWR?
@@
 Wire Wire Line
 	20250 9050 20300 9050
-Text HLabel 16350 9600 0    50   Input ~ 0
-CLOCK
 Wire Wire Line
 	21600 9550 21600 10050
@@
 SUM1
 $Comp
-L Connector_Generic:Conn_01x04 J6
+L Connector_Generic:Conn_01x05 J6
 U 1 1 667B0CDE
-P 14800 2000
-F 0 "J6" V 14718 1512 50  0001 R CNN
-F 1 "Conn_01x04" V 14673 1512 50  0001 R CNN
-F 2 "Connector_PinHeader_2.54mm:PinHeader_1x04_P2.54mm_Vertical" H 14800 2000 50  0001 C CNN
-F 3 "~" H 14800 2000 50  0001 C CNN
-	1    14800 2000
+P 14900 2000
+F 0 "J6" V 14818 1512 50  0001 R CNN
+F 1 "Conn_01x05" V 14773 1512 50  0001 R CNN
+F 2 "Connector_PinHeader_2.54mm:PinHeader_1x05_P2.54mm_Vertical" H 14900 2000 50  0001 C CNN
+F 3 "~" H 14900 2000 50  0001 C CNN
+	1    14900 2000
 	0    -1   -1   0
 $EndComp
@@
 Text HLabel 14900 2200 3    59   Input ~ 0
 F2
-Text HLabel 15000 2200 3    59   Input ~ 0
-F3
-Text HLabel 17650 13400 3    59   Input ~ 0
-F0
-Text HLabel 17750 13400 3    59   Input ~ 0
-F1
-Text HLabel 17850 13400 3    59   Input ~ 0
-F2
-Text HLabel 18150 13400 3    59   Input ~ 0
-F3
-Wire Wire Line
-	18250 13400 18300 13400
-Wire Wire Line
-	18300 13400 18300 13500
-Wire Wire Line
-	18300 13500 18400 13500
-Connection ~ 18300 13400
-Wire Wire Line
-	18300 13400 18350 13400
 $Comp
 L power:GND #PWR?
@@
 SHL
 Text Label 9100 13150 2    59   ~ 0
-NOT_OUT
+INVERT
 $Comp
 L power:VCC #PWR0172
@@
 Wire Wire Line
 	11150 10400 10850 10400
-Wire Bus Line
-	12050 2550 13050 2550
-Wire Bus Line
-	10450 2550 11450 2550
 Connection ~ 10850 10400
 Wire Wire Line
@@
 	1    0    0    -1
 $EndComp
+Wire Wire Line
+	18150 11950 18150 11550
+Connection ~ 18150 11950
+Wire Wire Line
+	18250 11900 18250 11550
+Connection ~ 18250 11900
+Text Label 18250 11550 1    50   ~ 0
+SHR
+Text Label 18150 11550 1    50   ~ 0
+SHL
+Text Label 18050 12400 1    50   ~ 0
+XOR_OUT
+Text Label 17850 12400 1    50   ~ 0
+AND_OUT
+Text Label 17950 12400 1    50   ~ 0
+OR_OUT
+Text Label 18350 12400 1    50   ~ 0
+PASS
+Text Label 21000 3000 0    59   ~ 0
+PASS
+Text Label 16350 9600 2    59   ~ 0
+CLOCK
+Text Label 17650 13400 3    50   ~ 0
+F0
+Text Label 17750 13400 3    50   ~ 0
+F1
+Text Label 17850 13400 3    50   ~ 0
+F2
+Text HLabel 15000 2200 3    59   Input ~ 0
+INVERT
+Wire Wire Line
+	18300 13500 18400 13500
+Wire Wire Line
+	18300 13400 18350 13400
+Wire Wire Line
+	18250 13400 18300 13400
+Connection ~ 18300 13400
+Wire Wire Line
+	18300 13400 18300 13500
+Text HLabel 15100 2200 3    59   Input ~ 0
+ALU_EN
+$Comp
+L 74xx:74LS245 U?
+U 1 1 60F108D3
+P 11600 15950
+AR Path="/607C44AD/60F108D3" Ref="U?"  Part="1"
+AR Path="/607ABD46/60F108D3" Ref="U?"  Part="1"
+AR Path="/609B123A/60F108D3" Ref="U?"  Part="1"
+AR Path="/609B2005/60F108D3" Ref="U?"  Part="1"
+AR Path="/60CD6BAA/609B2005/60F108D3" Ref="U?"  Part="1"
+AR Path="/60F108D3" Ref="U28"  Part="1"
+AR Path="/6099DAC6/60F108D3" Ref="U?"  Part="1"
+F 0 "U28" V 11554 16794 50  0001 L CNN
+F 1 "74LS245" V 11700 15800 50  0000 L CNN
+F 2 "Package_DIP:DIP-20_W7.62mm" H 11600 15950 50  0001 C CNN
+F 3 "http://www.ti.com/lit/gpn/sn74LS08" H 11600 15950 50  0001 C CNN
+	1    11600 15950
+	0    -1   -1   0
+$EndComp
+$Comp
+L power:GND #PWR?
+U 1 1 60F108DD
+P 12000 16500
+AR Path="/607C44AD/60F108DD" Ref="#PWR?"  Part="1"
+AR Path="/607ABD46/60F108DD" Ref="#PWR?"  Part="1"
+AR Path="/609B123A/60F108DD" Ref="#PWR?"  Part="1"
+AR Path="/609B2005/60F108DD" Ref="#PWR?"  Part="1"
+AR Path="/60CD6BAA/609B2005/60F108DD" Ref="#PWR?"  Part="1"
+AR Path="/60F108DD" Ref="#PWR0175"  Part="1"
+AR Path="/6099DAC6/60F108DD" Ref="#PWR?"  Part="1"
+F 0 "#PWR0175" H 12000 16250 50  0001 C CNN
+F 1 "GND" H 12005 16327 50  0000 C CNN
+F 2 "" H 12000 16500 50  0001 C CNN
+F 3 "" H 12000 16500 50  0001 C CNN
+	1    12000 16500
+	1    0    0    -1
+$EndComp
+Wire Wire Line
+	12000 16500 12000 16450
+$Comp
+L power:GND #PWR?
+U 1 1 60F108E8
+P 12450 15950
+AR Path="/607C44AD/60F108E8" Ref="#PWR?"  Part="1"
+AR Path="/607ABD46/60F108E8" Ref="#PWR?"  Part="1"
+AR Path="/609B123A/60F108E8" Ref="#PWR?"  Part="1"
+AR Path="/609B2005/60F108E8" Ref="#PWR?"  Part="1"
+AR Path="/60CD6BAA/609B2005/60F108E8" Ref="#PWR?"  Part="1"
+AR Path="/60F108E8" Ref="#PWR0176"  Part="1"
+AR Path="/6099DAC6/60F108E8" Ref="#PWR?"  Part="1"
+F 0 "#PWR0176" H 12450 15700 50  0001 C CNN
+F 1 "GND" V 12455 15822 50  0000 R CNN
+F 2 "" H 12450 15950 50  0001 C CNN
+F 3 "" H 12450 15950 50  0001 C CNN
+	1    12450 15950
+	0    -1   -1   0
+$EndComp
+Wire Wire Line
+	12450 15950 12400 15950
+$Comp
+L power:VCC #PWR?
+U 1 1 60F108F3
+P 10750 15950
+AR Path="/607C44AD/60F108F3" Ref="#PWR?"  Part="1"
+AR Path="/607ABD46/60F108F3" Ref="#PWR?"  Part="1"
+AR Path="/609B123A/60F108F3" Ref="#PWR?"  Part="1"
+AR Path="/609B2005/60F108F3" Ref="#PWR?"  Part="1"
+AR Path="/60CD6BAA/609B2005/60F108F3" Ref="#PWR?"  Part="1"
+AR Path="/60F108F3" Ref="#PWR0177"  Part="1"
+AR Path="/6099DAC6/60F108F3" Ref="#PWR?"  Part="1"
+F 0 "#PWR0177" H 10750 15800 50  0001 C CNN
+F 1 "VCC" V 10765 16078 50  0000 L CNN
+F 2 "" H 10750 15950 50  0001 C CNN
+F 3 "" H 10750 15950 50  0001 C CNN
+	1    10750 15950
+	0    -1   -1   0
+$EndComp
+Wire Wire Line
+	10750 15950 10800 15950
+Wire Wire Line
+	12100 16450 12100 16500
+Wire Wire Line
+	12100 16500 12250 16500
+Wire Wire Line
+	12250 16500 12250 16600
+Text Label 12250 16600 3    59   ~ 0
+ALU_EN
+Wire Wire Line
+	10050 14450 10050 15250
+Wire Wire Line
+	10050 15250 11100 15250
+Wire Wire Line
+	11100 15250 11100 15450
+Wire Wire Line
+	10350 14450 10350 15100
+Wire Wire Line
+	10350 15100 11200 15100
+Wire Wire Line
+	11200 15100 11200 15450
+Wire Wire Line
+	10650 14450 10650 15000
+Wire Wire Line
+	10650 15000 11300 15000
+Wire Wire Line
+	11300 15000 11300 15450
+Wire Wire Line
+	10950 14450 10950 14900
+Wire Wire Line
+	10950 14900 11400 14900
+Wire Wire Line
+	11400 14900 11400 15450
+Wire Wire Line
+	11500 15450 11500 14900
+Wire Wire Line
+	11500 14900 12200 14900
+Wire Wire Line
+	12200 14900 12200 14450
+Wire Wire Line
+	12500 14450 12500 15000
+Wire Wire Line
+	12500 15000 11600 15000
+Wire Wire Line
+	11600 15000 11600 15450
+Wire Wire Line
+	11700 15450 11700 15100
+Wire Wire Line
+	11700 15100 12800 15100
+Wire Wire Line
+	12800 15100 12800 14450
+Wire Wire Line
+	13100 14450 13100 15200
+Wire Wire Line
+	13100 15200 11800 15200
+Wire Wire Line
+	11800 15200 11800 15450
+$Comp
+L power:VCC #PWR?
+U 1 1 613ECA25
+P 18150 13400
+AR Path="/607C44AD/613ECA25" Ref="#PWR?"  Part="1"
+AR Path="/6089B4B7/613ECA25" Ref="#PWR?"  Part="1"
+AR Path="/60CD6BAA/6089B4B7/613ECA25" Ref="#PWR?"  Part="1"
+AR Path="/608804D8/613ECA25" Ref="#PWR?"  Part="1"
+AR Path="/613ECA25" Ref="#PWR0178"  Part="1"
+F 0 "#PWR0178" H 18150 13250 50  0001 C CNN
+F 1 "VCC" V 18165 13528 50  0000 L CNN
+F 2 "" H 18150 13400 50  0001 C CNN
+F 3 "" H 18150 13400 50  0001 C CNN
+	1    18150 13400
+	-1   0    0    1
+$EndComp
+Wire Bus Line
+	12050 2550 13050 2550
+Wire Bus Line
+	10450 2550 11450 2550
 $EndSCHEMATC

Commit message: BiDirectional Shift Register component
Parts:
- renumbered J1 to J?, J2 to J?, J3 to J?, J4 to J?, J5 to J?, J6 to J?, U25 to U?, U11 to U?, U4 to U?, U26 to U?, U27 to U?
