File: ALU-ADD-SUB/ALU.sch (KiCad schematic (older format))
At the start: 98 parts, among them J1 Conn_01x02, J2 Conn_01x08, J3 Conn_01x08, J4 Conn_01x08, J5 Conn_01x02, J6 Conn_01x08, J8 Conn_01x02, U11 74LS245, U12 74LS283, U13 74LS283, U14 74LS86, U15 74LS86

Commit message: Added Add/Sub Module
Parts:
- removed C? (x3): CP1, Capacitor_THT:C_Radial_D6.3mm_H11.0mm_P2.50mm, symbol Device:CP1
- removed D? (x24): LED, LED_THT:LED_D5.0mm, symbol Device:LED
- removed J8, J?: Conn_01x02, Connector_PinHeader_2.54mm:PinHeader_1x02_P2.54mm_Vertical, symbol Connector_Generic:Conn_01x02
- removed J? (x2): Conn_01x08, Connector_PinHeader_2.54mm:PinHeader_1x08_P2.54mm_Vertical, symbol Connector_Generic:Conn_01x08
- removed RN? (x3): R_Network08_US, Resistor_THT:R_Array_SIP9, symbol Device:R_Network08_US
- removed U? (x4): 74LS245, Package_DIP:DIP-20_W7.62mm, symbol 74xx:74LS245
- removed U? (x8): 74LS86, symbol 74xx:74LS86
- removed U? (x2): 74LS86, Package_DIP:DIP-14_W7.62mm, symbol 74xx:74LS86
- removed U? (x10): 74LS32, Package_DIP:DIP-14_W7.62mm, symbol 74xx:74LS32
- removed U? (x10): 74LS08, Package_DIP:DIP-14_W7.62mm, symbol 74xx:74LS08
- added C1, C2, C3: CP1, Capacitor_THT:C_Radial_D6.3mm_H11.0mm_P2.50mm, symbol Device:CP1
- added D10, D11, D12, D13, D14, D15, D16, D17, D18, D19, D20, D21, D22, D23, D24, D29, D30, D31, D32, D33, D34, D35, D36, D9: LED, LED_THT:LED_D5.0mm, symbol Device:LED
- added J7, J8: Conn_01x08, Connector_PinHeader_2.54mm:PinHeader_1x08_P2.54mm_Vertical, symbol Connector_Generic:Conn_01x08
- added J7, J9: Conn_01x02, Connector_PinHeader_2.54mm:PinHeader_1x02_P2.54mm_Vertical, symbol Connector_Generic:Conn_01x02
- added RN2, RN3, RN4: R_Network08_US, Resistor_THT:R_Array_SIP9, symbol Device:R_Network08_US
- added U1, U7: 74LS08, Package_DIP:DIP-14_W7.62mm, symbol 74xx:74LS08
- added U10, U3: 74LS86, Package_DIP:DIP-14_W7.62mm, symbol 74xx:74LS86
- added U2, U8: 74LS32, Package_DIP:DIP-14_W7.62mm, symbol 74xx:74LS32
- added U4, U5, U6, U9: 74LS245, Package_DIP:DIP-20_W7.62mm, symbol 74xx:74LS245
- J5: value Conn_01x02 -> Conn_01x04; footprint Connector_PinHeader_2.54mm:PinHeader_1x02_P2.54mm_Vertical -> Connector_PinHeader_2.54mm:PinHeader_1x04_P2.54mm_Vertical; symbol Connector_Generic:Conn_01x02 -> Connector_Generic:Conn_01x04
- gave numbers to parts that had none: 9
Connections:
- wire segments 331 -> 330
Other:
- moved on the sheet: RN1

Commit message: BiDirectional Shift Register component
Parts:
- removed C1, C2, C3: CP1, Capacitor_THT:C_Radial_D6.3mm_H11.0mm_P2.50mm, symbol Device:CP1
- removed D10, D11, D12, D13, D14, D15, D16, D17, D18, D19, D20, D21, D22, D23, D24, D29, D30, D31, D32, D33, D34, D35, D36, D9: LED, LED_THT:LED_D5.0mm, symbol Device:LED
- removed J7: Conn_01x08, Connector_PinHeader_2.54mm:PinHeader_1x08_P2.54mm_Vertical, symbol Connector_Generic:Conn_01x08
- removed J9: Conn_01x02, Connector_PinHeader_2.54mm:PinHeader_1x02_P2.54mm_Vertical, symbol Connector_Generic:Conn_01x02
- removed RN2, RN3, RN4: R_Network08_US, Resistor_THT:R_Array_SIP9, symbol Device:R_Network08_US
- removed U1, U7: 74LS08, Package_DIP:DIP-14_W7.62mm, symbol 74xx:74LS08
- removed U10, U3: 74LS86, Package_DIP:DIP-14_W7.62mm, symbol 74xx:74LS86
- removed U2, U8: 74LS32, Package_DIP:DIP-14_W7.62mm, symbol 74xx:74LS32
- removed U4, U5, U6, U9: 74LS245, Package_DIP:DIP-20_W7.62mm, symbol 74xx:74LS245
Connections:
- net labels removed: AND_OUT, OR_OUT, PASS, XOR_OUT
- wire segments 330 -> 152
Other:
- note added: "SUM REG OUT"
- note removed: "AND"
- note removed: "OR"
- note removed: "PASS"
- note removed: "XOR"
