File: ALU-CONTROL/ALU.sch (KiCad schematic (older format))
At the start: 55 parts, among them J1 Conn_01x02, J2 Conn_01x08, J3 Conn_01x08, J4 Conn_01x08, J5 Conn_01x04, J6 Conn_01x08, J7 Conn_01x02, U1 74LS08, U10 74LS245, U2 74LS245, U3 74LS08, U4 74LS32, U5 74LS86, U6 74LS245, U7 74LS32, U8 74LS245, U9 74LS86

Commit message: Adding Programmable RAM Module
Parts:
- removed D1, D10, D11, D12, D13, D14, D15, D16, D17, D18, D19, D2, D20, D21, D22, D23, D24, D25, D26, D27, D28, D3, D4, D5, D6, D7, D8, D9: LED, LED_THT:LED_D5.0mm, symbol Device:LED
- removed J3, J6: Conn_01x08, Connector_PinHeader_2.54mm:PinHeader_1x08_P2.54mm_Vertical, symbol Connector_Generic:Conn_01x08
- removed J5: Conn_01x04, Connector_PinHeader_2.54mm:PinHeader_1x04_P2.54mm_Vertical, symbol Connector_Generic:Conn_01x04
- removed J7: Conn_01x02, Connector_PinHeader_2.54mm:PinHeader_1x02_P2.54mm_Vertical, symbol Connector_Generic:Conn_01x02
- removed R1, R2, R3, R4: R_Small_US, Resistor_THT:R_Axial_DIN0207_L6.3mm_D2.5mm_P10.16mm_Horizontal, symbol Device:R_Small_US
- removed RN1, RN2, RN3: R_Network08_US, Resistor_THT:R_Array_SIP9, symbol Device:R_Network08_US
- removed U10, U2, U6, U8: 74LS245, Package_DIP:DIP-20_W7.62mm, symbol 74xx:74LS245
- removed unit 2 of U3
- removed U4, U7: 74LS32, Package_DIP:DIP-14_W7.62mm, symbol 74xx:74LS32
- removed U5, U9: 74LS86, Package_DIP:DIP-14_W7.62mm, symbol 74xx:74LS86
- added C4: CP1, Capacitor_THT:C_Radial_D6.3mm_H11.0mm_P2.50mm, symbol Device:CP1
- added J5: Conn_01x03, Connector_PinHeader_2.54mm:PinHeader_1x03_P2.54mm_Vertical, symbol Connector_Generic:Conn_01x03
- added J6: Conn_01x05, Connector_PinHeader_2.54mm:PinHeader_1x05_P2.54mm_Vertical, symbol Connector_Generic:Conn_01x05
- added R1, R2, R3, R4, R5, R6, R7: R_US, Resistor_THT:R_Axial_DIN0207_L6.3mm_D2.5mm_P10.16mm_Horizontal, symbol Device:R_US
- added U10: 74LS02, Package_DIP:DIP-14_W7.62mm, symbol 74xx:74LS02
- added U11: 74LS08, Package_DIP:DIP-14_W7.62mm, symbol 74xx:74LS08
- added U2: 74LS138, Package_DIP:DIP-16_W7.62mm, symbol 74xx:74LS138
- added U4, U6: 74LS04, Package_DIP:DIP-14_W7.62mm, symbol 74xx:74LS04
- added U5, U8: 74LS157, Package_DIP:DIP-16_W7.62mm, symbol 74xx:74LS157
- added U7: 74LS245, Package_DIP:DIP-20_W7.62mm, symbol 74xx:74LS245
Connections:
- net labels added: ALU_EN, ALU_OUT1, ALU_OUT2, ALU_OUT3, ALU_OUT4, ALU_OUT5, ALU_OUT6, ALU_OUT7, ALU_OUT8, CARRY_OUT, EQ, F0, F1, F2, INVERT, NEG, SHL, SHR, SUB, SUM1, SUM2, SUM3, SUM4, SUM5, SUM6, SUM7, SUM8, SUM_HIGH_BIT, SUM_OUT, ZE
- net labels removed: A1, A2, A3, A4, A5, A6, A7, A8, A[1..8], B1, B2, B3, B4, B5, B6, B7, B8, B[1..8]
- wire segments 212 -> 104
- no-connect marks 0 -> 3
Other:
- note added: "ALU"
- note added: "ALU OUT"
- note added: "AND all the outputs of the NOR\nverifies that all bits are 0 (LOW)"
- note added: "EQUAL"
- note added: "FLAGS"
- note added: "If INVERT is active (LOW), then\nthe result of the ALU out will be\ninverted"
- note added: "MAIN OUTPUT w/ Invert"
- note added: "Multiplexer"
- note added: "NOR all the bits from the result\nof the SUM/SUB module"
- note added: "To simply Invert an address\njust set PASS and INVERT\nactive, and the result will be\nthe inverse of A"
- note added: "Unused NOT gate from\nOUT w/ Invert"
- note removed: "AND"
- note removed: "B DATA IN"
- note removed: "OR"
- note removed: "PASS"
- note removed: "XOR"
