File: RAM_PROGRAMMER/RAM_PROGRAMMER.sch (KiCad schematic (older format))
At the start: 56 parts, among them J1 Conn_01x02, J2 Conn_01x08, J3 Conn_01x08, J4 Conn_01x08, J5 Conn_01x02, J6 Conn_01x04, J7 Conn_01x11, SW1 SW_Push, U1 ATmega328-PU, U10 74LS245, U2 IS61C1024-15N, U3 74HC595, U4 74LS245, U5 74HC595, U6 74LS157, U7 74LS157, U8 74LS157, U9 74LS157, Y1 Crystal

Commit message: Added RAM Programmer module
Parts:
- removed J2: Conn_01x08, Connector_PinHeader_2.54mm:PinHeader_1x08_P2.54mm_Vertical, symbol Connector_Generic:Conn_01x08
- removed J5: Conn_01x02, Connector_PinHeader_2.54mm:PinHeader_1x02_P2.54mm_Vertical, symbol Connector_Generic:Conn_01x02
- removed U10, U4: 74LS245, Package_DIP:DIP-20_W7.62mm, symbol 74xx:74LS245
- removed U2: IS61C1024-15N, Package_DIP:DIP-32_W7.62mm, symbol Memory_RAM:IS61C1024-15N
- removed U5: 74HC595, Package_DIP:DIP-16_W7.62mm, symbol 74xx:74HC595
- added C10, C8, C9: CP_Small, Capacitor_THT:C_Radial_D5.0mm_H7.0mm_P2.00mm, symbol Device:CP_Small
- added D26, D27, D28, D29, D30, D31, D32, D33, D34, D35, D36, D37, D38, D39, D40, D41: LED, LED_THT:LED_D3.0mm, symbol Device:LED
- added J10, J11, J5, J8, J9: Conn_01x08, Connector_PinHeader_2.54mm:PinHeader_1x08_P2.54mm_Vertical, symbol Connector_Generic:Conn_01x08
- added J2: Conn_01x07, Connector_PinHeader_2.54mm:PinHeader_1x07_P2.54mm_Vertical, symbol Connector_Generic:Conn_01x07
- added R4: R_Small_US, Resistor_THT:R_Axial_DIN0207_L6.3mm_D2.5mm_P10.16mm_Horizontal, symbol Device:R_Small_US
- added RN4, RN5: R_Network08_US, Resistor_THT:R_Array_SIP9, symbol Device:R_Network08_US
- added U10: IS61C1024-15N, Package_DIP:DIP-32_W7.62mm, symbol Memory_RAM:IS61C1024-15N
- added U11, U12, U13, U14: 74LS173, Package_DIP:DIP-16_W7.62mm, symbol 74xx:74LS173
- added U15, U16: 74LS245, Package_DIP:DIP-20_W7.62mm, symbol 74xx:74LS245
- added U17: 74HC595, Package_DIP:DIP-16_W7.62mm, symbol 74xx:74HC595
- added U2: 74LS04, Package_DIP:DIP-14_W7.62mm, symbol 74xx:74LS04
- added U4: 74LS32, Package_DIP:DIP-14_W7.62mm, symbol 74xx:74LS32
- added U5: 74LS08, Package_DIP:DIP-14_W7.62mm, symbol 74xx:74LS08
- J6: value Conn_01x04 -> Conn_01x05; footprint Connector_PinHeader_2.54mm:PinHeader_1x04_P2.54mm_Vertical -> Connector_PinHeader_2.54mm:PinHeader_1x05_P2.54mm_Vertical; symbol Connector_Generic:Conn_01x04 -> Connector_Generic:Conn_01x05
Connections:
- net labels added: ACTIVE, CLOCK, ENABLE_RAM_WRITE_PROG, MAR_IN, MAR_RST, MEM_IN, MEM_RST, VCC, unused?
- net labels removed: A1, A2, A3, A4, A5, A6, A7, A8, ADR1, ADR2, ADR3, ADR4, ADR5, ADR6, ADR7, ADR8, ADR_IN1, ADR_IN2, ADR_IN3, ADR_IN4, ADR_IN5, ADR_IN6, ADR_IN7, ADR_IN8, D1, D2, D3, D4, D5, D6, D7, D8, DATA1, DATA2, DATA3, DATA4, DATA5, DATA6, DATA7, DATA8, DATA_IN1, DATA_IN2, DATA_IN3, DATA_IN4, DATA_IN5, DATA_IN6, DATA_IN7, DATA_IN8, PROG_RAM_WE, RAM_OE, RAM_READY
- wire segments 296 -> 774
Other:
- note added: "1"
- note added: "2"
- note added: "3"
- note added: "4"
- note added: "5"
- note added: "6"
- note added: "7"
- note added: "8"
- note added: "ATMEGA"
- note added: "BUS"
- note added: "Connect ACTIVE\nto HALT on\nComputer Clock"
- note added: "MAIN RAM DATA"
- note added: "MANUAL ADDRESS DATA"
- note added: "MANUAL RAM DATA"
- note added: "MAR"
- note added: "MEMORY DATA\nREGISTER"
- note added: "MUX"
- note added: "RAM"
- note added: "RAM OUT"
- note added: "UNO\nBREAKOUT"
- note removed: "<=="
- note removed: "FROM MAR"
- note removed: "Memory Data Register"
- note removed: "RAM I/O OUT"
- moved on the sheet: C3, C4, C5, C6, C7
