File: SOUND/sound 3.sch (KiCad schematic (older format))
At the start: 19 parts, among them J1 Conn_01x02, J2 Conn_01x02, J3 Conn_01x01, J5 Screw_Terminal_01x02, J6 Conn_01x10, J7 Screw_Terminal_01x02, U1 74LS193, U2 LM555xN, U3 74LS193, U4 74LS193, U5 74LS193, U6 74LS273

Commit message: Updating Sound Module
Parts:
- gave numbers to parts that had none: 1
Changed lines of the file:
@@
 	4150 1800 4150 1850
 $Comp
-L Analog_Switch:CD4052B U?
+L Analog_Switch:CD4052B U7
 U 1 1 61E57DDB
 P 4450 5250
-F 0 "U?" V 4350 5200 50  0000 L CNN
+F 0 "U7" V 4350 5200 50  0000 L CNN
 F 1 "CD4052B" V 4200 5050 50  0000 L CNN
 F 2 "Package_DIP:DIP-16_W7.62mm" H 4600 4500 50  0001 L CNN
@@
 P 3650 5100
 AR Path="/60BC5540/61E7B772" Ref="#PWR?"  Part="1"
-AR Path="/61E7B772" Ref="#PWR?"  Part="1"
-F 0 "#PWR?" H 3650 4950 50  0001 C CNN
+AR Path="/61E7B772" Ref="#PWR0116"  Part="1"
+F 0 "#PWR0116" H 3650 4950 50  0001 C CNN
 F 1 "VCC" H 3665 5273 50  0000 C CNN
 F 2 "" H 3650 5100 50  0001 C CNN
@@
 P 5250 5400
 AR Path="/60BC5540/61E89424" Ref="#PWR?"  Part="1"
-AR Path="/61E89424" Ref="#PWR?"  Part="1"
-F 0 "#PWR?" H 5250 5150 50  0001 C CNN
+AR Path="/61E89424" Ref="#PWR0123"  Part="1"
+F 0 "#PWR0123" H 5250 5150 50  0001 C CNN
 F 1 "GND" H 5255 5227 50  0000 C CNN
 F 2 "" H 5250 5400 50  0001 C CNN
