File: ALU-74LS181-BREAKOUT/kicad/ALU-181.sch (KiCad schematic (older format))
At the start: 20 parts, among them J1 Conn_01x02, J2 Screw_Terminal_01x02, J3 Conn_01x08, J4 Conn_01x08, J5 Conn_01x08, J6 Conn_01x06, J7 Conn_01x03, J8 Conn_01x03, U1 74LS181, U2 74LS181, U3 74LS02, U4 74LS04, U5 74LS245

Commit message: Updating components
Parts:
- renumbered C1 to C9, D1 to D23, D3 to D24, D4 to D25, J1 to J13, J2 to J14, J6 to J15, J4 to J16, J8 to J17, J5 to J18, J3 to J19, J7 to J20, R1 to R7, R3 to R8, R4 to R9, U5 to U10, U2 to U11, U4 to U7, U3 to U8, U1 to U9
Connections:
- net labels added: EQ, GT
- wire segments 110 -> 142
