File: COUNTER/COUNTER.sch (KiCad schematic (older format))
At the start: 24 parts, among them J1 Conn_01x08, J10 Conn_01x04, J2 Conn_01x03, J3 Conn_01x08, U46 74LS161, U47 74LS245, U48 74LS161

Commit message: More Additions, Counter, ALU, Clock
Parts:
- J2: value Conn_01x03 -> Conn_01x04; footprint Connector_PinHeader_2.54mm:PinHeader_1x03_P2.54mm_Vertical -> Connector_PinHeader_2.54mm:PinHeader_1x04_P2.54mm_Vertical; symbol Connector_Generic:Conn_01x03 -> Connector_Generic:Conn_01x04
Connections:
- net OE: now also J2.4 (Pin_4)
Changed lines of the file:
@@
 	1    0    0    -1
 $EndComp
-Text HLabel 6450 1150 0    50   Input ~ 0
+Text HLabel 6450 1000 0    50   Input ~ 0
 CLOCK
 Text HLabel 4700 1900 1    50   Input ~ 0
 RESET
-Text HLabel 6450 1050 0    50   Input ~ 0
+Text HLabel 6450 900  0    50   Input ~ 0
 RESET
-Text HLabel 6450 950  0    50   Input ~ 0
+Text HLabel 6450 800  0    50   Input ~ 0
 JUMP
 $Comp
-L Connector_Generic:Conn_01x03 J2
+L Connector_Generic:Conn_01x04 J2
 U 1 1 60844354
-P 6650 1050
-F 0 "J2" H 6730 1046 50  0000 L CNN
-F 1 "Conn_01x03" H 6730 951 50  0001 L CNN
-F 2 "Connector_PinHeader_2.54mm:PinHeader_1x03_P2.54mm_Vertical" H 6650 1050 50  0001 C CNN
-F 3 "~" H 6650 1050 50  0001 C CNN
-	1    6650 1050
+P 6650 900
+F 0 "J2" H 6730 896 50  0000 L CNN
+F 1 "Conn_01x04" H 6730 801 50  0001 L CNN
+F 2 "Connector_PinHeader_2.54mm:PinHeader_1x04_P2.54mm_Vertical" H 6650 900 50  0001 C CNN
+F 3 "~" H 6650 900 50  0001 C CNN
+	1    6650 900
 	1    0    0    -1
 $EndComp
@@
 Text HLabel 6450 2000 0    50   Input ~ 0
 D8
+Text HLabel 6450 1100 0    50   Input ~ 0
+OE
 $EndSCHEMATC

Commit message: Updating components
Parts:
- removed D44, D45, D46, D47, D48, D49, D50, D51: LED, LED_THT:LED_D5.0mm, symbol Device:LED
- removed R11, R12, R13, R14, R15, R16, R17, R18: R_US, Resistor_THT:R_Axial_DIN0207_L6.3mm_D2.5mm_P10.16mm_Horizontal, symbol Device:R_US
- added BAR1: HDSP-4830_2, Display:HDSP-4830, symbol LED:HDSP-4830_2
- added J1: Screw_Terminal_01x02, TerminalBlock_Phoenix:TerminalBlock_Phoenix_MKDS-1,5-2_1x02_P5.00mm_Horizontal, symbol Connector:Screw_Terminal_01x02
- added RN1: R_Network08, Resistor_THT:R_Array_SIP9, symbol Device:R_Network08
- J22: renamed from J2; value Conn_01x04 -> Conn_01x05; footprint Connector_PinHeader_2.54mm:PinHeader_1x04_P2.54mm_Vertical -> Connector_PinHeader_2.54mm:PinHeader_1x05_P2.54mm_Vertical; symbol Connector_Generic:Conn_01x04 -> Connector_Generic:Conn_01x05
- renumbered J3 to J23, J1 to J24, U46 to U12, U48 to U14
Connections:
- net GND: now also J10.1 (Pin_1), J1.1 (Pin_1), RN1.1 (common); no longer J10.2 (Pin_2)
- net VCC: now also J10.2 (Pin_2), J1.2 (Pin_2); no longer J10.1 (Pin_1), U14.10 (CET), U14.7 (CEP)
- net at U14.14 (Q0), U47.11 (B7): now also BAR1.1 (A)
- net at U14.13 (Q1), U47.12 (B6): now also BAR1.2 (A)
- net at U14.12 (Q2), U47.13 (B5): now also BAR1.3 (A)
- net at U14.11 (Q3), U47.14 (B4): now also BAR1.4 (A)
- net at U12.14 (Q0), U47.15 (B3): now also BAR1.5 (A)
- net at U12.13 (Q1), U47.16 (B2): now also BAR1.6 (A)
- net at U12.12 (Q2), U47.17 (B1): now also BAR1.7 (A)
- net at U12.11 (Q3), U47.18 (B0): now also BAR1.8 (A)
- new net: BAR1.13 (K), RN1.9 (R8)
- new net: BAR1.14 (K), RN1.8 (R7)
- new net: BAR1.15 (K), RN1.7 (R6)
- new net: BAR1.16 (K), RN1.6 (R5)
- new net: BAR1.17 (K), RN1.5 (R4)
- new net: BAR1.18 (K), RN1.4 (R3)
- new net: BAR1.19 (K), RN1.3 (R2)
- new net: BAR1.20 (K), RN1.2 (R1)
- new net CE: J22.5 (Pin_5), U14.10 (CET), U14.7 (CEP)
- no-connect marks 1 -> 5
Other:
- moved on the sheet: J23, J24
