File: RAM/RAM/RAM.sch (KiCad schematic (older format))
At the start: 24 parts, among them J1 Conn_01x19, J2 Conn_01x05, J3 Conn_01x02, J4 Screw_Terminal_01x02, J6 Conn_01x08, J7 Conn_01x08, U1 IS61C1024-15N, U2 74LS245, U3 74LS245, U4 74LS00, U6 74LS32

Commit message: Updating components
Parts:
- renumbered C1 to C13, C2 to C14, C3 to C15, C4 to C16, D1 to D50, D2 to D51, D3 to D52, D4 to D53, D5 to D54, D6 to D55, D7 to D56, D8 to D57, J3 to J29, J1 to J30, J4 to J31, J2 to J32, J6 to J33, J7 to J34, RN1 to RN9, U4 to U23, U1 to U24, U6 to U25, U3 to U26, U2 to U27
Other:
- moved on the sheet: J30, J33, J34
