File: STORAGE-REGISTER-SINGLE/REGISTER.sch (KiCad schematic (older format))
At the start: 28 parts, among them J1 Screw_Terminal_01x02, J2 Conn_01x08, J3 Conn_01x02, J5 Conn_01x08, J6 Conn_01x05, J8 Conn_01x08, U1 74LS245, U2 74LS173, U3 74LS173

Commit message: Updating components
Parts:
- renumbered C4 to C1, C1 to C2, C2 to C3, C3 to C4, J2 to J1, J6 to J2, J5 to J3, J8 to J4, J3 to J5, J1 to J6
