File: CLOCK/CLOCK.kicad_pcb (KiCad board)
At the start: 4 copper layers, 96.5 x 78.5 mm, 45 parts, among them J1 Screw_Terminal_01x02, J2 Conn_01x08, J3 Conn_01x02, J34 Conn_01x08, J5 Conn_01x08, SW1 SW_Push, SW13 SW_DIP_x08, SW2 SW_dPDT, U1 4-pin-crystal-1mhz, U10 74LS86, U11 74LS173, U2 74LS193, U3 74LS173, U4 74LS193, U5 74LS193, U6 74LS193, U7 LM555xN, U8 74LS04, U9 74LS08

Commit message: Updating Clock Module
Connections:
- SW2 pad 2: GND -> Net-(SW2-Pad2)
- SW2 pad 4: Net-(SW2-Pad4) -> GND

Commit message: [Final] Clock Module
Parts:
- removed the R3 at (135.9, 96.3)
- removed REF** (x4): MountingHole_3mm, MountingHole:MountingHole_3mm
- added R1: R_Small_US, Resistor_THT:R_Axial_DIN0207_L6.3mm_D2.5mm_P10.16mm_Horizontal, F.Cu at (122.1, 27.6)
- added SW4: SW_SPDT, 8-bit-diy-computer:SPDT-SlideSwitch, F.Cu at (139.9, 90.1)
- J5: renamed from J34; value Conn_01x08 -> Conn_01x04; footprint Connector_PinHeader_2.54mm:PinHeader_2x08_P2.54mm_Vertical -> Connector_PinHeader_2.54mm:PinHeader_2x04_P2.54mm_Vertical
- SW2: value SW_dPDT -> SW_Push; footprint 8-bit-diy-computer:dpdt_tht_push_switch -> Button_Switch_THT:SW_PUSH_6mm
- moved SW2 63.0 mm to (106.7, 38.9), turned to 0 degrees
- moved C2 0.51 mm to (74.4, 97.9)
- moved U10 0.28 mm to (136.7, 81.8)
- moved U8 0.14 mm to (136.7, 70.0)
- renumbered C3 to C1, C4 to C2, C1 to C3, C2 to C4, D55 to D10, D54 to D2, D2 to D9, J2 to J1, J5 to J2, J1 to J4, R1 to R3, R5 to R4, R4 to R5, SW13 to SW1, SW1 to SW3, U3 to U1, U7 to U11, U11 to U2, U1 to U3, U2 to U4, U4 to U5, U5 to U6, U6 to U7
Connections:
- net +5V renamed VCC
- net /1MHz_Pulse renamed 1MHz_Pulse
- net /A0 renamed A0
- net /A1 renamed A1
- net /A2 renamed A2
- net /A3 renamed A3
- net /A4 renamed A4
- net /A5 renamed A5
- net /A6 renamed A6
- net /A7 renamed A7
- net /CLOCK_OUT renamed CLOCK_OUT
- net /HALT renamed HALT
- net Net-(J2-Pad1) renamed BUS_01
- net Net-(J2-Pad2) renamed BUS_02
- net Net-(J2-Pad3) renamed BUS_03
- net Net-(J2-Pad4) renamed BUS_04
- net Net-(J2-Pad5) renamed BUS_05
- net Net-(J2-Pad6) renamed BUS_06
- net Net-(J2-Pad7) renamed BUS_07
- net Net-(J2-Pad8) renamed BUS_08
- net Net-(U7-Pad3) renamed Monostable_Pulse
- D9 pad 2: Net-(D2-Pad2) -> MODE
- J3 pad 2: /SET_SPEED -> SET_SPEED
- J5 pad 1: Net-(J34-Pad1) -> Frequency
- J5 pad 3: Net-(J34-Pad1) -> Frequency
- J5 pad 5: Net-(J34-Pad1) -> Frequency
- J5 pad 7: Net-(J34-Pad1) -> Frequency
- SW2 pad 1: Net-(SW2-Pad1) -> GND
- SW2 pad 2: Net-(SW2-Pad2) -> SET_SPEED
- U1 pad 10: /SET_SPEED -> SET_SPEED
- U1 pad 9: /SET_SPEED -> SET_SPEED
- U2 pad 10: /SET_SPEED -> SET_SPEED
- U2 pad 9: /SET_SPEED -> SET_SPEED
- U6 pad 2: Net-(J34-Pad12) -> Net-(U6-Pad2)
- U6 pad 3: Net-(J34-Pad10) -> Net-(U6-Pad3)
- U6 pad 6: Net-(J34-Pad14) -> Net-(U6-Pad6)
- U6 pad 7: Net-(J34-Pad16) -> Net-(U6-Pad7)
- U8 pad 1: Net-(D2-Pad2) -> MODE
- U9 pad 12: Net-(D2-Pad2) -> MODE
- U9 pad 13: Net-(J34-Pad1) -> Frequency
Routing:
- net SET_SPEED: track 0.00 -> 135.0 mm
- net /SET_SPEED: track 92.9 -> 0.00 mm
- net Net-(D2-Pad2): track 70.6 -> 0.00 mm
- net MODE: track 0.00 -> 62.8 mm
- net Net-(J34-Pad1): track 50.1 -> 0.00 mm
- net Frequency: track 0.00 -> 50.1 mm
- net Net-(J34-Pad12): track 37.9 -> 0.00 mm
- net Net-(J34-Pad10): track 30.5 -> 0.00 mm
- net Net-(J34-Pad14): track 27.3 -> 0.00 mm
- net Net-(J34-Pad16): track 26.5 -> 0.00 mm
Other:
- board text added: "0.22μf"
- board text added: "100μf"
- board text added: "1K PULL UP"
- board text added: "47μf"
- board text added: "4K Ω"
- board text added: "PROG"
- board text added: "RUN"
- board text added: "RUN MODE"
- board text added: "SET FREQ"
- board text removed: "MANUAL MODE"
- board text removed: "MODE"
- board text removed: "PULL UP"
