File: Modules/display-module/DISPLAY.sch (KiCad schematic (older format))
At the start: 18 parts, among them J1 Screw_Terminal_01x02, J2 Conn_01x08, J3 Conn_01x03, U1 HDSP-7503, U1555 NE55P, U2 74LS08, U2444 74LS76, U3 74LS273, U4 HDSP-7503, U4332 74LS139, U5 HDSP-7503, U6 HDSP-7503, U9 AT28C256

Commit message: [Display] Semi-final Display Module
Parts:
- added R1, R?: R_US, Resistor_THT:R_Axial_DIN0207_L6.3mm_D2.5mm_P10.16mm_Horizontal, symbol Device:R_US
- added SW1: SW_SPST, Button_Switch_THT:SW_DIP_SPSTx01_Slide_9.78x4.72mm_W7.62mm_P2.54mm, symbol Switch:SW_SPST
- J3: value Conn_01x03 -> Conn_01x05; footprint Connector_PinHeader_2.54mm:PinHeader_1x03_P2.54mm_Vertical -> Connector_PinHeader_2.54mm:PinHeader_1x05_P2.54mm_Vertical; symbol Connector_Generic:Conn_01x03 -> Connector_Generic:Conn_01x05
Connections:
- net A0: now also U2444.14 (~Q), U2444.6 (C)
- net A_SEG: now also U9.18 (IO6); no longer U9.11 (IO0)
- net B_SEG: now also U9.17 (IO5); no longer U9.12 (IO1)
- net CLOCK: now also J3.3 (Pin_3); no longer J3.2 (Pin_2)
- net C_SEG: now also U9.16 (IO4); no longer U9.13 (IO2)
- net DP_SEG: now also U1.5 (DP), U4.5 (DP), U5.5 (DP), U6.5 (DP)
- net E_SEG: now also U9.13 (IO2); no longer U9.16 (IO4)
- net F_SEG: now also U9.12 (IO1); no longer U9.17 (IO5)
- net GND: now also R1.1, R?.1; no longer U9.23 (A11)
- net G_SEG: now also U9.11 (IO0); no longer U9.18 (IO6)
- net OI: now also J3.2 (Pin_2); no longer J3.1 (Pin_1)
- net RST: now also J3.4 (Pin_4); no longer J3.3 (Pin_3)
- net VCC: now also SW1.1 (A)
- net SIGNED: now reaches U9.21 (A10)
- net SIGNED: now also J3.5 (Pin_5), R1.2, SW1.2 (B)
- new net HEX: J3.1 (Pin_1), R?.2, U9.23 (A11)
- no-connect marks 6 -> 3

Commit message: [General] Updates
Parts:
- gave numbers to parts that had none: 1
Connections:
- net at C133.2, U1555.2 (TR): now also R1452.2, U1555.6 (THR)
Changed lines of the file:
@@
 HEX
 $Comp
-L Device:R_US R?
+L Device:R_US R2
 U 1 1 610AB23E
 P 5100 3600
-F 0 "R?" V 4987 3600 50  0001 C CNN
+F 0 "R2" V 4987 3600 50  0001 C CNN
 F 1 "R_US" V 4986 3600 50  0001 C CNN
 F 2 "Resistor_THT:R_Axial_DIN0207_L6.3mm_D2.5mm_P10.16mm_Horizontal" V 5140 3590 50  0001 C CNN
@@
 	5250 3600 5300 3600
 Connection ~ 5300 3600
+Wire Wire Line
+	3250 1650 3250 1500
+Wire Wire Line
+	3250 1500 2850 1500
+Wire Wire Line
+	2850 1500 2850 2550
+Wire Wire Line
+	2850 2550 4300 2550
+Wire Wire Line
+	4300 2550 4300 2050
+Connection ~ 3250 1650
+Connection ~ 4300 2050
 $EndSCHEMATC
