File: Modules/alu-module/ALU-181.kicad_pcb (KiCad board)
At the start: 4 copper layers, 144 x 67.3 mm, 34 parts, among them J1 Conn_01x08, J17 Conn_01x03, J2 Conn_01x12, J20 Conn_01x03, J3 Screw_Terminal_01x02, J4 Conn_01x08, U1 74LS245, U10 74LS245, U11 74LS181, U2 74LS245, U3 74LS173, U4 74LS173, U5 74LS173, U6 74LS173, U7 74LS04, U8 74LS02, U9 74LS181

Commit message: [General] Updates
Other:
- board text added: "01011 NOT B 10011 XNOR 11111 A 10101 B"
- board text added: "01100 SUB 10010 ADD 01101 XOR 10111 AND 11101 OR"
- board text added: "11000 SHL A 11110 DEC A 00001 NOT A 00011 NOR 01001 NAND"
- board text added: "ALU A Register B Register"
- board text added: "Cn"
- board text added: "S0|S1|S2|S3|MD"
- board text removed: "ALU / A Register / B Register"
Changed lines of the file:
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@@
   (general
     (thickness 1.6)
-    (drawings 69)
+    (drawings 84)
     (tracks 1010)
     (zones 0)
@@
       (drillshape 0)
       (scaleselection 1)
-      (outputdirectory "../gerber/"))
+      (outputdirectory "gerber/"))
   )
   (net 0 "")
@@
     )
   )
+  (gr_text Cn (at 91.948 91.44) (layer F.SilkS)
+    (effects (font (size 1 1) (thickness 0.15)))
+  )
+  (gr_text -GND (at 86.614 88.9 90) (layer F.SilkS)
+    (effects (font (size 1 1) (thickness 0.15)))
+  )
+  (gr_text +VCC (at 97.282 88.9 90) (layer F.SilkS)
+    (effects (font (size 1 1) (thickness 0.15)))
+  )
+  (gr_line (start 72.644 94.234) (end 74.168 94.234) (layer F.SilkS) (width 0.12))
+  (gr_line (start 73.66 101.854) (end 74.168 101.854) (layer F.SilkS) (width 0.12))
+  (gr_line (start 72.644 96.774) (end 74.168 96.774) (layer F.SilkS) (width 0.12))
+  (gr_line (start 72.644 101.854) (end 73.66 101.854) (layer F.SilkS) (width 0.12))
+  (gr_line (start 72.644 99.314) (end 73.66 99.314) (layer F.SilkS) (width 0.12))
+  (gr_line (start 72.644 104.394) (end 73.66 104.394) (layer F.SilkS) (width 0.12))
+  (gr_line (start 133.858 58.928) (end 133.858 63.754) (layer F.SilkS) (width 0.12))
+  (gr_line (start 122.174 59.436) (end 122.174 64.262) (layer F.SilkS) (width 0.12))
+  (gr_text S0|S1|S2|S3|MD (at 112.522 56.388) (layer F.SilkS)
+    (effects (font (size 0.8 0.8) (thickness 0.1)) (justify left))
+  )
+  (gr_text "01011 NOT B\n10011 XNOR\n11111 A\n10101 B\n\n" (at 134.366 61.976) (layer F.SilkS)
+    (effects (font (size 1 1) (thickness 0.1)) (justify left))
+  )
+  (gr_text "11000 SHL A\n11110 DEC A\n00001 NOT A\n00011 NOR\n01001 NAND" (at 122.936 61.976) (layer F.SilkS)
+    (effects (font (size 1 1) (thickness 0.1)) (justify left))
+  )
+  (gr_text "01100 SUB\n10010 ADD\n01101 XOR\n10111 AND\n11101 OR" (at 112.522 61.976) (layer F.SilkS)
+    (effects (font (size 1 1) (thickness 0.1)) (justify left))
+  )
   (gr_line (start 211.328 121.92) (end 211.328 120.904) (layer Edge.Cuts) (width 0.05))
   (gr_line (start 67.31 121.92) (end 211.328 121.92) (layer Edge.Cuts) (width 0.05))
@@
     (effects (font (size 1 1) (thickness 0.15)) (justify right))
   )
-  (gr_text theWickedWebDev/8-bit-computer (at 95.758 119.38) (layer F.SilkS)
+  (gr_text theWickedWebDev/8-bit-computer (at 96.266 119.888) (layer F.SilkS)
     (effects (font (size 0.8 0.8) (thickness 0.1)) (justify right))
   )
-  (gr_text "ALU / A Register / B Register" (at 115.824 58.674) (layer F.SilkS)
-    (effects (font (size 2 2) (thickness 0.15)))
+  (gr_text "ALU\nA Register\nB Register" (at 90.424 60.706) (layer F.SilkS)
+    (effects (font (size 2 2) (thickness 0.15)) (justify left))
   )
   (gr_text X (at 78.486 116.586) (layer F.SilkS)

Commit message: [ALU] Updated ALU - needs work
Parts:
- removed J20: Conn_01x03, Connector_PinHeader_2.54mm:PinHeader_1x03_P2.54mm_Vertical
- J2: value Conn_01x12 -> Conn_01x15; footprint Connector_PinHeader_2.54mm:PinHeader_1x12_P2.54mm_Vertical -> Connector_PinHeader_2.54mm:PinHeader_1x15_P2.54mm_Vertical
- moved J2 7.62 mm to (70.6, 74.9)
Connections:
- J2 pad 1: ALU_S0 -> A_GT_B
- J2 pad 10: A_REGISTER_IN -> B_REGISTER_OUT
- J2 pad 11: RESET -> B_REGISTER_IN
- J2 pad 12: CLOCK -> A_REGISTER_OUT
- J2 pad 2: ALU_S1 -> A_EQ_B
- J2 pad 3: ALU_S2 -> NOT_CARRY
- J2 pad 4: ALU_S3 -> ALU_S0
- J2 pad 5: ALU_MODE -> ALU_S1
- J2 pad 6: ALU_OUT -> ALU_S2
- J2 pad 7: B_REGISTER_OUT -> ALU_S3
- J2 pad 8: B_REGISTER_IN -> ALU_MODE
- J2 pad 9: A_REGISTER_OUT -> ALU_OUT
- U10 pad 19: ALU_OUT -> NOT_ALU_OUT
- U7 pad 10: (no net) -> Net-(U7-Pad10)
- U7 pad 11: (no net) -> Net-(U7-Pad11)
- U7 pad 12: (no net) -> Net-(U7-Pad12)
- U7 pad 13: (no net) -> Net-(U7-Pad13)
- U7 pad 3: (no net) -> ALU_OUT
- U7 pad 4: (no net) -> NOT_ALU_OUT
- U7 pad 5: (no net) -> Net-(U7-Pad5)
- U7 pad 6: (no net) -> Net-(U7-Pad6)
- U7 pad 8: (no net) -> Net-(U7-Pad8)
- U7 pad 9: (no net) -> Net-(U7-Pad9)
Routing:
- net NOT_ALU_OUT: track 0.00 -> 36.4 mm
- net ALU_OUT: track 90.0 -> 121.7 mm
- net A_EQ_B: track 136.2 -> 134.8 mm
