File: Modules/alu-module/ALU-181.sch (KiCad schematic (older format))
At the start: 30 parts, among them J1 Conn_01x08, J17 Conn_01x03, J2 Conn_01x12, J20 Conn_01x03, J3 Screw_Terminal_01x02, J4 Conn_01x08, U1 74LS245, U10 74LS245, U11 74LS181, U2 74LS245, U3 74LS173, U4 74LS173, U5 74LS173, U6 74LS173, U7 74LS04, U8 74LS02, U9 74LS181

Commit message: [ALU] Updated ALU - needs work
Parts:
- removed J20: Conn_01x03, Connector_PinHeader_2.54mm:PinHeader_1x03_P2.54mm_Vertical, symbol Connector_Generic:Conn_01x03
- added unit 2 of U7
- added unit 3 of U7
- added unit 4 of U7
- added unit 5 of U7
- added unit 6 of U7
- J2: value Conn_01x12 -> Conn_01x15; footprint Connector_PinHeader_2.54mm:PinHeader_1x12_P2.54mm_Vertical -> Connector_PinHeader_2.54mm:PinHeader_1x15_P2.54mm_Vertical; symbol Connector_Generic:Conn_01x12 -> Connector_Generic:Conn_01x15
Connections:
- net ALU_MODE: now also J2.8 (Pin_8); no longer J2.5 (Pin_5)
- net ALU_OUT: now also J2.9 (Pin_9), U7.3; no longer J2.6 (Pin_6), U10.19 (CE)
- net ALU_S0: now also J2.4 (Pin_4); no longer J2.1 (Pin_1)
- net ALU_S1: now also J2.5 (Pin_5); no longer J2.2 (Pin_2)
- net ALU_S2: now also J2.6 (Pin_6); no longer J2.3 (Pin_3)
- net ALU_S3: now also J2.7 (Pin_7); no longer J2.4 (Pin_4)
- net A_EQ_B: now also J2.2 (Pin_2)
- net A_GT_B: now also J2.1 (Pin_1)
- net A_REGISTER_IN: now also J2.13 (Pin_13); no longer J2.10 (Pin_10)
- net A_REGISTER_OUT: now also J2.12 (Pin_12); no longer J2.9 (Pin_9)
- net B_REGISTER_IN: now also J2.11 (Pin_11); no longer J2.8 (Pin_8)
- net B_REGISTER_OUT: now also J2.10 (Pin_10); no longer J2.7 (Pin_7)
- net CLOCK: now also J2.15 (Pin_15); no longer J2.12 (Pin_12)
- net NOT_CARRY: now also J2.3 (Pin_3)
- net RESET: now also J2.14 (Pin_14); no longer J2.11 (Pin_11)
- new net NOT_ALU_OUT: U10.19 (CE), U7.4
