File: Modules/counter-module/kicad/COUNTER.kicad_pcb (KiCad board)
At the start: 4 copper layers, 69.1 x 45.3 mm, 15 parts, among them J1 Screw_Terminal_01x02, J10 Conn_01x04, J22 Conn_01x06, J23 Conn_01x08, J24 Conn_01x08, U12 74LS161, U14 74LS161, U47 74LS245

Commit message: [Counter] Updates after printing
Connections:
- net Y1 renamed OUT_01
- net Y2 renamed OUT_02
- net Y3 renamed OUT_03
- net Y4 renamed OUT_04
- net Y5 renamed OUT_05
- net Y6 renamed OUT_06
- net Y7 renamed OUT_07
- net Y8 renamed OUT_08
- U12 pad 11: B0 -> B7
- U12 pad 12: B1 -> B6
- U12 pad 13: B2 -> B5
- U12 pad 14: B3 -> B4
- U14 pad 11: B4 -> B3
- U14 pad 12: B5 -> B2
- U14 pad 13: B6 -> B1
- U14 pad 14: B7 -> B0
Routing:
- net B4: track 33.8 -> 65.3 mm
- net B5: track 33.8 -> 63.6 mm
- net B6: track 33.8 -> 63.3 mm
- net B7: track 34.4 -> 58.2 mm
- net B1: track 37.0 -> 52.9 mm
- net B2: track 37.0 -> 48.5 mm
- net B3: track 37.0 -> 43.8 mm
- net B0: track 37.0 -> 41.5 mm
Other:
- board text added: "v3"
