File: Modules/counter-module/kicad/COUNTER.sch (KiCad schematic (older format))
At the start: 11 parts, among them J1 Screw_Terminal_01x02, J10 Conn_01x04, J22 Conn_01x06, J23 Conn_01x08, J24 Conn_01x08, U12 74LS161, U14 74LS161, U47 74LS245

Commit message: [Counter] Updates after printing
Connections:
- net B0: now also U14.14 (Q0); no longer U12.11 (Q3)
- net B1: now also U14.13 (Q1); no longer U12.12 (Q2)
- net B2: now also U14.12 (Q2); no longer U12.13 (Q1)
- net B3: now also U14.11 (Q3); no longer U12.14 (Q0)
- net B4: now also U12.14 (Q0); no longer U14.11 (Q3)
- net B5: now also U12.13 (Q1); no longer U14.12 (Q2)
- net B6: now also U12.12 (Q2); no longer U14.13 (Q1)
- net B7: now also U12.11 (Q3); no longer U14.14 (Q0)
- net Y1 renamed OUT_01
- net Y2 renamed OUT_02
- net Y3 renamed OUT_03
- net Y4 renamed OUT_04
- net Y5 renamed OUT_05
- net Y6 renamed OUT_06
- net Y7 renamed OUT_07
- net Y8 renamed OUT_08
Other:
- moved on the sheet: BAR1, J22, J23, J24, RN1, U12, U14
