File: Modules/control-module/control.kicad_pcb (KiCad board)
At the start: 2 copper layers, 29 parts, among them J1 Conn_01x02, J10 Conn_1x04, J11 Conn_1x04, J2 Conn_01x08, J3 Conn_01x10, J4 Conn_2x08, J5 Conn_01x02, J50 Screw_Terminal_01x02, J7 Conn_1x08, J9 Conn_01x02, SW6 SW_Push, U1 74LS161, U2 74LS173, U7 74LS04

Commit message: [General] Updates
Parts:
- removed D79, D80: LED, LED_THT:LED_D3.0mm
- removed EEPROM3: AT28C256, 8-bit-computer:DIP_Socket-40_W11.9_W12.7_W15.24_W17.78_W18.5_3M_240-1280-00-0602J
- removed J1, J9: Conn_01x02, Connector_PinHeader_2.54mm:PinHeader_1x02_P2.54mm_Vertical
- removed J10, J11: Conn_1x04, Connector_PinHeader_2.54mm:PinHeader_1x04_P2.54mm_Vertical
- removed J7: Conn_1x08, Connector_PinHeader_2.54mm:PinHeader_1x08_P2.54mm_Vertical
- added BAR4: HDSP-4850_2, Display:HDSP-4850, F.Cu at (134.3, 85.0)
- added BAR5: HDSP-4850_2, Display:HDSP-4850, F.Cu at (134.3, 105.1)
- added C1: CP1, Capacitor_THT:C_Disc_D3.8mm_W2.6mm_P2.50mm, F.Cu at (26.1, 60.4)
- added C3: CP1, Capacitor_THT:C_Disc_D3.8mm_W2.6mm_P2.50mm, F.Cu at (26.3, 86.5)
- added C4: CP1, Capacitor_THT:C_Disc_D3.8mm_W2.6mm_P2.50mm, F.Cu at (26.6, 113.4)
- added C6: CP1, Capacitor_THT:C_Disc_D3.8mm_W2.6mm_P2.50mm, F.Cu at (126.2, 42.8)
- added D1: LED, LED_THT:LED_D3.0mm, F.Cu at (141.7, 63.9)
- added D2: LED, LED_THT:LED_D3.0mm, F.Cu at (146.2, 63.9)
- added J12: Conn_01x04, Connector_PinHeader_2.54mm:PinHeader_1x04_P2.54mm_Vertical, F.Cu at (109.2, 38.3)
- added J8: Conn_01x08, Connector_PinHeader_2.54mm:PinHeader_1x08_P2.54mm_Vertical, F.Cu at (166.3, 116.7)
- added R1: R_Small_US, Resistor_THT:R_Axial_DIN0207_L6.3mm_D2.5mm_P10.16mm_Horizontal, F.Cu at (157.2, 115.5)
- added R2: R_Small_US, Resistor_THT:R_Axial_DIN0207_L6.3mm_D2.5mm_P10.16mm_Horizontal, F.Cu at (144.2, 115.5)
- added R3: R_Small_US, Resistor_THT:R_Axial_DIN0207_L6.3mm_D2.5mm_P10.16mm_Horizontal, F.Cu at (152.3, 68.0)
- added R4: R_Small_US, Resistor_THT:R_Axial_DIN0207_L6.3mm_D2.5mm_P10.16mm_Horizontal, F.Cu at (157.2, 68.0)
- added REF**: MountingHole_3mm_Pad_Via, MountingHole:MountingHole_3mm_Pad_Via, F.Cu at (25.3, 35.7)
- added REF**: MountingHole_3mm_Pad_Via, MountingHole:MountingHole_3mm_Pad_Via, F.Cu at (25.3, 145.7)
- added REF**: MountingHole_3mm_Pad_Via, MountingHole:MountingHole_3mm_Pad_Via, F.Cu at (168.8, 145.7)
- added REF**: MountingHole_3mm_Pad_Via, MountingHole:MountingHole_3mm_Pad_Via, F.Cu at (168.8, 35.7)
- added RN1: R_Network08, Resistor_THT:R_Array_SIP9, F.Cu at (135.6, 73.6)
- added RN2: R_Network08, Resistor_THT:R_Array_SIP9, F.Cu at (135.6, 93.6)
- added U3: 74LS245, Package_DIP:DIP-20_W7.62mm, F.Cu at (129.7, 105.8)
- added U4: 74LS173, Package_DIP:DIP-16_W7.62mm, F.Cu at (134.3, 127.7)
- added U5: 74LS173, Package_DIP:DIP-16_W7.62mm, F.Cu at (106.9, 127.7)
- added U6: 74LS138, Package_DIP:DIP-16_W7.62mm, F.Cu at (106.9, 95.9)
- added U8: 74LS138, Package_DIP:DIP-16_W7.62mm, F.Cu at (106.9, 83.0)
- C2: value CP_Small -> CP1; footprint Capacitor_THT:C_Radial_D5.0mm_H7.0mm_P2.00mm -> Capacitor_THT:C_Disc_D3.8mm_W2.6mm_P2.50mm
- C5: footprint Capacitor_THT:C_Radial_D5.0mm_H7.0mm_P2.00mm -> Capacitor_THT:CP_Radial_D8.0mm_P3.80mm
- J2: value Conn_01x08 -> Screw_Terminal_01x04; footprint Connector_PinHeader_2.54mm:PinHeader_1x08_P2.54mm_Vertical -> TerminalBlock_Phoenix:TerminalBlock_Phoenix_MKDS-1,5-4_1x04_P5.00mm_Horizontal
- J3: value Conn_01x10 -> Conn_01x25; footprint Connector_PinHeader_2.54mm:PinHeader_1x29_P2.54mm_Vertical -> Connector_PinHeader_2.54mm:PinHeader_1x25_P2.54mm_Vertical
- J4: value Conn_2x08 -> Screw_Terminal_01x04; footprint Connector_PinHeader_2.54mm:PinHeader_2x08_P2.54mm_Vertical -> TerminalBlock_Phoenix:TerminalBlock_Phoenix_MKDS-1,5-4_1x04_P5.00mm_Horizontal
- J5: value Conn_01x02 -> Conn_01x03; footprint Connector_PinHeader_2.54mm:PinHeader_1x02_P2.54mm_Vertical -> TerminalBlock_Phoenix:TerminalBlock_Phoenix_MKDS-1,5-3_1x03_P5.00mm_Horizontal
- moved C5 167.9 mm to (46.2, 38.0)
- moved J50 157.4 mm to (39.6, 37.5), turned to 180 degrees
- moved J4 144.6 mm to (73.3, 37.5), turned to 180 degrees
- moved BAR2 137.0 mm to (81.5, 134.5), turned to 270 degrees
- moved BAR3 126.2 mm to (107.6, 134.5), turned to 270 degrees
- moved J2 116.7 mm to (96.7, 37.5), turned to 180 degrees
- moved EEPROM4 98.8 mm to (64.3, 59.4), turned to 90 degrees
- moved BAR1 95.4 mm to (133.8, 134.5), turned to 270 degrees
- moved SW6 93.5 mm to (133.0, 36.0)
- moved J5 92.1 mm to (157.7, 37.5), turned to 180 degrees
- moved U2 87.7 mm to (106.6, 55.8), turned to 90 degrees
- moved U1 74.6 mm to (106.9, 68.0), turned to 90 degrees
- moved U7 74.6 mm to (131.0, 55.8), turned to 90 degrees
- moved RN14 72.1 mm to (136.6, 147.0), turned to 180 degrees
- moved C2 71.3 mm to (134.0, 62.6)
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Connections:
- net /FLAG1 renamed FLAG1
- net /FLAG2 renamed FLAG2
- net /FLAG3 renamed FLAG3
- net /STEP1 renamed STEP1
- net /STEP2 renamed STEP2
- net /STEP3 renamed STEP3
- BAR1 pad 1: /μ10 -> A_REGISTER_OUT
- BAR1 pad 10: /μ1 -> A_REGISTER_IN
- BAR1 pad 2: /μ9 -> IN_MUX_EN
- BAR1 pad 3: /μ8 -> TONE_REGISTER_IN
- BAR1 pad 4: /μ7 -> OUTPUT_REGISTER_IN
- BAR1 pad 5: /μ6 -> RAM_IN
- BAR1 pad 6: /μ5 -> MAR2_IN
- BAR1 pad 7: /μ4 -> MAR1_IN
- BAR1 pad 8: /μ3 -> SCRATCH_REGISTER_IN
- BAR1 pad 9: /μ2 -> B_REGISTER_IN
- BAR2 pad 1: /μ20 -> ALU_S0
- BAR2 pad 10: /μ11 -> SCRATCH_REGISTER_OUT
- BAR2 pad 2: /μ19 -> TONE_OCTAVE_1
- BAR2 pad 3: /μ18 -> TONE_OCTAVE_2
- BAR2 pad 4: /μ17 -> RAM_WRITE
- BAR2 pad 5: /D16 -> OUT_MUX_EN
- BAR2 pad 6: /μ15 -> ALU_OUT
- BAR2 pad 7: /μ14 -> PROGRAM_COUNTER_OUT
- BAR2 pad 8: /μ13 -> INSTRUCTION_REG_OUT
- BAR2 pad 9: /μ12 -> RAM_OUT
- BAR3 pad 1: /D30 -> FLAG_IN
- BAR3 pad 10: /μ21 -> ALU_S1
- BAR3 pad 2: /μ29 -> STEP_RESET
- BAR3 pad 3: /μ28 -> PROGRAM_COUNTER_ENABLE
- BAR3 pad 4: /μ27 -> INSTRUCTION_REG_IN
- BAR3 pad 5: /μ26 -> HALT
- BAR3 pad 6: /μ25 -> MASTER_RESET
- BAR3 pad 7: /μ24 -> ALU_MODE
- BAR3 pad 8: /μ23 -> ALU_S3
- BAR3 pad 9: /μ22 -> ALU_S2
- EEPROM1 pad 1: /INST8 -> INST7
- EEPROM1 pad 11: /μ1 -> ALU_MODE
- EEPROM1 pad 12: /μ2 -> ALU_S3
- EEPROM1 pad 13: /μ3 -> ALU_S2
- EEPROM1 pad 15: /μ4 -> ALU_S1
- EEPROM1 pad 16: /μ5 -> ALU_S0
- EEPROM1 pad 17: /μ6 -> TONE_OCTAVE_1
- EEPROM1 pad 18: /μ7 -> TONE_OCTAVE_2
- EEPROM1 pad 19: /μ8 -> RAM_WRITE
- EEPROM1 pad 2: /INST6 -> INST5
- EEPROM1 pad 21: /INST4 -> INST3
- EEPROM1 pad 23: /INST5 -> INST4
- EEPROM1 pad 24: /INST3 -> INST2
- EEPROM1 pad 25: /INST2 -> INST1
- EEPROM1 pad 26: /INST7 -> INST6
- EEPROM1 pad 3: /INST1 -> INST0
- EEPROM2 pad 1: /INST8 -> INST7
- EEPROM2 pad 11: /μ9 -> OUT_MUX_00
- EEPROM2 pad 12: /μ10 -> OUT_MUX_01
- EEPROM2 pad 13: /μ11 -> OUT_MUX_02
- EEPROM2 pad 15: /μ12 -> OUT_MUX_EN
- EEPROM2 pad 16: /μ13 -> IN_MUX_00
- EEPROM2 pad 17: /μ14 -> IN_MUX_01
- EEPROM2 pad 18: /μ15 -> IN_MUX_02
- EEPROM2 pad 19: /D16 -> IN_MUX_EN
- EEPROM2 pad 2: /INST6 -> INST5
- EEPROM2 pad 21: /INST4 -> INST3
- EEPROM2 pad 23: /INST5 -> INST4
- EEPROM2 pad 24: /INST3 -> INST2
- EEPROM2 pad 25: /INST2 -> INST1
- EEPROM2 pad 26: /INST7 -> INST6
- EEPROM2 pad 3: /INST1 -> INST0
- EEPROM4 pad 1: /INST8 -> INST7
- EEPROM4 pad 11: /μ25 -> JUMP
- EEPROM4 pad 12: /μ26 -> SET_CLOCK_FREQ
- EEPROM4 pad 13: /μ27 -> FLAG_IN
- EEPROM4 pad 15: /μ28 -> STEP_RESET
- EEPROM4 pad 16: /μ29 -> PROGRAM_COUNTER_ENABLE
- EEPROM4 pad 17: /FLAG_IN -> INSTRUCTION_REG_IN
- EEPROM4 pad 18: /μ31 -> HALT
- EEPROM4 pad 19: /μ32 -> MASTER_RESET
- EEPROM4 pad 2: /INST6 -> INST5
- EEPROM4 pad 21: /INST4 -> INST3
- EEPROM4 pad 23: /INST5 -> INST4
- EEPROM4 pad 24: /INST3 -> INST2
- EEPROM4 pad 25: /INST2 -> INST1
- EEPROM4 pad 26: /INST7 -> INST6
- EEPROM4 pad 3: /INST1 -> INST0
- J2 pad 1: /INST1 -> MASTER_RESET
- J2 pad 2: /INST2 -> MASTER_RESET
- J2 pad 3: /INST3 -> MASTER_RESET
- J2 pad 4: /INST4 -> MASTER_RESET
- J3 pad 1: /μ29 -> IN_MUX_EN
- J3 pad 10: /μ20 -> OUT_MUX_EN
- J3 pad 11: /μ19 -> ALU_OUT
- J3 pad 12: /μ18 -> PROGRAM_COUNTER_OUT
- J3 pad 13: /μ17 -> INSTRUCTION_REG_OUT
- J3 pad 14: /D16 -> RAM_OUT
- J3 pad 15: /μ15 -> SCRATCH_REGISTER_OUT
- J3 pad 16: /μ14 -> A_REGISTER_OUT
- J3 pad 17: /μ13 -> ALU_MODE
- J3 pad 18: /μ12 -> ALU_S3
- J3 pad 19: /μ11 -> ALU_S2
- J3 pad 2: /μ28 -> TONE_REGISTER_IN
- J3 pad 20: /μ10 -> ALU_S1
- J3 pad 21: /μ9 -> ALU_S0
- J3 pad 22: /μ8 -> TONE_OCTAVE_1
- J3 pad 23: /μ7 -> TONE_OCTAVE_2
- J3 pad 24: /μ6 -> RAM_WRITE
- J3 pad 25: /μ5 -> JUMP
- J3 pad 3: /μ27 -> OUTPUT_REGISTER_IN
- J3 pad 4: /μ26 -> RAM_IN
- J3 pad 5: /μ25 -> MAR2_IN
- J3 pad 6: /μ24 -> MAR1_IN
- J3 pad 7: /μ23 -> SCRATCH_REGISTER_IN
- J3 pad 8: /μ22 -> B_REGISTER_IN
- J3 pad 9: /μ21 -> A_REGISTER_IN
- J4 pad 1: /μ32 -> Net-(J4-Pad1)
- J4 pad 2: /μ32 -> Net-(J4-Pad1)
- J4 pad 3: /μ32 -> Net-(J4-Pad1)
- J4 pad 4: /μ32 -> Net-(J4-Pad1)
- J5 pad 1: Net-(J5-Pad1) -> CLOCK_IN
- J5 pad 2: Net-(J5-Pad1) -> HALT
- J50 pad 1: Net-(J50-Pad1) -> GND
- J50 pad 2: GND -> VCC
- SW6 pad 1: /μ32 -> MASTER_RESET
- U2 pad 10: /FLAG_IN -> FLAG_IN
- U2 pad 15: /μ32 -> MASTER_RESET
- U2 pad 9: /FLAG_IN -> FLAG_IN
- U7 pad 1: /μ32 -> MASTER_RESET
- U7 pad 10: Net-(J11-Pad4) -> (no net)
- U7 pad 11: Net-(J10-Pad1) -> (no net)
- U7 pad 13: Net-(J5-Pad1) -> CLOCK_IN
- U7 pad 2: Net-(J4-Pad10) -> Net-(J4-Pad1)
- U7 pad 3: Net-(J10-Pad4) -> (no net)
- U7 pad 4: Net-(J11-Pad1) -> (no net)
- U7 pad 5: Net-(J10-Pad3) -> (no net)
- U7 pad 6: Net-(J11-Pad2) -> (no net)
- U7 pad 8: Net-(J11-Pad3) -> (no net)
- U7 pad 9: Net-(J10-Pad2) -> (no net)
Routing:
- net VCC: track 0.00 -> 454.3 mm
- net MASTER_RESET: track 0.00 -> 295.7 mm, vias 0 -> 2
- net INSTRUCTION_REG_OUT: track 0.00 -> 254.7 mm
- net OUT_MUX_EN: track 0.00 -> 253.3 mm, vias 0 -> 1
- net SCRATCH_REGISTER_OUT: track 0.00 -> 242.8 mm
- net RAM_OUT: track 0.00 -> 231.7 mm
- net INST0: track 0.00 -> 231.2 mm
- net RAM_WRITE: track 0.00 -> 221.7 mm
- net IN_MUX_EN: track 0.00 -> 219.7 mm, vias 0 -> 2
- net TONE_OCTAVE_2: track 0.00 -> 215.6 mm
- net PROGRAM_COUNTER_OUT: track 0.00 -> 210.7 mm
- net INST1: track 0.00 -> 209.7 mm
- net HALT: track 0.00 -> 209.7 mm, vias 0 -> 1
- net TONE_OCTAVE_1: track 0.00 -> 208.1 mm
- net SET_CLOCK_FREQ: track 0.00 -> 206.9 mm
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- added copper zone on B.Cu, net GND
Other:
- board outline added: 150.6 x 117.1 mm
- copper layers 2 -> 4
- board text added: "(Active High)"
- board text added: "(Active Low)"
- board text added: "+"
- board text added: "-"
- board text added: "AI"
- board text added: "AO"
- board text added: "B0"
- board text added: "B1"
- board text added: "B2"
- board text added: "B3"
- board text added: "B4"
- board text added: "B5"
- board text added: "B6"
- board text added: "B7"
- board text added: "BI"
- board text added: "Buffer"
- board text added: "CE"
- board text added: "CLK"
- board text added: "CLOCK"
- board text added: "CO"
- board text added: "CRY"
- board text added: "Demultiplexer"
- board text added: "EQ"
- board text added: "FI"
- board text added: "FLAG1"
- board text added: "FLAG2"
- board text added: "FLAG3"
- board text added: "FLAG4"
- board text added: "FLG4"
- board text added: "FREQ"
- board text added: "Flags Register"
- board text added: "GT"
- board text added: "HALT"
- board text added: "HLT"
- board text added: "II"
- board text added: "IME"
- board text added: "INST0"
- board text added: "INST1"
- board text added: "INST2"
- board text added: "INST3"
- board text added: "INST4"
- board text added: "INST5"
- board text added: "INST6"
- board text added: "INST7"
- board text added: "IO"
- board text added: "Inst. Register"
- board text added: "Inverter"
- board text added: "JP"
- board text added: "JUMP"
- board text added: "LO"
- board text added: "MA1"
- board text added: "MA2"
- board text added: "MASTER RESET"
- board text added: "MD"
- board text added: "MR"
- board text added: "OI"
- board text added: "OME"
- board text added: "RESET"
- board text added: "RI"
- board text added: "RO"
- board text added: "RW"
- board text added: "S0"
- board text added: "S1"
- board text added: "S2"
- board text added: "S3"
- board text added: "SI"
- board text added: "SO"
- board text added: "SR"
- board text added: "STEP1"
- board text added: "STEP2"
- board text added: "STEP3"
- board text added: "Step Counter"
- board text added: "T01"
- board text added: "T02"
- board text added: "TI"
- board text added: "TO1"
- board text added: "TO2"
- board text added: "x"

Commit message: [Micocode] Updating Control - WIP
Routing:
- net CLOCK: track 179.1 -> 178.0 mm
- net INSTRUCTION_REG_IN: track 181.9 -> 181.3 mm
- net FLAG4: track 203.0 -> 202.5 mm
