File: Modules/control-module/control.sch (KiCad schematic (older format))
At the start: 29 parts, among them J1 Conn_01x02, J10 Conn_1x04, J11 Conn_1x04, J2 Conn_01x08, J3 Conn_01x10, J4 Conn_2x08, J5 Conn_01x02, J50 Screw_Terminal_01x02, J7 Conn_1x08, J9 Conn_01x02, SW6 SW_Push, U1 74LS161, U2 74LS173, U7 74LS04

Commit message: [General] Updates
Parts:
- removed C2: CP_Small, Capacitor_THT:C_Radial_D5.0mm_H7.0mm_P2.00mm, symbol Device:CP_Small
- removed D79, D80: LED, LED_THT:LED_D3.0mm, symbol Device:LED
- removed EEPROM3: AT28C256, 8-bit-computer:DIP_Socket-40_W11.9_W12.7_W15.24_W17.78_W18.5_3M_240-1280-00-0602J, symbol control-rescue:AT28C256-AT28C256-CONTROL_LOGIC-rescue
- removed J1, J9: Conn_01x02, Connector_PinHeader_2.54mm:PinHeader_1x02_P2.54mm_Vertical, symbol Connector_Generic:Conn_01x02
- removed J10, J11: Conn_1x04, Connector_PinHeader_2.54mm:PinHeader_1x04_P2.54mm_Vertical, symbol Connector_Generic:Conn_01x04
- removed J2: Conn_01x08, Connector_PinHeader_2.54mm:PinHeader_1x08_P2.54mm_Vertical, symbol Connector_Generic:Conn_01x08
- removed J4: Conn_2x08, Connector_PinHeader_2.54mm:PinHeader_2x08_P2.54mm_Vertical, symbol Connector_Generic:Conn_02x08_Top_Bottom
- removed J7: Conn_1x08, Connector_PinHeader_2.54mm:PinHeader_1x08_P2.54mm_Vertical, symbol Connector_Generic:Conn_01x08
- removed unit 2 of U7
- removed unit 3 of U7
- removed unit 4 of U7
- removed unit 5 of U7
- added BAR4, BAR5: HDSP-4850_2, Display:HDSP-4850, symbol LED:HDSP-4830_2
- added C1, C2, C3, C4, C6: CP1, Capacitor_THT:C_Disc_D3.8mm_W2.6mm_P2.50mm, symbol Device:CP1
- added D1, D2: LED, LED_THT:LED_D3.0mm, symbol Device:LED
- added J12: Conn_01x04, Connector_PinHeader_2.54mm:PinHeader_1x04_P2.54mm_Vertical, symbol Connector_Generic:Conn_01x04
- added J2, J4: Screw_Terminal_01x04, TerminalBlock_Phoenix:TerminalBlock_Phoenix_MKDS-1,5-4_1x04_P5.00mm_Horizontal, symbol Connector:Screw_Terminal_01x04
- added J8: Conn_01x08, Connector_PinHeader_2.54mm:PinHeader_1x08_P2.54mm_Vertical, symbol Connector_Generic:Conn_01x08
- added R1, R2, R3, R4: R_Small_US, Resistor_THT:R_Axial_DIN0207_L6.3mm_D2.5mm_P10.16mm_Horizontal, symbol Device:R_Small_US
- added RN1, RN2: R_Network08, Resistor_THT:R_Array_SIP9, symbol Device:R_Network08
- added U3: 74LS245, Package_DIP:DIP-20_W7.62mm, symbol 74xx:74LS245
- added U4, U5: 74LS173, Package_DIP:DIP-16_W7.62mm, symbol 74xx:74LS173
- added U6, U8: 74LS138, Package_DIP:DIP-16_W7.62mm, symbol 74xx:74LS138
- C5: footprint Capacitor_THT:C_Radial_D5.0mm_H7.0mm_P2.00mm -> Capacitor_THT:CP_Radial_D8.0mm_P3.80mm
- J3: value Conn_01x10 -> Conn_01x25; footprint Connector_PinHeader_2.54mm:PinHeader_1x29_P2.54mm_Vertical -> Connector_PinHeader_2.54mm:PinHeader_1x25_P2.54mm_Vertical; symbol Connector_Generic:Conn_01x29 -> Connector_Generic:Conn_01x25
- J5: value Conn_01x02 -> Conn_01x03; footprint Connector_PinHeader_2.54mm:PinHeader_1x02_P2.54mm_Vertical -> TerminalBlock_Phoenix:TerminalBlock_Phoenix_MKDS-1,5-3_1x03_P5.00mm_Horizontal; symbol Connector_Generic:Conn_01x02 -> Connector:Screw_Terminal_01x03
Connections:
- net labels added: ALU_MODE, ALU_OUT, ALU_S0, ALU_S1, ALU_S2, ALU_S3, A_REGISTER_IN, A_REGISTER_OUT, BUS_00, BUS_01, BUS_02, BUS_03, BUS_04, BUS_05, BUS_06, BUS_07, B_REGISTER_IN, CLOCK_IN, HALT, INST0, INSTRUCTION_REG_IN, INSTRUCTION_REG_OUT, IN_MUX_00, IN_MUX_01, IN_MUX_02, IN_MUX_EN, JUMP, MAR1_IN, MAR2_IN, MASTER_RESET, OUTPUT_REGISTER_IN, OUT_MUX_00, OUT_MUX_01, OUT_MUX_02, OUT_MUX_EN, PROGRAM_COUNTER_ENABLE, PROGRAM_COUNTER_OUT, RAM_IN, RAM_OUT, RAM_WRITE, SCRATCH_REGISTER_IN, SCRATCH_REGISTER_OUT, SET_CLOCK_FREQ, TONE_OCTAVE_1, TONE_OCTAVE_2, TONE_REGISTER_IN
- net labels removed: D1, D10, D11, D12, D13, D14, D15, D16, D17, D18, D19, D2, D20, D21, D22, D23, D24, D25, D26, D27, D28, D29, D3, D30, D31, D32, D4, D5, D6, D7, D8, D9, INST8, μ1, μ10, μ11, μ12, μ13, μ14, μ15, μ16, μ17, μ18, μ19, μ2, μ20, μ21, μ22, μ23, μ24, μ25, μ26, μ27, μ28, μ29, μ3, μ31, μ32, μ4, μ5, μ6, μ7, μ8, μ9
- wire segments 249 -> 105
- no-connect marks 6 -> 11
Other:
- note added: "4-bit Storage"
- note added: "ALU / OCTAVE / RAM WRITE"
- note added: "BUS CONNECT"
- note added: "Buffered Output"
- note added: "CLOCK"
- note added: "CONTROL LINE OUTPUT"
- note added: "C[1..3] 0.1uF ceramic"
- note added: "Connections"
- note added: "FLAGS\nINPUT"
- note added: "INSTRUCTION REGISTER"
- note added: "MAIN CONTROLS"
- note added: "Microcode EEPROMs"
- note added: "Multiplexer Control (READ/WRITE)"
- note added: "Output 2 Bus MUX (Active LOW outputs)"
- note added: "RESET"
- note added: "Smoothing Capacitors"
- note added: "Write MUX (Active LOW outputs)"
- note removed: "CONNECTIONS"
- note removed: "EEPROMS"
- note removed: "RESET & INVERT"
- note removed: "SPARE INVERTER PINS"
- moved on the sheet: C5, EEPROM1, EEPROM2, EEPROM4, J50, U1, U2
