File: modules/stack-pointer/stack-pointer.sch (KiCad schematic (older format))
At the start: 11 parts

Commit message: saving
Parts:
- removed C1: CL05A106MQ5NUNC, Capacitor_SMD:C_0402_1005Metric, symbol Device:C
- removed C5: SMD-ECAP-5x5.8, Capacitor_SMD:CP_Elec_5x5.8, symbol Device:CP1_Small
- removed U?: 74LS283, symbol 74xx:74LS283
- removed U? (x4): SN74HC193DR, Package_SO:SO-16_3.9x9.9mm_P1.27mm, symbol 74xx:74LS193
- added C1: SMD-ECAP-5x5.8, Capacitor_SMD:CP_Elec_5x5.8, symbol Device:CP1_Small
- added C2, C3, C4, C5, C6, C7, C8, C9: CL05A106MQ5NUNC, Capacitor_SMD:C_0402_1005Metric, symbol Device:C
- added D10, D12, D2, D4, D7: 19-217/BHC-ZL1M2RY/3T, LED_SMD:LED_0603_1608Metric, symbol Device:LED
- added D11, D13, D15, D16, D17, D18, D19, D20, D21, D22, D23, D3, D5, D8: 19-217/GHC-YR1S2/3T, LED_SMD:LED_0603_1608Metric, symbol Device:LED
- added D14, D6: NCD0805R1, LED_SMD:LED_0805_2012Metric, symbol Device:LED
- added J1: Conn_01x09, Connector_PinHeader_2.54mm:PinHeader_1x09_P2.54mm_Vertical, symbol Connector_Generic:Conn_01x09
- added J2, J3: Conn_01x16, Connector_PinHeader_2.54mm:PinHeader_1x16_P2.54mm_Vertical, symbol Connector_Generic:Conn_01x16
- added R10, R11, R12, R13, R14, R15, R16, R17, R18, R19, R2, R20, R21, R22, R23, R3, R4, R5, R6, R7, R8: 0402WGF1001TCE, Resistor_SMD:R_0402_1005Metric, symbol Device:R_Small_US
- added U1, U4, U5, U8: 74LS169, Package_DIP:DIP-16_W7.62mm, symbol 74xx:74LS169
- added U2, U3, U6, U7: 74HC245D,653, Package_SO:SO-20_12.8x7.5mm_P1.27mm, symbol 74xx:74LS245
- D1: JCLC (none) -> C72043
- D9: value 19-217/BHC-ZL1M2RY/3T -> 19-217/GHC-YR1S2/3T; Color BLU -> GRN; JCLC (none) -> C72043; JLCPCB C72041 -> C72043
- R1, R9: JCLC (none) -> C11702
Connections:
- net labels added: BUS2_00, BUS2_01, BUS2_02, BUS2_03, BUS2_04, BUS2_05, BUS2_06, BUS2_07, BUS2_08, BUS2_09, BUS2_10, BUS2_11, BUS2_12, BUS2_13, BUS2_14, BUS2_15, BUS_00, BUS_01, BUS_02, BUS_03, BUS_04, BUS_05, BUS_06, BUS_07, BUS_08, BUS_09, BUS_10, BUS_11, BUS_12, BUS_13, BUS_14, BUS_15, CARRY, CLOCK, INC_DEC, Q0, Q1, Q10, Q11, Q12, Q13, Q14, Q15, Q2, Q3, Q4, Q5, Q6, Q7, Q8, Q9, ~ADR_BUS_1, ~ADR_BUS_2, ~EN, ~LOAD
- net labels removed: A0, EN
- wire segments 0 -> 16
Other:
- note added: "INC\n————\n1 - UP\n0 - DOWN"
