File: modules/01_BACKPLANES/FULL-assembly-backplane/FULL-assembly-backplane.kicad_pcb (KiCad board)
At the start: 2 copper layers, 224.5 x 230.1 mm, 34 parts, among them J1 Conn_01x16, J10 Conn_01x16, J11 Conn_01x16, J12 Conn_01x16, J13 Conn_01x16, J14 Conn_01x16, J15 Conn_01x16, J16 Conn_01x16, J17 Conn_01x16, J18 Conn_01x11, J19 Conn_01x11, J2 Conn_01x16, J20 Conn_01x11, J21 Conn_01x11, J22 Conn_01x37, J23 Conn_01x04, J24 Conn_01x04, J3 Conn_01x08, J32 Conn_01x32, J33 Conn_01x32, J34 Conn_01x32, J35 Conn_01x32, J36 Conn_01x32, J37 Conn_01x26, J4 Conn_01x08, J5 Conn_01x16, J6 Conn_01x16, J7 Conn_01x16, J8 Conn_01x16, J9 Conn_01x16

Commit message: biggggg update and react app
Parts:
- removed the J1 at (178.3, 124.5)
- removed the J2 at (221.5, 124.5)
- removed J22: Conn_01x37, Connector_PinSocket_2.54mm:PinSocket_1x40_P2.54mm_Vertical
- removed J23, J24: Conn_01x04, Connector_PinHeader_2.54mm:PinHeader_1x04_P2.54mm_Vertical
- removed the J3 at (178.3, 157.5)
- removed REF** (x4): MountingHole_3mm_Pad_Via, MountingHole:MountingHole_3mm_Pad_Via
- added J1: Conn_01x16, Connector_PinHeader_2.54mm:PinHeader_1x16_P2.54mm_Vertical, F.Cu at (400.3, 94.7)
- added J1: Conn_01x09, Connector_PinHeader_2.54mm:PinHeader_1x09_P2.54mm_Vertical, B.Cu at (348.0, 157.7)
- added J1: Conn_01x08, Connector_PinHeader_2.54mm:PinHeader_1x08_P2.54mm_Vertical, B.Cu at (340.9, 16.8)
- added J1: Conn_01x04, Connector_PinHeader_2.54mm:PinHeader_1x04_P2.54mm_Vertical, B.Cu at (365.0, 169.4)
- added J1: Conn_01x10, Connector_PinHeader_2.54mm:PinHeader_1x10_P2.54mm_Vertical, B.Cu at (658.4, 117.6)
- added J2: Conn_01x16, Connector_PinHeader_2.54mm:PinHeader_1x16_P2.54mm_Vertical, F.Cu at (443.5, 94.7)
- added J2: Conn_01x09, Connector_PinHeader_2.54mm:PinHeader_1x09_P2.54mm_Vertical, B.Cu at (351.3, 201.9)
- added J2: Conn_01x08, Connector_PinHeader_2.54mm:PinHeader_1x08_P2.54mm_Vertical, B.Cu at (370.1, 157.7)
- added J2: Conn_01x23, Connector_PinHeader_2.54mm:PinHeader_1x23_P2.54mm_Vertical, B.Cu at (328.7, 79.8)
- added J2: Conn_01x08, Connector_PinHeader_2.54mm:PinHeader_1x08_P2.54mm_Vertical, B.Cu at (676.1, 145.5)
- added J25: Conn_01x32, Connector_PinSocket_2.54mm:PinSocket_1x32_P2.54mm_Vertical, F.Cu at (126.7, 165.4)
- added J26: Conn_01x32, Connector_PinSocket_2.54mm:PinSocket_1x32_P2.54mm_Vertical, F.Cu at (126.7, 191.3)
- added J3: Conn_01x08, Connector_PinHeader_2.54mm:PinHeader_1x08_P2.54mm_Vertical, F.Cu at (400.3, 127.8)
- added J3: Conn_01x07, Connector_PinHeader_2.54mm:PinHeader_1x07_P2.54mm_Vertical, B.Cu at (414.0, 44.7)
- added J3: Conn_01x02, Connector_PinHeader_2.54mm:PinHeader_1x02_P2.54mm_Vertical, B.Cu at (701.5, 117.6)
- added J43: Barrel_Jack, Connector_BarrelJack:BarrelJack_Horizontal, F.Cu at (41.3, 172.0)
- moved J37 238.4 mm to (43.2, 69.6)
- moved J5 232.8 mm to (70.6, 61.7)
- moved J4 224.0 mm to (468.9, 127.8)
- moved J11 218.0 mm to (70.6, 116.8)
- moved J18 207.0 mm to (245.1, 18.0)
- moved J6 207.0 mm to (264.4, 52.1)
- moved J7 207.0 mm to (219.7, 52.1)
- moved J21 176.7 mm to (245.1, 110.5)
- moved J12 176.7 mm to (264.4, 144.5)
- moved J13 176.5 mm to (219.5, 144.5)
- moved J17 147.4 mm to (365.8, 91.7), turned to 270 degrees
- moved J8 134.3 mm to (70.6, 70.4), turned to 0 degrees
- moved J10 111.6 mm to (219.7, 98.3)
- moved J19 111.6 mm to (245.1, 64.3)
- moved J9 111.6 mm to (264.4, 98.3)
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Connections:
- net /BUS0 renamed BUS0
- net /BUS1 renamed BUS1
- net /BUS2 renamed BUS2
- net /BUS3 renamed BUS3
- net /BUS4 renamed BUS4
- net /BUS5 renamed BUS5
- net /BUS6 renamed BUS6
- net /BUS7 renamed BUS7
- net /IN_BRW renamed Net-(J19-Pad1)
- net /IN_CRY renamed Net-(J19-Pad2)
- net /IN_DEC renamed Net-(J19-Pad7)
- net /IN_INC renamed Net-(J19-Pad6)
- net /L0 renamed L0
- net /L1 renamed L1
- net /L2 renamed L2
- net /L3 renamed L3
- net /L4 renamed L4
- net /L5 renamed L5
- net /L6 renamed L6
- net /L7 renamed L7
- net /M0 renamed M0
- net /M1 renamed M1
- net /M2 renamed M2
- net /M3 renamed M3
- net /M4 renamed M4
- net /M5 renamed M5
- net /M6 renamed M6
- net /M7 renamed M7
- net /MAR_BRW renamed Net-(J20-Pad1)
- net /MAR_CRY renamed Net-(J20-Pad2)
- net /MAR_DEC renamed Net-(J20-Pad7)
- net /MAR_INC renamed Net-(J20-Pad6)
- net /PC_BRW renamed Net-(J21-Pad1)
- net /PC_CRY renamed Net-(J21-Pad2)
- net /RESET renamed RESET
- net /SP_BRW renamed Net-(J18-Pad1)
- net /SP_CRY renamed Net-(J18-Pad2)
- net /~IN_BO renamed ~IN_BO
- net /~MAR_BO renamed ~MAR_BO
- net /~PC_BO renamed ~PC_BO
- net /~SP_BO renamed ~SP_BO
- J18 pad 3: /~SP_AD -> ~SP_ADDR
- J18 pad 5: /~SP_LD -> ~LD_STACK_P
- J18 pad 6: /SP_INC -> SP_INC
- J18 pad 7: /SP_DEC -> SP_DEC
- J19 pad 3: /~IN_AD -> Net-(J19-Pad3)
- J19 pad 5: /~IN_LD -> ~IN_LD
- J20 pad 3: /~MAR_AD -> Net-(J20-Pad3)
- J20 pad 5: /~MAR_LD -> ~MAR_LD
- J21 pad 3: /~PC_AD -> ~PC_ADDR
- J21 pad 5: /~PC_LD -> ~PC_LD
- J21 pad 6: /PC_INC -> PC_INC
- J21 pad 7: /PC_DEC -> PC_DEC
- J32 pad 1: MSB_O1 -> MSB_C
- J32 pad 2: LSB_O1 -> LSB_C
- J32 pad 3: O1 -> O_C
- J32 pad 4: I1 -> I_C
- J33 pad 1: MSB_O2 -> MSB_D
- J33 pad 2: LSB_O2 -> LSB_D
- J33 pad 3: O2 -> O_D
- J33 pad 4: I2 -> I_D
- J34 pad 1: MSB_O3 -> MSB_E
- J34 pad 2: LSB_O3 -> LSB_E
- J34 pad 3: O3 -> O_E
- J34 pad 4: I3 -> I_E
- J35 pad 1: MSB_O4 -> MSB_F
- J35 pad 2: LSB_O4 -> LSB_F
- J35 pad 3: O4 -> O_F
- J35 pad 4: I4 -> I_F
- J36 pad 1: MSB_O5 -> MSB_SCR_0
- J36 pad 2: LSB_O5 -> LSB_SCR_0
- J36 pad 3: O5 -> O_SCR_0
- J36 pad 4: I5 -> I_SCR_0
- J4 pad 1: /TX_SEL -> TX_SEL
- J4 pad 2: /TX_LSB -> TX_LS_IN
- J4 pad 3: /TX_MSB -> TX_MSB_IN
- J4 pad 4: /~TX_LSBO -> ~TX_LSB
- J4 pad 5: /~TX_MSBO -> ~TX_MSB
- J4 pad 6: /~TX_ADDO -> ~TX_ADDR
Routing:
- net CLOCK: track 724.8 -> 0.00 mm, vias 6 -> 0
- net L0: track 597.2 -> 0.00 mm, vias 2 -> 0
- net L1: track 592.2 -> 0.00 mm, vias 2 -> 0
- net L2: track 586.1 -> 0.00 mm, vias 2 -> 0
- net L3: track 585.3 -> 0.00 mm, vias 2 -> 0
- net L4: track 582.0 -> 0.00 mm, vias 2 -> 0
- net L5: track 578.7 -> 0.00 mm, vias 2 -> 0
- net BUS7: track 576.5 -> 0.00 mm, vias 1 -> 0
- net L6: track 575.4 -> 0.00 mm, vias 2 -> 0
- net L7: track 572.2 -> 0.00 mm, vias 2 -> 0
- net M0: track 568.9 -> 0.00 mm, vias 2 -> 0
- net BUS6: track 568.6 -> 0.00 mm, vias 1 -> 0
- net M1: track 566.1 -> 0.00 mm, vias 2 -> 0
- net M2: track 564.1 -> 0.00 mm, vias 2 -> 0
- net M3: track 561.7 -> 0.00 mm, vias 2 -> 0
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- removed copper zone on F.Cu, net GND
- removed copper zone on B.Cu, net VCC
Other:
- board outline removed
- board text added: "992k RAM | 32K ROM"
- board text added: "ALU"
- board text added: "ASL"
- board text added: "ASR"
- board text added: "C"
- board text added: "CF"
- board text added: "CONSTANT"
- board text added: "D"
- board text added: "E"
- board text added: "EQF"
- board text added: "F"
- board text added: "F0"
- board text added: "F1"
- board text added: "F2"
- board text added: "F3"
- board text added: "FI"
- board text added: "FI0"
- board text added: "FI6"
- board text added: "FRI"
- board text added: "GTF"
- board text added: "HT"
- board text added: "IO0"
- board text added: "IO1"
- board text added: "IO2"
- board text added: "IO3"
- board text added: "IO4"
- board text added: "IO5"
- board text added: "IO6"
- board text added: "IO7"
- board text added: "Interrupt Flags"
- board text added: "LB"
- board text added: "LCI"
- board text added: "LTF"
- board text added: "MD"
- board text added: "MEMORY"
- board text added: "MR"
- board text added: "OF"
- board text added: "SCRATCH 0"
- board text added: "SCRATCH 1"
- board text added: "SF"
- board text added: "Xtal"
- board text added: "ZF"
- board text added: "~CL0"
- board text added: "~CL1"
- board text added: "~CL2"
- board text added: "~CP"
- board text added: "~CS"
- board text added: "~DIV"
- board text added: "~DS"
- board text added: "~IR0"
- board text added: "~IR1"
- board text added: "~IR2"
- board text added: "~LO"
- board text added: "~MR"
- board text added: "~OE"
- board text added: "~REQ0"
- board text added: "~REQ1"
- board text added: "~WE"
- board text removed: "+Vcc"
- board text removed: "-Gnd"
- board text removed: "I1"
- board text removed: "I2"
- board text removed: "I3"
- board text removed: "I4"
- board text removed: "I5"
- board text removed: "MAR0"
- board text removed: "MAR1"
- board text removed: "MAR10"
- board text removed: "MAR11"
- board text removed: "MAR12"
- board text removed: "MAR13"
- board text removed: "MAR14"
- board text removed: "MAR15"
- board text removed: "MAR2"
- board text removed: "MAR3"
- board text removed: "MAR4"
- board text removed: "MAR5"
- board text removed: "MAR6"
- board text removed: "MAR7"
- board text removed: "MAR8"
- board text removed: "MAR9"
- board text removed: "PC_DEC"
- board text removed: "PC_INC"
- board text removed: "RESET"
- board text removed: "SP_DEC"
- board text removed: "SP_INC"
- board text removed: "TX_LSB"
- board text removed: "TX_MSB"
- board text removed: "TX_SEL"
- board text removed: "~IN_AD"
- board text removed: "~IN_LD"
- board text removed: "~LSB1"
- board text removed: "~LSB2"
- board text removed: "~LSB3"
- board text removed: "~LSB4"
- board text removed: "~LSB5"
- board text removed: "~MAR_AD"
- board text removed: "~MAR_LD"
- board text removed: "~MSB1"
- board text removed: "~MSB2"
- board text removed: "~MSB3"
- board text removed: "~MSB4"
- board text removed: "~MSB5"
- board text removed: "~O1"
- board text removed: "~O2"
- board text removed: "~O3"
- board text removed: "~O4"
- board text removed: "~O5"
- board text removed: "~PC_AD"
- board text removed: "~PC_LD"
- board text removed: "~SP_AD"
- board text removed: "~SP_LD"
- board text removed: "~TX_ADD0"
- board text removed: "~TX_LSBO"
- board text removed: "~TX_MSBO"
