File: PCB-Modules/99_IN PROGRESS/control-unit-grp-1/control-unit.kicad_pcb (KiCad board)
At the start: 4 copper layers, 11 parts, among them J1 Conn_01x22, J2 Conn_01x22, J3 Conn_01x14, U2 74LS154, U3 74LS08, U4 74LS258, U40 74LS154, U5 74LS258, U6 74LS154, U7 74HC04, U8 74LS157

Commit message: large save haahh
Parts:
- removed J1, J2: Conn_01x22, Connector_PinHeader_2.54mm:PinHeader_1x22_P2.54mm_Vertical
- removed J3: Conn_01x14, Connector_PinHeader_2.54mm:PinHeader_1x14_P2.54mm_Vertical
- removed U40: 74LS154, Package_SO:TSSOP-24_4.4x7.8mm_P0.65mm
- removed U8: 74LS157, Package_SO:TSSOP-16_4.4x5mm_P0.65mm
- added U1: 74LS154, Package_SO:TSSOP-24_4.4x7.8mm_P0.65mm, F.Cu at (120.1, 64.1)
- U4: value 74LS258 -> 74HC04; footprint Package_SO:TSSOP-16_4.4x5mm_P0.65mm -> Package_SO:TSSOP-14_4.4x5mm_P0.65mm
- U5: value 74LS258 -> 74LS157
- U6: value 74LS154 -> 74LS258; footprint Package_SO:TSSOP-24_4.4x7.8mm_P0.65mm -> Package_SO:TSSOP-16_4.4x5mm_P0.65mm
- U7: value 74HC04 -> 74LS258; footprint Package_SO:TSSOP-14_4.4x5mm_P0.65mm -> Package_SO:TSSOP-16_4.4x5mm_P0.65mm
- moved U2 26.0 mm to (128.9, 64.1), turned to 0 degrees
- moved U3 25.0 mm to (137.6, 62.7), turned to 0 degrees
- moved U4 17.0 mm to (146.4, 62.7), turned to 0 degrees
- moved U7 13.9 mm to (137.6, 69.3), turned to 0 degrees
- moved U6 13.3 mm to (163.9, 62.7), turned to 0 degrees
- moved U5 11.6 mm to (155.1, 62.7), turned to 0 degrees
Connections:
- U4 pad 1: ~SHIFT_A_RIGHT -> ~ALU_MODE_0_CARRY_IN_EN
- U4 pad 10: GND -> Net-(U4-Pad10)
- U4 pad 11: GND -> Net-(U4-Pad11)
- U4 pad 13: GND -> Net-(U4-Pad13)
- U4 pad 14: GND -> VCC
- U4 pad 2: GND -> Net-(U3-Pad13)
- U4 pad 3: VCC -> Net-(U4-Pad3)
- U4 pad 4: SHA_SEL_01 -> Net-(U4-Pad4)
- U4 pad 5: VCC -> (no net)
- U4 pad 6: GND -> (no net)
- U4 pad 7: SHA_SEL_00 -> GND
- U4 pad 8: GND -> Net-(U4-Pad8)
- U5 pad 1: ~LOAD_A_REGISTER -> Net-(U3-Pad6)
- U5 pad 11: GND -> EEPROM_2
- U5 pad 12: Net-(U5-Pad12) -> ALU_FUNC_3
- U5 pad 14: GND -> EEPROM_3
- U5 pad 15: ~LOAD_A_REGISTER -> GND
- U5 pad 2: VCC -> EEPROM_0
- U5 pad 4: SHA_SEL_01 -> ALU_FUNC_0
- U5 pad 5: VCC -> EEPROM_1
- U5 pad 7: SHA_SEL_00 -> ALU_FUNC_1
- U5 pad 9: Net-(U5-Pad9) -> ALU_FUNC_2
- U6 pad 1: ~ALU_FLAG_REG_IN -> ~SHIFT_A_RIGHT
- U6 pad 10: ~JUMP_JNB_JAE_JNC -> GND
- U6 pad 11: ~JUMP_JBE_JNA -> GND
- U6 pad 12: GND -> Net-(U6-Pad12)
- U6 pad 13: ~JUMP_JA_JNBE -> GND
- U6 pad 14: ~JUMP_JL_JNG -> GND
- U6 pad 15: ~JUMP_JGE_JNL -> Net-(U3-Pad3)
- U6 pad 16: ~JUMP_JLE_JNG -> VCC
- U6 pad 2: ~JUMP -> GND
- U6 pad 3: ~JUMP_JO -> VCC
- U6 pad 4: ~JUMP_JNO -> SHA_SEL_01
- U6 pad 5: ~JUMP_JS -> VCC
- U6 pad 6: ~JUMP_JNS -> GND
- U6 pad 7: ~JUMP_JE_JZ -> SHA_SEL_00
- U6 pad 8: ~JUMP_JNE_JNZ -> GND
- U6 pad 9: ~JUMP_JB_JNAE_JC -> Net-(U6-Pad9)
- U7 pad 1: ~ALU_MODE_0_CARRY_IN_EN -> ~LOAD_A_REGISTER
- U7 pad 10: Net-(U7-Pad10) -> GND
- U7 pad 11: Net-(U7-Pad11) -> GND
- U7 pad 13: Net-(U7-Pad13) -> GND
- U7 pad 14: VCC -> GND
- U7 pad 2: Net-(U3-Pad13) -> VCC
- U7 pad 3: Net-(U7-Pad3) -> GND
- U7 pad 4: Net-(U7-Pad4) -> SHA_SEL_01
- U7 pad 5: (no net) -> VCC
- U7 pad 6: (no net) -> GND
- U7 pad 7: GND -> SHA_SEL_00
- U7 pad 8: Net-(U7-Pad8) -> GND
Routing:
- net EEPROM_2: track 86.2 -> 0.00 mm, vias 4 -> 0
- net EEPROM_3: track 85.2 -> 0.00 mm, vias 2 -> 0
- net EEPROM_1: track 56.2 -> 0.00 mm, vias 2 -> 0
- net ~LOAD_A_REGISTER: track 55.8 -> 0.00 mm
- net EEPROM_0: track 55.3 -> 0.00 mm, vias 2 -> 0
- net ~ALU_FLAG_REG_IN: track 48.2 -> 0.00 mm
- net ~JUMP: track 46.7 -> 0.00 mm
- net ~JUMP_JO: track 44.9 -> 0.00 mm
- net ~SET_INTERRUPT_FREQ: track 44.5 -> 0.00 mm
- net ~JUMP_JNO: track 43.0 -> 0.00 mm
- net ~JUMP_JS: track 41.1 -> 0.00 mm
- net ~TRANSMIT_UART: track 41.0 -> 0.00 mm
- net ~JUMP_JNS: track 39.2 -> 0.00 mm
- net ~WRITE_MEMORY: track 37.5 -> 0.00 mm
- net ~JUMP_JE_JZ: track 37.3 -> 0.00 mm
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