File: PCB-Modules/99_IN PROGRESS/control-unit-grp-1/control-unit.sch (KiCad schematic (older format))
At the start: 0 parts

Commit message: large save haahh
Parts:
- added J1, J2: Conn_01x22, Connector_PinHeader_2.54mm:PinHeader_1x22_P2.54mm_Vertical, symbol Connector_Generic:Conn_01x22
- added J3: Conn_01x14, Connector_PinHeader_2.54mm:PinHeader_1x14_P2.54mm_Vertical, symbol Connector_Generic:Conn_01x14
- added U1, U2: 74LS154, Package_SO:TSSOP-24_4.4x7.8mm_P0.65mm, symbol 74xx:74LS154
- added U3: 74LS08, Package_SO:TSSOP-14_4.4x5mm_P0.65mm, symbol 74xx:74LS08
- added U4: 74HC04, Package_SO:TSSOP-14_4.4x5mm_P0.65mm, symbol 74xx:74HC04
- added U5: 74LS157, Package_SO:TSSOP-16_4.4x5mm_P0.65mm, symbol 74xx:74LS157
- added U6, U7: 74LS258, Package_SO:TSSOP-16_4.4x5mm_P0.65mm, symbol 74xx:74LS258
Connections:
- net labels added: ALU_CARRY_IN, ALU_FUNC_0, ALU_FUNC_1, ALU_FUNC_2, ALU_FUNC_3, ALU_MODE, CARRY_FLAG, EEPROM_0, EEPROM_1, EEPROM_2, EEPROM_3, GND, SHA_SEL_00, SHA_SEL_01, VCC, ~ALU_FLAG_REG_IN, ~ALU_MODE_0_CARRY_IN_EN, ~ALU_MODE_0_EN, ~ALU_MODE_1_EN, ~CLEAR_INT_0, ~CLEAR_INT_1, ~CLEAR_INT_2, ~HALT, ~INC_PC, ~JUMP, ~JUMP_JA_JNBE, ~JUMP_JBE_JNA, ~JUMP_JB_JNAE_JC, ~JUMP_JE_JZ, ~JUMP_JGE_JNL, ~JUMP_JG_JNLE, ~JUMP_JLE_JNG, ~JUMP_JL_JNG, ~JUMP_JNB_JAE_JNC, ~JUMP_JNE_JNZ, ~JUMP_JNO, ~JUMP_JNS, ~JUMP_JO, ~JUMP_JS, ~LOAD_A_REGISTER, ~LOAD_B_REGISTER, ~LOAD_CODE_SEGMENT, ~LOAD_CONSTANT_REGISTER, ~LOAD_C_REGISTER, ~LOAD_DATA_SEGMENT, ~LOAD_D_REGISTER, ~LOAD_E_REGISTER, ~LOAD_F_REGISTER, ~LOAD_INSTRUCTION_REGISTER, ~LOAD_MAR, ~LOAD_OUTPUT_1, ~LOAD_OUTPUT_2, ~LOAD_STACK_POINTER, ~LOAD_SYNTH_1, ~LOAD_SYNTH_2, ~LOAD_TX_LSB_REGISTER, ~LOAD_TX_MSB_REGISTER, ~RESET, ~SET_INTERRUPT_FREQ, ~SHIFT_A_LEFT, ~SHIFT_A_RIGHT, ~SP_DEC, ~SP_INC, ~TRANSMIT_UART, ~WRITE_MEMORY, ~WRITE_MUX0_EN, ~WRITE_MUX1_EN, ~WRITE_MUX2_EN
- wire segments 1 -> 63
- no-connect marks 0 -> 13
Other:
- note added: "01 - SHIFT RIGHT\n10 - SHIFT LEFT\n11 - LOAD A"
- note added: "ALU - LHS\nNoop / SHL / SHR / LOAD A"
- note added: "ALU\n"
- note added: "GROUP 1\nWRITE / LOAD / SET"
- note added: "If\n~SHIFT_A_RIGHT~ is LOW, AND\n~LOAD_A_REGISTER~ is LOW, then\nLoad A\nelse,\nNOOP\n\nIf ~LOAD_A_REGISTER~ is HIGH,\nthen this MUX outputs Tri-State"
- note added: "If\n~SHIFT_A_RIGHT~ or\n~SHIFT_A_LEFT~ is Active (LOW)\nthen this MUX is selected\n\nif both are HIGH, this MUX outputs\ntri-state (High impediance)"
- note added: "LDA"
- note added: "Logic Gate Power"
- note added: "NOOP"
- note added: "SHL"
- note added: "SHR"
- note added: "Unused Logic Gates"
- note added: "Used for ALU Mode"
- note removed: "GROUP 1"
- note removed: "GROUP 2"
