File: PCB-Modules/99_IN PROGRESS/ALU/ALU_Control_and_Output/Control_and_Output.kicad_pcb (KiCad board)
At the start: 4 copper layers, 39.6 x 26.9 mm, 7 parts, among them J3 Conn_01x08, J4 Conn_01x12, U1 74LS04, U11 74LS245, U12 74LS138, U2 74LS04, U3 74LS245

Commit message: Documentation and Cleanup
Parts:
- added C1: C, Capacitor_SMD:C_0805_2012Metric, F.Cu at (97.3, 98.6)
- added C2: C, Capacitor_SMD:C_0805_2012Metric, F.Cu at (119.9, 98.6)
- added C3: C, Capacitor_SMD:C_0805_2012Metric, F.Cu at (202.4, 99.6)
- added C4: C, Capacitor_SMD:C_0805_2012Metric, F.Cu at (168.3, 97.8)
- added C5: C_Polarized, Capacitor_SMD:CP_Elec_4x3, F.Cu at (209.6, 94.5)
- added J1: Conn_01x08, Connector_PinSocket_2.54mm:PinSocket_1x08_P2.54mm_Vertical, B.Cu at (96.4, 90.0)
- added J2: Conn_01x08, Connector_PinSocket_2.54mm:PinSocket_1x08_P2.54mm_Vertical, B.Cu at (120.1, 90.0)
- added J5: Conn_01x12, Connector_PinSocket_2.54mm:PinSocket_1x11_P2.54mm_Vertical, B.Cu at (197.7, 89.9)
- added J6: Conn_01x08, Connector_PinSocket_2.54mm:PinSocket_1x08_P2.54mm_Vertical, B.Cu at (96.3, 117.9)
- added U10: 74LS21, Package_SO:SOIC-14_3.9x8.7mm_P1.27mm, F.Cu at (209.8, 105.1)
- added U4: 74LS574, Package_SO:SO-20_5.3x12.6mm_P1.27mm, F.Cu at (125.3, 105.2)
- added U5: 74LS245, Package_SO:TSSOP-20_4.4x6.5mm_P0.65mm, F.Cu at (138.2, 101.1)
- added U6: 74HC640, Package_SO:SO-20_5.3x12.6mm_P1.27mm, F.Cu at (151.4, 105.2)
- added U7: 74LS00, Package_SO:TSSOP-14_4.4x5mm_P0.65mm, F.Cu at (199.8, 105.2)
- added U8: 74LS00, Package_SO:TSSOP-14_4.4x5mm_P0.65mm, F.Cu at (163.6, 105.2)
- added U9: 74LS08, Package_SO:TSSOP-14_4.4x5mm_P0.65mm, F.Cu at (190.8, 105.2)
- J3: value Conn_01x08 -> Conn_01x11; footprint Connector_PinHeader_2.54mm:PinHeader_1x08_P2.54mm_Vertical -> Connector_PinHeader_2.54mm:PinHeader_1x11_P2.54mm_Vertical
- J4: value Conn_01x12 -> Conn_01x08; footprint Connector_PinHeader_2.54mm:PinHeader_1x12_P2.54mm_Vertical -> Connector_PinSocket_2.54mm:PinSocket_1x08_P2.54mm_Vertical
- U1: value 74LS04 -> 74LS08
- U11: footprint Package_SO:TSSOP-20_4.4x5mm_P0.5mm -> Package_SO:TSSOP-20_4.4x6.5mm_P0.65mm
- U12: value 74LS138 -> 74LS04; footprint Package_SO:TSSOP-16_4.4x5mm_P0.65mm -> Package_SO:TSSOP-14_4.4x5mm_P0.65mm
- U2: value 74LS04 -> 74LS574; footprint Package_SO:TSSOP-14_4.4x5mm_P0.65mm -> Package_SO:SO-20_5.3x12.6mm_P1.27mm
- U3: value 74LS245 -> 74LS154; footprint Package_SO:TSSOP-20_4.4x5mm_P0.5mm -> Package_SO:SOIC-24W_7.5x15.4mm_P1.27mm
- moved U3 109.8 mm to (177.1, 105.2)
- moved J3 106.6 mm to (164.1, 117.8)
- moved J4 97.5 mm to (145.9, 90.0)
- moved U12 70.4 mm to (113.5, 108.0)
- moved U11 66.2 mm to (138.2, 110.0)
- moved U1 54.1 mm to (113.5, 99.3)
- moved U2 52.6 mm to (102.1, 105.2)
Connections:
- J3 pad 1: Q0 -> ~{SHIFTER_SHL}
- J3 pad 2: Q1 -> ADC_SBB
- J3 pad 3: Q2 -> ~{AND}
- J3 pad 4: Q3 -> ~{OR}
- J3 pad 5: Q4 -> ~{XOR}
- J3 pad 6: Q5 -> ADDER_OUT
- J3 pad 7: Q6 -> ~{SHIFTER_SHR}
- J3 pad 8: Q7 -> ~{SHIFTER_ARI}
- J4 pad 1: ~MUX_ROTATE_OUT -> BUS0
- J4 pad 2: ~MUX_SHIFT_OUT -> BUS1
- J4 pad 3: ~MUX_XOR -> BUS2
- J4 pad 4: ~MUX_OR -> BUS3
- J4 pad 5: ~MUX_AND -> BUS4
- J4 pad 6: EEPROM_0 -> BUS5
- J4 pad 7: EEPROM_1 -> BUS6
- J4 pad 8: EEPROM_2 -> BUS7
- U1 pad 1: Q0 -> Net-(U1-Pad1)
- U1 pad 10: Net-(U1-Pad10) -> /~{ASL}
- U1 pad 11: Q4 -> ~{SHIFTER_SHL}
- U1 pad 13: Q5 -> /~{ROL}
- U1 pad 2: Net-(U1-Pad2) -> CLOCK
- U1 pad 3: Q1 -> Net-(U1-Pad3)
- U1 pad 4: Net-(U1-Pad4) -> Net-(U12-Pad8)
- U1 pad 5: Q2 -> CLOCK
- U1 pad 8: Net-(U1-Pad8) -> Net-(U1-Pad12)
- U1 pad 9: Q3 -> /~{SHL}
- U11 pad 11: OUT7 -> Q7
- U11 pad 12: OUT6 -> Q6
- U11 pad 13: OUT5 -> Q5
- U11 pad 14: OUT4 -> Q4
- U11 pad 15: OUT3 -> Q3
- U11 pad 16: OUT2 -> Q2
- U11 pad 17: OUT1 -> Q1
- U11 pad 18: OUT0 -> Q0
- U11 pad 19: Net-(U11-Pad19) -> ~{A}
- U11 pad 2: Q0 -> A0
- U11 pad 3: Q1 -> A1
- U11 pad 4: Q2 -> A2
- U11 pad 5: Q3 -> A3
- U11 pad 6: Q4 -> A4
- U11 pad 7: Q5 -> A5
- U11 pad 8: Q6 -> A6
- U11 pad 9: Q7 -> A7
- U12 pad 1: EEPROM_0 -> GND
- U12 pad 10: Net-(U12-Pad10) -> Net-(U1-Pad1)
- U12 pad 11: ~MUX_ROTATE_OUT -> ~{LATCH_ACCUMULATOR}
- U12 pad 12: ~MUX_SHIFT_OUT -> unconnected-(U12-Pad12)
- U12 pad 13: ~MUX_XOR -> GND
- U12 pad 14: ~MUX_OR -> VCC
- U12 pad 2: EEPROM_1 -> unconnected-(U12-Pad2)
- U12 pad 3: EEPROM_2 -> GND
- U12 pad 4: GND -> unconnected-(U12-Pad4)
- U12 pad 5: VCC -> GND
- U12 pad 6: EEPROM_7 -> unconnected-(U12-Pad6)
- U12 pad 7: Net-(U12-Pad7) -> GND
- U12 pad 8: GND -> Net-(U12-Pad8)
- U12 pad 9: Net-(U12-Pad9) -> ~{LATCH_B}
- U2 pad 1: Q6 -> GND
- U2 pad 10: Net-(U2-Pad10) -> GND
- U2 pad 11: VCC -> Net-(U1-Pad3)
- U2 pad 12: Net-(U2-Pad12) -> A7
- U2 pad 13: VCC -> A6
- U2 pad 14: VCC -> A5
- U2 pad 2: Net-(U2-Pad2) -> BUS0
- U2 pad 3: Q7 -> BUS1
- U2 pad 4: Net-(U2-Pad4) -> BUS2
- U2 pad 5: EEPROM_6 -> BUS3
- U2 pad 6: Net-(U11-Pad19) -> BUS4
- U2 pad 7: GND -> BUS5
- U2 pad 8: Net-(U2-Pad8) -> BUS6
- U2 pad 9: VCC -> BUS7
- U3 pad 1: VCC -> ~{A}
- U3 pad 10: GND -> ~{XOR}
- U3 pad 11: OUT7 -> /~{SHL}
- U3 pad 12: OUT6 -> GND
- U3 pad 13: OUT5 -> /~{SHR}
- U3 pad 14: OUT4 -> /~{ASL}
- U3 pad 15: OUT3 -> /~{ASR}
- U3 pad 16: OUT2 -> /~{ROR}
- U3 pad 17: OUT1 -> /~{ROL}
- U3 pad 18: OUT0 -> ~{ENABLE}
- U3 pad 19: EEPROM_6 -> ~{ENABLE}
- U3 pad 2: Net-(U1-Pad2) -> /~{ADD}
- U3 pad 20: VCC -> ALU_FUNC_3
- U3 pad 3: Net-(U1-Pad4) -> /~{ADC}
- U3 pad 4: Net-(U1-Pad6) -> /~{SUB}
- U3 pad 5: Net-(U1-Pad8) -> /~{SBB}
- U3 pad 6: Net-(U1-Pad10) -> /~{INC}
- U3 pad 7: Net-(U1-Pad12) -> /~{DEC}
- U3 pad 8: Net-(U2-Pad2) -> ~{AND}
- U3 pad 9: Net-(U2-Pad4) -> ~{OR}
Routing:
- net VCC: track 28.5 -> 193.2 mm, vias 8 -> 11
- net /~{ASL}: track 0.00 -> 131.4 mm, vias 0 -> 4
- net GND: track 13.7 -> 132.2 mm, vias 6 -> 22
- net /~{SHL}: track 0.00 -> 117.3 mm, vias 0 -> 2
- net /~{ROL}: track 0.00 -> 105.9 mm, vias 0 -> 4
- net BUS7: track 0.00 -> 94.9 mm, vias 0 -> 3
- net BUS6: track 0.00 -> 93.9 mm, vias 0 -> 3
- net BUS5: track 0.00 -> 92.2 mm, vias 0 -> 3
- net ~{SHIFTER_SHL}: track 0.00 -> 91.1 mm, vias 0 -> 1
- net BUS3: track 0.00 -> 90.2 mm, vias 0 -> 3
- net BUS4: track 0.00 -> 89.3 mm, vias 0 -> 3
- net BUS2: track 0.00 -> 87.8 mm, vias 0 -> 3
- net /~{SBB}: track 0.00 -> 85.7 mm, vias 0 -> 4
- net BUS1: track 0.00 -> 85.6 mm, vias 0 -> 3
- net BUS0: track 0.00 -> 84.1 mm, vias 0 -> 3
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- added copper zone on B.Cu, net GND
- added copper zone on F.Cu, net VCC
- removed copper zone on In2.Cu, net GND
- removed copper zone on In1.Cu, net VCC
Other:
- board size 39.6 x 26.9 mm -> 126.9 x 32.7 mm
- copper layers 4 -> 2
- net class Default removed
- board text added: "A0"
- board text added: "A1"
- board text added: "A2"
- board text added: "A3"
- board text added: "A4"
- board text added: "A5"
- board text added: "A6"
- board text added: "A7"
- board text added: "ALU Controller"
- board text added: "AdcSbb"
- board text added: "B0"
- board text added: "B1"
- board text added: "B2"
- board text added: "B3"
- board text added: "B4"
- board text added: "B5"
- board text added: "B6"
- board text added: "B7"
- board text added: "BUS0"
- board text added: "BUS1"
- board text added: "BUS2"
- board text added: "BUS3"
- board text added: "BUS4"
- board text added: "BUS5"
- board text added: "BUS6"
- board text added: "BUS7"
- board text added: "CLK"
- board text added: "FUNC0"
- board text added: "FUNC1"
- board text added: "FUNC2"
- board text added: "FUNC3"
- board text added: "FUNC4"
- board text added: "FUNC5"
- board text added: "JLCJLCJLCJLC"
- board text added: "OpMuxSel"
- board text added: "~{2'S}"
- board text added: "~{ACC IN}"
- board text added: "~{AND}"
- board text added: "~{ARI}"
- board text added: "~{Adder}"
- board text added: "~{B IN}"
- board text added: "~{OR}"
- board text added: "~{ROT}"
- board text added: "~{SHL}"
- board text added: "~{SHR}"
- board text added: "~{XOR}"
- board text removed: "Control Unit & Output"
- board text removed: "E0"
- board text removed: "E1"
- board text removed: "E2"
- board text removed: "E6"
- board text removed: "E7"
- board text removed: "~AND"
- board text removed: "~OR"
- board text removed: "~ROT"
- board text removed: "~SH"
- board text removed: "~XOR"
