File: PCB-Modules/99_IN PROGRESS/ALU/Arithmetic/Arithmetic.kicad_pcb (KiCad board)
At the start: 4 copper layers, 56.6 x 39.4 mm, 18 parts, among them J1 Conn_01x08, J2 Conn_01x08, J3 Conn_01x08, J4 Conn_01x08, U1 74LS157, U2 74LS157, U3 74LS86, U32 74LS04, U33 74LS08, U34 74LS32, U4 74LS86, U5 74LS283, U6 74LS283, U7 74LS245

Commit message: Documentation and Cleanup
Connections:
- net ~ADDER_OUT renamed ~{ADDER_OUT}
Other:
- net class Default removed
- board text added: "~{OE}"
- board text removed: "~OE"
