File: PCB-Modules/99_IN PROGRESS/memory/RAM-MODULE.kicad_pcb (KiCad board)
At the start: 4 copper layers, 79.2 x 75.7 mm, 56 parts, among them J1 Conn_01x09, J2 Conn_01x08, J3 Conn_01x16, U1 IS61C5128AL-10KLI, U2 IS61C5128AL-10KLI, U3 74LS173, U4 74LS173, U5 74LS157, U6 74LS32, U7 74LS04, U8 74LS32, U9 28C256

Commit message: Documentation and Cleanup
Parts:
- removed D10, D11, D12, D13, D14, D15, D16, D17: LED, LED_SMD:LED_0805_2012Metric
- removed R21, R22, R23: R_US, Resistor_SMD:R_0805_2012Metric
- added BT1: Battery_Cell, Battery:BatteryHolder_Keystone_106_1x20mm, F.Cu at (139.1, 74.1)
- added C5: C_Polarized, Capacitor_SMD:CP_Elec_4x3, F.Cu at (167.3, 127.2)
- added SW1: SW_DPDT_x2, Connector_PinHeader_2.54mm:PinHeader_1x03_P2.54mm_Vertical, F.Cu at (168.5, 51.9)
- added U10: 74LS245, Package_SO:TSSOP-20_4.4x6.5mm_P0.65mm, F.Cu at (145.7, 118.3)
- added U11: 74LS245, Package_SO:TSSOP-20_4.4x6.5mm_P0.65mm, F.Cu at (145.7, 107.5)
- added U12: 74LS173, Package_SO:TSSOP-16_4.4x5mm_P0.65mm, F.Cu at (168.9, 118.3)
- added U13: 74LS245, Package_SO:TSSOP-20_4.4x6.5mm_P0.65mm, F.Cu at (161.6, 118.3)
- added U14: 74LS245, Package_SO:TSSOP-20_4.4x6.5mm_P0.65mm, F.Cu at (161.6, 107.5)
- added U15: 74LS32, Package_SO:TSSOP-14_4.4x5mm_P0.65mm, F.Cu at (140.7, 95.9)
- added U16: 74LS04, Package_SO:TSSOP-14_4.4x5mm_P0.65mm, F.Cu at (155.3, 95.9)
- added U17: 74LS32, Package_SO:TSSOP-14_4.4x5mm_P0.65mm, F.Cu at (148.0, 95.9)
- added U18: ICL7673, Package_DIP:DIP-8_W7.62mm, F.Cu at (150.5, 54.7)
- D1, D2: value LED -> BAT54; footprint LED_SMD:LED_0805_2012Metric -> Diode_SMD:D_SOD-323F
- J1: value Conn_01x09 -> Conn_01x16; footprint Connector_PinHeader_2.54mm:PinHeader_1x09_P2.54mm_Vertical -> Connector_PinHeader_2.54mm:PinHeader_1x16_P2.54mm_Vertical
- U1: value IS61C5128AL-10KLI -> 28C256; footprint Package_SO:SOJ-36_10.16x23.49mm_P1.27mm -> Socket:DIP_Socket-28_W11.9_W12.7_W15.24_W17.78_W18.5_3M_228-1277-00-0602J
- U2: value IS61C5128AL-10KLI -> 74LS574; footprint Package_SO:SOJ-36_10.16x23.49mm_P1.27mm -> Package_SO:SOIC-20W_7.5x12.8mm_P1.27mm
- U3: value 74LS173 -> IS61C5128AL-10KLI; footprint Package_SO:TSSOP-16_4.4x5mm_P0.65mm -> Package_SO:SOJ-36_10.16x23.49mm_P1.27mm
- U4: value 74LS173 -> 74LS574; footprint Package_SO:TSSOP-16_4.4x5mm_P0.65mm -> Package_SO:SOIC-20W_7.5x12.8mm_P1.27mm
- U5: value 74LS157 -> IS61C5128AL-10KLI; footprint Package_SO:TSSOP-16_4.4x5mm_P0.65mm -> Package_SO:SOJ-36_10.16x23.49mm_P1.27mm
- U6: value 74LS32 -> 74LS173; footprint Package_SO:TSSOP-14_4.4x5mm_P0.65mm -> Package_SO:TSSOP-16_4.4x5mm_P0.65mm
- U7: value 74LS04 -> 74LS245; footprint Package_SO:TSSOP-14_4.4x5mm_P0.65mm -> Package_SO:TSSOP-20_4.4x6.5mm_P0.65mm
- U8: value 74LS32 -> 74LS245; footprint Package_SO:TSSOP-14_4.4x5mm_P0.65mm -> Package_SO:TSSOP-20_4.4x6.5mm_P0.65mm
- U9: value 28C256 -> 74LS173; footprint Package_DIP:DIP-28_W15.24mm_Socket -> Package_SO:TSSOP-16_4.4x5mm_P0.65mm
- moved C1 152.6 mm to (146.0, 50.9), turned to -90 degrees
- moved R10 149.0 mm to (150.6, 132.7), turned to -90 degrees
- moved U9 148.3 mm to (153.0, 118.3)
- moved U6 142.9 mm to (137.3, 118.3)
- moved J2 135.6 mm to (105.8, 45.4)
- moved U7 132.3 mm to (128.7, 118.3)
- moved U8 131.8 mm to (128.7, 107.5)
- moved J3 130.0 mm to (168.4, 136.5)
- moved C2 128.2 mm to (155.9, 104.7)
- moved R1 127.5 mm to (162.2, 50.9)
- moved R18 122.0 mm to (123.4, 126.1)
- moved D9 119.8 mm to (132.8, 70.6), turned to 90 degrees
- moved R9 114.0 mm to (148.1, 132.7)
- moved R17 112.7 mm to (93.3, 85.8), turned to -90 degrees
- moved R13 112.0 mm to (158.3, 132.7), turned to -90 degrees
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Connections:
- D1 pad 1: Net-(D1-Pad1) -> ~{ENABLE_RAM_LOW}
- D1 pad 2: /IO0 -> /BATTERY_ACTIVE
- D2 pad 1: Net-(D2-Pad1) -> ~{ENABLE_RAM_HIGH}
- D2 pad 2: /IO1 -> /BATTERY_ACTIVE
- D3 pad 2: /IO2 -> SEG0
- D4 pad 2: /IO3 -> SEG1
- D5 pad 2: /IO4 -> SEG2
- D6 pad 2: /IO5 -> SEG3
- D7 pad 2: /IO6 -> ~{ENABLE_RAM_HIGH}
- D8 pad 2: /IO7 -> ~{ENABLE_RAM_LOW}
- D9 pad 2: MODE -> ~{ENABLE_ROM}
- J1 pad 1: +5V -> ADDR_BUS15
- J1 pad 2: GND -> ADDR_BUS14
- J1 pad 3: ~{WE} -> ADDR_BUS13
- J1 pad 4: ~{OE} -> ADDR_BUS12
- J1 pad 5: ~{CS_IN} -> ADDR_BUS11
- J1 pad 6: ~{DS_IN} -> ADDR_BUS10
- J1 pad 7: CLOCK -> ADDR_BUS9
- J1 pad 8: MODE -> ADDR_BUS8
- J1 pad 9: MR -> ADDR_BUS7
- J2 pad 1: /IO7 -> BUS7
- J2 pad 2: /IO6 -> BUS6
- J2 pad 3: /IO5 -> BUS5
- J2 pad 4: /IO4 -> BUS4
- J2 pad 5: /IO3 -> BUS3
- J2 pad 6: /IO2 -> BUS2
- J2 pad 7: /IO1 -> BUS1
- J2 pad 8: /IO0 -> BUS0
- J3 pad 1: /A0 -> +5V
- J3 pad 10: /A9 -> ~{CODE_SEGMENT_OUT}
- J3 pad 11: /A10 -> ~{STACK_SEGMENT_OUT}
- J3 pad 12: /A11 -> ~{USE_DATA_SEGMENT}
- J3 pad 13: /A12 -> ~{USE_CODE_SEGMENT}
- J3 pad 14: /A13 -> ~{USE_STACK_SEGMENT}
- J3 pad 15: /A14 -> ~{READ}
- J3 pad 16: /A15 -> ~{WRITE}
- J3 pad 2: /A1 -> GND
- J3 pad 3: /A2 -> RESET
- J3 pad 4: /A3 -> CLOCK
- J3 pad 5: /A4 -> ~{LATCH_MAR}
- J3 pad 6: /A5 -> ~{LATCH_DATA_SEGMENT}
- J3 pad 7: /A6 -> ~{LATCH_CODE_SEGMENT}
- J3 pad 8: /A7 -> ~{LATCH_STACK_SEGMENT}
- J3 pad 9: /A8 -> ~{DATA_SEGMENT_OUT}
- R1 pad 1: Net-(D1-Pad1) -> /BATTERY_ACTIVE
- R1 pad 2: GND -> VCC
- R10 pad 1: MR -> +5V
- R10 pad 2: GND -> ~{LATCH_STACK_SEGMENT}
- R11 pad 1: Net-(D11-Pad1) -> +5V
- R11 pad 2: GND -> ~{LATCH_CODE_SEGMENT}
- R12 pad 1: Net-(D12-Pad1) -> +5V
- R12 pad 2: GND -> ~{LATCH_DATA_SEGMENT}
- R13 pad 1: Net-(D13-Pad1) -> +5V
- R13 pad 2: GND -> ~{LATCH_MAR}
- R14 pad 1: Net-(D14-Pad1) -> GND
- R14 pad 2: GND -> Net-(D3-Pad1)
- R15 pad 1: Net-(D15-Pad1) -> GND
- R15 pad 2: GND -> Net-(D4-Pad1)
- R16 pad 1: Net-(D16-Pad1) -> GND
- R16 pad 2: GND -> Net-(D5-Pad1)
- R17 pad 1: ~{DS_IN} -> GND
- R17 pad 2: +5V -> Net-(D6-Pad1)
- R18 pad 1: MODE -> GND
- R18 pad 2: GND -> Net-(D7-Pad1)
- R19 pad 1: Net-(D10-Pad1) -> GND
- R19 pad 2: GND -> Net-(D8-Pad1)
- R2 pad 1: Net-(D2-Pad1) -> +5V
- R2 pad 2: GND -> ~{WRITE}
- R20 pad 1: Net-(D17-Pad1) -> GND
- R20 pad 2: GND -> Net-(D9-Pad1)
- R3 pad 1: Net-(D3-Pad1) -> +5V
- R3 pad 2: GND -> ~{READ}
- R4 pad 1: Net-(D4-Pad1) -> +5V
- R4 pad 2: GND -> ~{USE_STACK_SEGMENT}
- R5 pad 1: Net-(D5-Pad1) -> +5V
- R5 pad 2: GND -> ~{USE_CODE_SEGMENT}
- R6 pad 1: Net-(D6-Pad1) -> +5V
- R6 pad 2: GND -> ~{USE_DATA_SEGMENT}
- R7 pad 1: Net-(D7-Pad1) -> +5V
- R7 pad 2: GND -> ~{STACK_SEGMENT_OUT}
- R8 pad 1: Net-(D8-Pad1) -> +5V
- R8 pad 2: GND -> ~{CODE_SEGMENT_OUT}
- R9 pad 1: Net-(D9-Pad1) -> +5V
- R9 pad 2: GND -> ~{DATA_SEGMENT_OUT}
- U1 pad 1: /A0 -> MAR14
- U1 pad 10: GND -> MAR0
- U1 pad 11: /IO2 -> BUS0
- U1 pad 12: /IO3 -> BUS1
- U1 pad 13: ~{WE} -> BUS2
- U1 pad 14: /A5 -> GND
- U1 pad 15: /A6 -> BUS3
- U1 pad 16: /A7 -> BUS4
- U1 pad 17: /A8 -> BUS5
- U1 pad 18: /A9 -> BUS6
- U1 pad 19: unconnected-(U1-Pad19) -> BUS7
- U1 pad 2: /A1 -> MAR12
- U1 pad 20: /A10 -> ~{ENABLE_ROM}
- U1 pad 21: /A11 -> MAR10
- U1 pad 22: /A12 -> ~{READ}
- U1 pad 23: /A13 -> MAR11
- U1 pad 24: /A14 -> MAR9
- U1 pad 25: /IO4 -> MAR8
- U1 pad 26: /IO5 -> MAR13
- U1 pad 28: GND -> +5V
- U1 pad 3: /A2 -> MAR7
- U1 pad 4: /A3 -> MAR6
- U1 pad 5: /A4 -> MAR5
- U1 pad 6: Net-(U1-Pad6) -> MAR4
- U1 pad 7: /IO0 -> MAR3
- U1 pad 8: /IO1 -> MAR2
- U1 pad 9: +5V -> MAR1
- U2 pad 1: /A0 -> GND
- U2 pad 11: /IO2 -> Net-(U16-Pad12)
- U2 pad 12: /IO3 -> MAR7
- U2 pad 13: ~{WE} -> MAR6
- U2 pad 14: /A5 -> MAR5
- U2 pad 15: /A6 -> MAR4
- U2 pad 16: /A7 -> MAR3
- U2 pad 17: /A8 -> MAR2
- U2 pad 18: /A9 -> MAR1
- U2 pad 19: unconnected-(U2-Pad19) -> MAR0
- U2 pad 2: /A1 -> ADDR_BUS0
- U2 pad 20: /A10 -> +5V
- U2 pad 3: /A2 -> ADDR_BUS1
- U2 pad 4: /A3 -> ADDR_BUS2
- U2 pad 5: /A4 -> ADDR_BUS3
- U2 pad 6: Net-(U2-Pad6) -> ADDR_BUS4
- U2 pad 7: /IO0 -> ADDR_BUS5
- U2 pad 8: /IO1 -> ADDR_BUS6
- U2 pad 9: +5V -> ADDR_BUS7
- U3 pad 1: GND -> MAR0
- U3 pad 10: ~{CS_IN} -> GND
- U3 pad 11: /IO3 -> BUS2
- U3 pad 12: /IO2 -> BUS3
- U3 pad 13: /IO1 -> ~{WRITE}
- U3 pad 14: /IO0 -> MAR5
- U3 pad 15: MR -> MAR6
- U3 pad 16: +5V -> MAR7
- U3 pad 2: GND -> MAR1
- U3 pad 3: /CS0 -> MAR2
- U3 pad 4: /CS1 -> MAR3
- U3 pad 5: /CS2 -> MAR4
- U3 pad 6: /CS3 -> ~{ENABLE_RAM_LOW}
- U3 pad 7: CLOCK -> BUS0
- U3 pad 8: GND -> BUS1
- U3 pad 9: ~{CS_IN} -> VCC
- U4 pad 10: ~{DS_IN} -> GND
- U4 pad 11: /IO3 -> Net-(U16-Pad12)
- U4 pad 12: /IO2 -> MAR15
- U4 pad 13: /IO1 -> MAR14
- U4 pad 14: /IO0 -> MAR13
- U4 pad 15: MR -> MAR12
- U4 pad 16: +5V -> MAR11
- U4 pad 2: GND -> ADDR_BUS8
- U4 pad 3: /DS0 -> ADDR_BUS9
- U4 pad 4: /DS1 -> ADDR_BUS10
- U4 pad 5: /DS2 -> ADDR_BUS11
- U4 pad 6: /DS3 -> ADDR_BUS12
- U4 pad 7: CLOCK -> ADDR_BUS13
- U4 pad 8: GND -> ADDR_BUS14
- U4 pad 9: ~{DS_IN} -> ADDR_BUS15
- U5 pad 1: MODE -> MAR0
- U5 pad 10: /DS2 -> GND
- U5 pad 11: /CS2 -> BUS2
- U5 pad 12: /~{RAM_CS} -> BUS3
- U5 pad 13: /DS3 -> ~{WRITE}
- U5 pad 14: /CS3 -> MAR5
- U5 pad 15: GND -> MAR6
- U5 pad 16: +5V -> MAR7
- U5 pad 2: /CS0 -> MAR1
- U5 pad 3: /DS0 -> MAR2
- U5 pad 4: /A16 -> MAR3
- U5 pad 5: /CS1 -> MAR4
- U5 pad 6: /DS1 -> ~{ENABLE_RAM_HIGH}
- U5 pad 7: /A17 -> BUS0
- U5 pad 8: GND -> BUS1
- U5 pad 9: /A18 -> VCC
- U6 pad 1: /A15 -> GND
- U6 pad 10: Net-(U6-Pad10) -> ~{LATCH_DATA_SEGMENT}
- U6 pad 11: /~{ROM_EN} -> BUS3
- U6 pad 12: /~{RAM_CS} -> BUS2
- U6 pad 13: Net-(U6-Pad13) -> BUS1
- U6 pad 14: +5V -> BUS0
- U6 pad 2: /A16 -> GND
- U6 pad 4: /A17 -> Net-(U6-Pad4)
- U6 pad 5: /A18 -> Net-(U6-Pad5)
- U6 pad 6: Net-(U6-Pad10) -> Net-(U6-Pad6)
- U6 pad 7: GND -> CLOCK
- U6 pad 8: Net-(U6-Pad13) -> GND
- U6 pad 9: Net-(U6-Pad3) -> ~{LATCH_DATA_SEGMENT}
- U7 pad 1: /~{RAM_CS} -> GND
- U7 pad 10: unconnected-(U7-Pad10) -> GND
- U7 pad 12: unconnected-(U7-Pad12) -> GND
- U7 pad 14: +5V -> GND
- U7 pad 2: Net-(U2-Pad6) -> Net-(U6-Pad3)
- U7 pad 3: GND -> Net-(U6-Pad4)
- U7 pad 4: unconnected-(U7-Pad4) -> Net-(U6-Pad5)
- U7 pad 5: GND -> Net-(U6-Pad6)
- U7 pad 7: GND -> unconnected-(U7-Pad7)
- U7 pad 8: Net-(U7-Pad8) -> unconnected-(U7-Pad8)
- U7 pad 9: /~{ROM_EN} -> unconnected-(U7-Pad9)
- U8 pad 1: /~{RAM_CS} -> GND
- U8 pad 11: unconnected-(U8-Pad11) -> GND
- U8 pad 14: +5V -> GND
- U8 pad 2: Net-(U7-Pad8) -> Net-(U6-Pad3)
- U8 pad 3: Net-(U1-Pad6) -> Net-(U6-Pad4)
- U8 pad 4: GND -> Net-(U6-Pad5)
- U8 pad 5: GND -> Net-(U6-Pad6)
- U8 pad 7: GND -> unconnected-(U8-Pad7)
- U8 pad 9: GND -> unconnected-(U8-Pad9)
- U9 pad 1: /A14 -> GND
- U9 pad 10: /A0 -> ~{LATCH_CODE_SEGMENT}
- U9 pad 11: /IO0 -> BUS3
- U9 pad 12: /IO1 -> BUS2
- U9 pad 13: /IO2 -> BUS1
- U9 pad 14: GND -> BUS0
- U9 pad 15: /IO3 -> RESET
- U9 pad 16: /IO4 -> +5V
- U9 pad 2: /A12 -> GND
- U9 pad 3: /A7 -> Net-(U10-Pad2)
- U9 pad 4: /A6 -> Net-(U10-Pad3)
- U9 pad 5: /A5 -> Net-(U10-Pad4)
- U9 pad 6: /A4 -> Net-(U10-Pad5)
- U9 pad 7: /A3 -> CLOCK
- U9 pad 8: /A2 -> GND
- U9 pad 9: /A1 -> ~{LATCH_CODE_SEGMENT}
Routing:
- net GND: track 79.4 -> 556.0 mm, vias 29 -> 23
- net +5V: track 36.4 -> 449.7 mm, vias 12 -> 26
- net BUS0: track 0.00 -> 237.1 mm, vias 0 -> 4
- net /IO0: track 233.2 -> 0.00 mm, vias 4 -> 0
- net BUS1: track 0.00 -> 227.1 mm, vias 0 -> 4
- net /IO1: track 221.6 -> 0.00 mm, vias 4 -> 0
- net BUS2: track 0.00 -> 213.0 mm, vias 0 -> 4
- net BUS3: track 0.00 -> 208.3 mm, vias 0 -> 5
- net /IO3: track 207.7 -> 0.00 mm, vias 4 -> 0
- net /IO2: track 207.3 -> 0.00 mm, vias 4 -> 0
- net /BATTERY_ACTIVE: track 0.00 -> 192.9 mm, vias 0 -> 1
- net SEG3: track 0.00 -> 170.0 mm, vias 0 -> 8
- net /IO7: track 153.6 -> 0.00 mm, vias 1 -> 0
- net /IO6: track 151.6 -> 0.00 mm, vias 3 -> 0
- net SEG1: track 0.00 -> 151.1 mm, vias 0 -> 5
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- added copper zone on F.Cu, net GND
- removed copper zone on In2.Cu, net +5V
- removed copper zone on In1.Cu, net GND
Other:
- board size 79.2 x 75.7 mm -> 99.8 x 100.3 mm
- board text added: "1M RAM | 32K ROM"
- board text added: "BUS0"
- board text added: "BUS1"
- board text added: "BUS2"
- board text added: "BUS3"
- board text added: "BUS4"
- board text added: "BUS5"
- board text added: "BUS6"
- board text added: "BUS7"
- board text added: "CLK"
- board text added: "EN"
- board text added: "Gnd"
- board text added: "ROM $0000 - $7FFF RAM $8000 - $FFFFF"
- board text added: "S0"
- board text added: "S1"
- board text added: "S2"
- board text added: "S3"
- board text added: "Vcc"
- board text added: "X"
- board text added: "~{CSO}"
- board text added: "~{DSO}"
- board text added: "~{LCS}"
- board text added: "~{LDS}"
- board text added: "~{LMAR}"
- board text added: "~{LSS}"
- board text added: "~{RAMH}"
- board text added: "~{RAML}"
- board text added: "~{RD}"
- board text added: "~{ROM}"
- board text added: "~{SSO}"
- board text added: "~{UCS}"
- board text added: "~{UDS}"
- board text added: "~{USS}"
- board text added: "~{WR}"
- board text removed: "$0000 - $7FFF ROM $8000 - $FFFFF RAM"
- board text removed: "+"
- board text removed: "-"
- board text removed: "992k RAM | 32K ROM"
- board text removed: "CODE"
- board text removed: "CP"
- board text removed: "DATA"
- board text removed: "DS"
- board text removed: "Data"
- board text removed: "IO0"
- board text removed: "IO1"
- board text removed: "IO2"
- board text removed: "IO3"
- board text removed: "IO4"
- board text removed: "IO5"
- board text removed: "IO6"
- board text removed: "IO7"
- board text removed: "MD"
- board text removed: "MEMORY SEGMENTS"
- board text removed: "RAM 480K"
- board text removed: "RAM 512K"
- board text removed: "ROM 32K"
- board text removed: "~{CS}"
- board text removed: "~{DS}"
- board text removed: "~{OE}"
- board text removed: "~{WE}"
