File: PCB-Modules/99_IN PROGRESS/memory/RAM-MODULE.kicad_sch (KiCad schematic)
At the start: 56 parts, among them J1 Conn_01x09, J2 Conn_01x08, J3 Conn_01x16, U1 IS61C5128AL-10KLI, U2 IS61C5128AL-10KLI, U3 74LS173, U4 74LS173, U5 74LS157, U6 74LS32, U7 74LS04, U8 74LS32, U9 28C256

Commit message: Documentation and Cleanup
Parts:
- removed D1, D10, D11, D12, D13, D14, D15, D16, D17, D2: LED, LED_SMD:LED_0805_2012Metric, symbol Device:LED
- removed J1: Conn_01x09, Connector_PinHeader_2.54mm:PinHeader_1x09_P2.54mm_Vertical, symbol Connector_Generic:Conn_01x09
- removed R21, R22, R23: R_US, Resistor_SMD:R_0805_2012Metric, symbol Device:R_US
- removed U1, U2: IS61C5128AL-10KLI, Package_SO:SOJ-36_10.16x23.49mm_P1.27mm, symbol Memory_RAM:IS61C5128AL-10KLI
- removed U3, U4: 74LS173, Package_SO:TSSOP-16_4.4x5mm_P0.65mm, symbol 74xx:74LS173
- removed U5: 74LS157, Package_SO:TSSOP-16_4.4x5mm_P0.65mm, symbol 74xx:74LS157
- removed U6, U8: 74LS32, Package_SO:TSSOP-14_4.4x5mm_P0.65mm, symbol 74xx:74LS32
- removed U7: 74LS04, Package_SO:TSSOP-14_4.4x5mm_P0.65mm, symbol 74xx:74LS04
- removed U9: 28C256, Package_DIP:DIP-28_W15.24mm_Socket, symbol Memory_EEPROM:28C256
- added BT1: Battery_Cell, Battery:BatteryHolder_Keystone_106_1x20mm, symbol Device:Battery_Cell
- added C5: C_Polarized, Capacitor_SMD:CP_Elec_4x3, symbol Device:C_Polarized
- added D1, D2: BAT54, Diode_SMD:D_SOD-323F, symbol Diode:BAT54J
- added J1: Conn_01x16, Connector_PinHeader_2.54mm:PinHeader_1x16_P2.54mm_Vertical, symbol Connector_Generic:Conn_01x16
- added SW1: SW_DPDT_x2, Connector_PinHeader_2.54mm:PinHeader_1x03_P2.54mm_Vertical, symbol Switch:SW_DPDT_x2
- added U1: 28C256, Socket:DIP_Socket-28_W11.9_W12.7_W15.24_W17.78_W18.5_3M_228-1277-00-0602J, symbol Memory_EEPROM:28C256
- added U15, U17: 74LS32, symbol 74xx:74LS32
- added U16: 74LS04, symbol 74xx:74LS04
- added U18: ICL7673, Package_DIP:DIP-8_W7.62mm, symbol Stephen:ICL7673
- added U2, U4: 74LS574, Package_SO:SOIC-20W_7.5x12.8mm_P1.27mm, symbol 74xx:74LS574
- added U3, U5: IS61C5128AL-10KLI, Package_SO:SOJ-36_10.16x23.49mm_P1.27mm, symbol Memory_RAM:IS61C5128AL-10KLI
- J3: Control (none) -> Control Lines; L Address Bus -> (none)
- R1: Field4 (none) -> 2K
Connections:
- net A0 is gone; now on net +5V: J3.1 (Pin_1)
- net A1 is gone; now on net GND: J3.2 (Pin_2)
- net A3 is gone; now on net CLOCK: J3.4 (Pin_4)
- net MR is gone; now on net +5V: R10.1
- net ~{DS_IN} is gone; now on net GND: R17.1
- net +5V: now also R11.1, R12.1, R13.1, R2.1, R3.1, R4.1, R5.1, R6.1, R7.1, R8.1, R9.1, C5.1, U1.27 (~{WE}), U1.28 (VCC), U15.14 (VCC), U16.14 (VCC), U17.14 (VCC), U18.8 (Vp), U2.20 (VCC), U4.20 (VCC); no longer R17.2
- net GND: now also R14.1, R15.1, R16.1, R18.1, R19.1, R20.1, BT1.2 (-), C5.2, U1.14 (GND), U15.7 (GND), U16.7 (GND), U17.1, U17.10, U17.2, U17.4, U17.5, U17.7 (GND), U17.9, U18.4 (Gnd), U2.1 (OE), U2.10 (GND), U3.10 (GND), U3.28 (GND), U4.1 (OE), U4.10 (GND), U5.10 (GND), U5.28 (GND); no longer R1.2, R10.2, R11.2, R12.2, R13.2, R14.2, R15.2, R16.2, R18.2, R19.2, R2.2, R20.2, R3.2, R4.2, R5.2, R6.2, R7.2, R8.2, R9.2
- net BATTERY_ACTIVE: now reaches R1.1
- net BATTERY_ACTIVE: now also D1.2 (A), D2.2 (A), U18.6 (PBar)
- net at D3.1 (K): now also R14.2; no longer R3.1
- net at D4.1 (K): now also R15.2; no longer R4.1
- net at D5.1 (K): now also R16.2; no longer R5.1
- net at D6.1 (K): now also R17.2; no longer R6.1
- net at D7.1 (K): now also R18.2; no longer R7.1
- net at D8.1 (K): now also R19.2; no longer R8.1
- net at D9.1 (K): now also R20.2; no longer R9.1
- net A10 renamed ~{STACK_SEGMENT_OUT}
- net ~{STACK_SEGMENT_OUT}: now also R7.2
- net A11 renamed ~{USE_DATA_SEGMENT}
- net ~{USE_DATA_SEGMENT}: now also R6.2, U16.11
- net A12 renamed ~{USE_CODE_SEGMENT}
- net ~{USE_CODE_SEGMENT}: now also R5.2, U16.5
- net A13 renamed ~{USE_STACK_SEGMENT}
- net ~{USE_STACK_SEGMENT}: now also R4.2, U16.9
- net A14 renamed ~{READ}
- net ~{READ}: now also R3.2, U1.22 (~{OE}), U3.31 (~{OE}), U5.31 (~{OE})
- net A15 renamed ~{WRITE}
- net ~{WRITE}: now also R2.2, U3.13 (~{WE}), U5.13 (~{WE})
- net A2 renamed RESET
- net A4 renamed ~{LATCH_MAR}
- net ~{LATCH_MAR}: now also R13.2, U16.13
- net A5 renamed ~{LATCH_DATA_SEGMENT}
- net ~{LATCH_DATA_SEGMENT}: now also R12.2
- net A6 renamed ~{LATCH_CODE_SEGMENT}
- net ~{LATCH_CODE_SEGMENT}: now also R11.2
- net A7 renamed ~{LATCH_STACK_SEGMENT}
- net ~{LATCH_STACK_SEGMENT}: now also R10.2
- net A8 renamed ~{DATA_SEGMENT_OUT}
- net ~{DATA_SEGMENT_OUT}: now also R9.2
- net A9 renamed ~{CODE_SEGMENT_OUT}
- net ~{CODE_SEGMENT_OUT}: now also R8.2
- net IO0 renamed BUS0
- net BUS0: now also U1.11 (D0), U3.7 (I/O0), U5.7 (I/O0)
- net IO1 renamed BUS1
- net BUS1: now also U1.12 (D1), U3.8 (I/O1), U5.8 (I/O1)
- net IO2 renamed BUS2
- net BUS2: now also U1.13 (D2), U3.11 (I/O2), U5.11 (I/O2); no longer D3.2 (A)
- net IO3 renamed BUS3
- net BUS3: now also U1.15 (D3), U3.12 (I/O3), U5.12 (I/O3); no longer D4.2 (A)
- net IO4 renamed BUS4
- net BUS4: now also U1.16 (D4), U3.25 (I/O4), U5.25 (I/O4); no longer D5.2 (A)
- net IO5 renamed BUS5
- net BUS5: now also U1.17 (D5), U3.26 (I/O5), U5.26 (I/O5); no longer D6.2 (A)
- net IO6 renamed BUS6
- net BUS6: now also U1.18 (D6), U3.29 (I/O6), U5.29 (I/O6); no longer D7.2 (A)
- net IO7 renamed BUS7
- net BUS7: now also U1.19 (D7), U3.30 (I/O7), U5.30 (I/O7); no longer D8.2 (A)
- net MODE renamed ~{ENABLE_ROM}
- net ~{ENABLE_ROM}: now also U1.20 (~{CS}), U15.11, U16.3; no longer R18.1
- new net: BT1.1 (+), SW1.1 (A)
- new net: SW1.2 (B), U18.2 (Vs)
- new net: U16.12, U2.11 (Cp), U4.11 (Cp)
- new net: U16.4, U17.12
- new net: U15.10, U15.6
- new net: U15.12, U15.8
- new net: U15.3, U15.9
- new net ADDR_BUS0: J1.16 (Pin_16), U2.2 (D0)
- new net ADDR_BUS1: J1.15 (Pin_15), U2.3 (D1)
- new net ADDR_BUS10: J1.6 (Pin_6), U4.4 (D2)
- new net ADDR_BUS11: J1.5 (Pin_5), U4.5 (D3)
- new net ADDR_BUS12: J1.4 (Pin_4), U4.6 (D4)
- new net ADDR_BUS13: J1.3 (Pin_3), U4.7 (D5)
- new net ADDR_BUS14: J1.2 (Pin_2), U4.8 (D6)
- new net ADDR_BUS15: J1.1 (Pin_1), U4.9 (D7)
- new net ADDR_BUS2: J1.14 (Pin_14), U2.4 (D2)
- new net ADDR_BUS3: J1.13 (Pin_13), U2.5 (D3)
- new net ADDR_BUS4: J1.12 (Pin_12), U2.6 (D4)
- new net ADDR_BUS5: J1.11 (Pin_11), U2.7 (D5)
- new net ADDR_BUS6: J1.10 (Pin_10), U2.8 (D6)
- new net ADDR_BUS7: J1.9 (Pin_9), U2.9 (D7)
- new net ADDR_BUS8: J1.8 (Pin_8), U4.2 (D0)
- new net ADDR_BUS9: J1.7 (Pin_7), U4.3 (D1)
- new net MAR0: U1.10 (A0), U2.19 (Q0), U3.1 (A0), U5.1 (A0)
- new net MAR1: U1.9 (A1), U2.18 (Q1), U3.2 (A1), U5.2 (A1)
- new net MAR10: U1.21 (A10), U3.20 (A10), U4.17 (Q2), U5.20 (A10)
- new net MAR11: U1.23 (A11), U3.21 (A11), U4.16 (Q3), U5.21 (A11)
- new net MAR12: U1.2 (A12), U3.22 (A12), U4.15 (Q4), U5.22 (A12)
- new net MAR13: U1.26 (A13), U3.23 (A13), U4.14 (Q5), U5.23 (A13)
- new net MAR14: U1.1 (A14), U3.24 (A14), U4.13 (Q6), U5.24 (A14)
- new net MAR15: U15.13, U3.32 (A15), U4.12 (Q7), U5.32 (A15)
- new net MAR2: U1.8 (A2), U2.17 (Q2), U3.3 (A2), U5.3 (A2)
- new net MAR3: U1.7 (A3), U2.16 (Q3), U3.4 (A3), U5.4 (A3)
- new net MAR4: U1.6 (A4), U2.15 (Q4), U3.5 (A4), U5.5 (A4)
- new net MAR5: U1.5 (A5), U2.14 (Q5), U3.14 (A5), U5.14 (A5)
- new net MAR6: U1.4 (A6), U2.13 (Q6), U3.15 (A6), U5.15 (A6)
- new net MAR7: U1.3 (A7), U2.12 (Q7), U3.16 (A7), U5.16 (A7)
- new net MAR8: U1.25 (A8), U3.17 (A8), U4.19 (Q0), U5.17 (A8)
- new net MAR9: U1.24 (A9), U3.18 (A9), U4.18 (Q1), U5.18 (A9)
- new net SEG0: D3.2 (A), U15.1, U3.33 (A16), U5.33 (A16)
- new net SEG1: D4.2 (A), U15.2, U3.34 (A17), U5.34 (A17)
- new net SEG2: D5.2 (A), U15.4, U3.35 (A18), U5.35 (A18)
- new net SEG3: D6.2 (A), U15.5, U16.1, U17.13
- new net USE_CODE_SEGMENT: U16.6
- new net USE_DATA_SEGMENT: U16.10
- new net USE_STACK_SEGMENT: U16.8
- new net VCC: R1.2, U18.1 (VO), U3.27 (VDD), U3.9 (VDD), U5.27 (VDD), U5.9 (VDD)
- new net ~{ENABLE_RAM_HIGH}: D2.1 (K), D7.2 (A), U16.2, U5.6 (~{CE})
- new net ~{ENABLE_RAM_LOW}: D1.1 (K), D8.2 (A), U17.11, U3.6 (~{CE})
- no-connect marks 7 -> 5
Other:
- added sheet CODE SEGMENT (segment.kicad_sch)
- added sheet DATA SEGMENT (segment.kicad_sch)
- added sheet STACK SEGMENT (segment.kicad_sch)
- note added: "32K ROM | 1M RAM"
- note added: "Backup Battery Power Switching"
- note added: "CONNECTIONS"
- note added: "HIGH"
- note added: "LED INDICATORS"
- note added: "LOW"
- note added: "Logic Gate Power and Unused"
- note added: "MEMORY ADDRESS REGISTER"
- note added: "MEMORY CHIP SELECT LOGIC"
- note added: "MEMORY MODULE"
- note added: "MEMORY SEGMENTS"
- note added: "Make active LOW"
- note added: "PULL UPS"
- note added: "RAM & ROM w/ battery backup power"
- note added: "ROM $0000 - $7FFF RAM $8000 - $FFFFF"
- note added: "Smoothing Cap's"
- note added: "To RAM"
- note removed: "$0000:$7fff"
- note removed: "$8000:$FFFFF"
- note removed: "- 10ns Access Time"
- note removed: "- 150ns READ Time - 100ns WRITE Time - CMOS and TTL Compatible Inputs and Outputs"
- note removed: "CMOS STATIC RAM IS61C5128AL-10KLI"
- note removed: "Code Segment Reg."
- note removed: "Code Segment This is default active. It stays active when the CPU is fetching the next instruction to be decoded."
- note removed: "Connections"
- note removed: "Data I/O LEDs"
- note removed: "Data Segment Reg."
- note removed: "Data Segment This is default inactive. It is active when the CPU is either reading or writing to memory. ie. MOV $1:f733, #55 ie. MOV a, $0:f733"
- note removed: "High"
- note removed: "If A[15..18] are all LOW, and ~{RAM_CS} is LOW, then Enable ROM is LOW which makes ROM active. Same, if any A[15..18] or ~{RAM_CS} is HIGH, then ROM is disabled"
- note removed: "Indicator LEDs"
- note removed: "Logic Power"
- note removed: "Low"
- note removed: "MUX When ~{MODE} line is set to: LOW (default) it will be using the values from Cs for the ~{CE} and A16..A18 lines HIGH (default) it will be using the values from Ds for the ~{CE} and A16..A18 lines"
- note removed: "Memory Module"
- note removed: "Parallel EEPROM AT28C256-15"
- note removed: "Provides 992K Of RAM and 32K Of ROM. Address space from $0:$7fff is reserved from ROM and $8000:$fffff is reserved for RAM. The code segment (CS) and the data segment(DS) registers should be initialized at the start of your program. Setting ~{DS_IN} or ~{CS_IN} low will latch the value presented on the data bus into the corresponding segment register. A HIGH signal on the WE line will write to RA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"
- note removed: "Pull U/D"
- note removed: "ROM Enable"
- note removed: "Segment MUX"
- note removed: "Smoothing Caps"
- note removed: "Unused Gates"
- company: (none) -> theWickedWebDev/8-bit-computer
