File: PCB-Modules/00_PROTOTYPING/prototype-board/prototype-board.kicad_sch (KiCad schematic)
At the start: 104 parts, among them J1 Conn_02x08_Male, J10 Conn_01x09_Male, J11 Conn_01x09_Male, J12 Conn_01x09_Male, J13 Conn_01x09_Male, J14 Conn_02x18_Odd_Even, J15 Conn_02x18_Odd_Even, J16 Screw_Terminal_02x08, J17 Screw_Terminal_02x08, J18 Screw_Terminal_01x02, J19 Conn_01x03_Male, J2 Conn_02x08_Male, J20 Conn_01x03_Male, J21 Conn_02x20_Odd_Even, J22 Conn_02x05_Odd_Even, J23 Conn_02x05_Odd_Even, J24 Conn_01x08_Male, J25 Conn_01x03_Male, J26 Conn_01x03_Male, J3 Conn_02x08_Male, J4 Conn_02x08_Male, J5 Conn_02x18_Odd_Even, J6 Conn_02x18_Odd_Even, J7 Barrel_Jack, J8 Conn_02x24_Odd_Even, J9 Conn_02x24_Odd_Even, SW1 SW_Push, SW2 SW_Push, U1 6X70X2_breadboard, U10 0603WAF1001T5E, U11 0603WAF1001T5E, U12 0603WAF1001T5E, U13 0603WAF1001T5E, U14 0603WAF1001T5E, U15 0603WAF1001T5E, U16 0603WAF1001T5E, U17 0603WAF1001T5E, U18 0603WAF1001T5E, U19 0603WAF1001T5E, U2 power-rail-breadboard, U20 0603WAF1001T5E, U21 0603WAF1001T5E, U22 0603WAF1001T5E, U23 0603WAF1001T5E, U24 0603WAF1001T5E, U25 0603WAF1001T5E, U26 0603WAF1001T5E, U27 0603WAF1001T5E, U28 0603WAF1001T5E, U29 0603WAF1001T5E, U3 power-rail-breadboard, U30 0603WAF1001T5E, U31 0603WAF1001T5E, U32 0603WAF1001T5E, U33 0603WAF1001T5E, U34 0603WAF1001T5E, U35 0603WAF1001T5E, U36 0603WAF1001T5E, U39 74LS245, U4 0603WAF1001T5E, U5 0603WAF1001T5E, U6 0603WAF1001T5E, U68 74LS245, U7 0603WAF1001T5E, U8 0603WAF1001T5E, U9 0603WAF1001T5E

Commit message: STUPID UPDATE MAJOR SAVE
Parts:
- J14, J15: footprint Connector_PinHeader_2.54mm:PinHeader_2x18_P2.54mm_Vertical -> Stephenv6:Breadboard_PinHeader_2x18
- J5, J6: footprint Connector_PinHeader_2.54mm:PinHeader_2x18_P2.54mm_Vertical -> Stephenv6:Breadboard_PinSocket_2x18
- J8, J9: footprint Connector_PinHeader_2.54mm:PinHeader_2x24_P2.54mm_Vertical -> Stephenv6:Breadboard_PinHeader_2x24
Connections:
- net GND: now also J9.3 (Pin_3), J9.4 (Pin_4); no longer J9.45 (Pin_45), J9.46 (Pin_46)
- net VCC: now also J9.1 (Pin_1), J9.2 (Pin_2); no longer J9.47 (Pin_47), J9.48 (Pin_48)
- new net: J9.45 (Pin_45), J9.46 (Pin_46)
- new net: J9.47 (Pin_47), J9.48 (Pin_48)
Changed lines of the file:
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@@
       (effects (font (size 1.27 1.27)) (justify right) hide)
     )
-    (property "Footprint" "Connector_PinHeader_2.54mm:PinHeader_2x18_P2.54mm_Vertical" (id 2) (at 168.91 165.1 0)
+    (property "Footprint" "Stephenv6:Breadboard_PinSocket_2x18" (id 2) (at 168.91 165.1 0)
       (effects (font (size 1.27 1.27)) hide)
     )
@@
     (pin "1")
   )
-  (symbol (lib_id "Connector_Generic:Conn_02x24_Odd_Even") (at 273.05 120.65 0) (unit 1)
-    (in_bom yes) (on_board yes)
-    (property "Reference" "J9" (id 0) (at 274.32 143.1798 90)
-      (effects (font (size 1.27 1.27)) (justify right) hide)
-    )
-    (property "Value" "Conn_02x24_Odd_Even" (id 1) (at 275.463 143.1798 90)
-      (effects (font (size 1.27 1.27)) (justify right) hide)
-    )
-    (property "Footprint" "Connector_PinHeader_2.54mm:PinHeader_2x24_P2.54mm_Vertical" (id 2) (at 273.05 120.65 0)
-      (effects (font (size 1.27 1.27)) hide)
-    )
-    (property "Datasheet" "~" (id 3) (at 273.05 120.65 0)
+  (symbol (lib_id "Connector_Generic:Conn_02x24_Odd_Even") (at 273.05 123.19 0) (mirror x) (unit 1)
+    (in_bom yes) (on_board yes)
+    (property "Reference" "J9" (id 0) (at 274.32 100.6602 90)
+      (effects (font (size 1.27 1.27)) (justify right) hide)
+    )
+    (property "Value" "Conn_02x24_Odd_Even" (id 1) (at 275.463 100.6602 90)
+      (effects (font (size 1.27 1.27)) (justify right) hide)
+    )
+    (property "Footprint" "Stephenv6:Breadboard_PinHeader_2x24" (id 2) (at 273.05 123.19 0)
+      (effects (font (size 1.27 1.27)) hide)
+    )
+    (property "Datasheet" "~" (id 3) (at 273.05 123.19 0)
       (effects (font (size 1.27 1.27)) hide)
     )
@@
       (effects (font (size 1.27 1.27)) (justify right) hide)
     )
-    (property "Footprint" "Connector_PinHeader_2.54mm:PinHeader_2x24_P2.54mm_Vertical" (id 2) (at 358.14 118.11 0)
+    (property "Footprint" "Stephenv6:Breadboard_PinHeader_2x24" (id 2) (at 358.14 118.11 0)
       (effects (font (size 1.27 1.27)) hide)
     )
@@
       (effects (font (size 1.27 1.27)) (justify right) hide)
     )
-    (property "Footprint" "Connector_PinHeader_2.54mm:PinHeader_2x18_P2.54mm_Vertical" (id 2) (at 168.91 189.23 0)
+    (property "Footprint" "Stephenv6:Breadboard_PinSocket_2x18" (id 2) (at 168.91 189.23 0)
       (effects (font (size 1.27 1.27)) hide)
     )
@@
       (effects (font (size 1.27 1.27)) (justify right) hide)
     )
-    (property "Footprint" "Connector_PinHeader_2.54mm:PinHeader_2x18_P2.54mm_Vertical" (id 2) (at 220.98 165.1 0)
+    (property "Footprint" "Stephenv6:Breadboard_PinHeader_2x18" (id 2) (at 220.98 165.1 0)
       (effects (font (size 1.27 1.27)) hide)
     )
@@
       (effects (font (size 1.27 1.27)) (justify right) hide)
     )
-    (property "Footprint" "Connector_PinHeader_2.54mm:PinHeader_2x18_P2.54mm_Vertical" (id 2) (at 220.98 189.23 0)
+    (property "Footprint" "Stephenv6:Breadboard_PinHeader_2x18" (id 2) (at 220.98 189.23 0)
       (effects (font (size 1.27 1.27)) hide)
     )
@@
     )
     (path "/00000000-0000-0000-0000-00006259d3b6"
-      (reference "J5") (unit 1) (value "Conn_02x18_Odd_Even") (footprint "Connector_PinHeader_2.54mm:PinHeader_2x18_P2.54mm_Vertical")
+      (reference "J5") (unit 1) (value "Conn_02x18_Odd_Even") (footprint "Stephenv6:Breadboard_PinSocket_2x18")
     )
     (path "/00000000-0000-0000-0000-000061c8980d"
-      (reference "J6") (unit 1) (value "Conn_02x18_Odd_Even") (footprint "Connector_PinHeader_2.54mm:PinHeader_2x18_P2.54mm_Vertical")
+      (reference "J6") (unit 1) (value "Conn_02x18_Odd_Even") (footprint "Stephenv6:Breadboard_PinSocket_2x18")
     )
     (path "/00000000-0000-0000-0000-000061cea066"
@@
     )
     (path "/00000000-0000-0000-0000-000061f118d8"
-      (reference "J8") (unit 1) (value "Conn_02x24_Odd_Even") (footprint "Connector_PinHeader_2.54mm:PinHeader_2x24_P2.54mm_Vertical")
+      (reference "J8") (unit 1) (value "Conn_02x24_Odd_Even") (footprint "Stephenv6:Breadboard_PinHeader_2x24")
     )
     (path "/00000000-0000-0000-0000-000061d452de"
-      (reference "J9") (unit 1) (value "Conn_02x24_Odd_Even") (footprint "Connector_PinHeader_2.54mm:PinHeader_2x24_P2.54mm_Vertical")
+      (reference "J9") (unit 1) (value "Conn_02x24_Odd_Even") (footprint "Stephenv6:Breadboard_PinHeader_2x24")
     )
     (path "/00000000-0000-0000-0000-00006229c8c0"
@@
     )
     (path "/00000000-0000-0000-0000-00006261769c"
-      (reference "J14") (unit 1) (value "Conn_02x18_Odd_Even") (footprint "Connector_PinHeader_2.54mm:PinHeader_2x18_P2.54mm_Vertical")
+      (reference "J14") (unit 1) (value "Conn_02x18_Odd_Even") (footprint "Stephenv6:Breadboard_PinHeader_2x18")
     )
     (path "/00000000-0000-0000-0000-0000626176ce"
-      (reference "J15") (unit 1) (value "Conn_02x18_Odd_Even") (footprint "Connector_PinHeader_2.54mm:PinHeader_2x18_P2.54mm_Vertical")
+      (reference "J15") (unit 1) (value "Conn_02x18_Odd_Even") (footprint "Stephenv6:Breadboard_PinHeader_2x18")
     )
     (path "/00000000-0000-0000-0000-000062866ed2"
