File: PCB-Modules/99_IN PROGRESS/IO/IO-Controller/cpu-input-output-control.kicad_sch (KiCad schematic)
At the start: 33 parts, among them J1 Conn_01x06, J11 Conn_01x08, J16 Conn_01x08, J2 Conn_01x23, J21 PCIE-036-02-X-D-RA, J3 Conn_02x20_Odd_Even, J4 Conn_01x02, J5 Conn_01x15, J6 Conn_01x16, J7 Conn_01x03, J8 Conn_01x03, SW1 SW_Push, SW2 SW_SPDT, U1 74LS08, U2 74LS04, U3 74LS154, U4 debounced-btn, U5 CD4060, U6 74LS173, U7 74LS251, U8 CD4060, Y1 Crystal_GND24

Commit message: saving
Parts:
- added J?: Conn_01x08, Connector_PinHeader_2.54mm:PinHeader_1x08_P2.54mm_Vertical, symbol Connector_Generic:Conn_01x08
- added J?: Conn_01x09, Connector_PinHeader_2.54mm:PinHeader_1x09_P2.54mm_Vertical, symbol Connector_Generic:Conn_01x09
- J1: value Conn_01x06 -> Conn_01x07; footprint Connector_PinHeader_2.54mm:PinHeader_1x06_P2.54mm_Vertical -> Connector_PinHeader_2.54mm:PinHeader_1x07_P2.54mm_Vertical; symbol Connector_Generic:Conn_01x06 -> Connector_Generic:Conn_01x07
- J2: value Conn_01x23 -> Conn_01x24; footprint Connector_PinHeader_2.54mm:PinHeader_1x23_P2.54mm_Vertical -> Connector_PinHeader_2.54mm:PinHeader_1x24_P2.54mm_Vertical; symbol Connector_Generic:Conn_01x23 -> Connector_Generic:Conn_01x24
Connections:
- net BUS0: now also J?.1 (Pin_1)
- net BUS1: now also J?.2 (Pin_2)
- net BUS2: now also J?.3 (Pin_3)
- net BUS3: now also J?.4 (Pin_4)
- net BUS4: now also J?.5 (Pin_5)
- net BUS5: now also J?.6 (Pin_6)
- net BUS6: now also J?.7 (Pin_7)
- net BUS7: now also J?.8 (Pin_8)
- net CLOCK: now also J1.6 (Pin_6); no longer J1.5 (Pin_5)
- net GND: now also J2.23 (Pin_23), J?.2 (Pin_2); no longer J2.22 (Pin_22)
- net VCC: now also J2.24 (Pin_24), J?.1 (Pin_1); no longer J2.23 (Pin_23)
- net ~{CLOCK}: now also J1.7 (Pin_7); no longer J1.6 (Pin_6)
- net ~{PORT10_EN}: now also J2.20 (Pin_20); no longer J2.19 (Pin_19)
- net ~{PORT2_EN}: now also J2.14 (Pin_14); no longer J21.B16
- net ~{PORT3_EN}: now also J2.15 (Pin_15); no longer J2.14 (Pin_14)
- net ~{PORT5_EN}: now also J2.16 (Pin_16); no longer J2.15 (Pin_15)
- net ~{PORT7_EN}: now also J2.17 (Pin_17); no longer J2.16 (Pin_16)
- net ~{PORT8_EN}: now also J2.18 (Pin_18); no longer J2.17 (Pin_17)
- net ~{PORT9_EN}: now also J2.19 (Pin_19); no longer J2.18 (Pin_18)
- net ~{READ}: now also J2.22 (Pin_22); no longer J2.21 (Pin_21)
- net ~{RESET}: now also J1.5 (Pin_5); no longer J1.4 (Pin_4)
- net ~{WRITE}: now also J2.21 (Pin_21); no longer J2.20 (Pin_20)
- new net CPU_CLOCK: J?.3 (Pin_3)
- new net ~{CLR_TIMER_INT_REQ_0}: J?.8 (Pin_8)
- new net ~{CLR_TIMER_INT_REQ_1}: J?.9 (Pin_9)
- new net ~{MEM_REQUEST}: J1.4 (Pin_4), J21.B16
- new net ~{SET_RELOAD_VALUE0}: J?.4 (Pin_4)
- new net ~{SET_RELOAD_VALUE1}: J?.5 (Pin_5)
- new net ~{TIMER_INT_REQ_0}: J?.6 (Pin_6)
- new net ~{TIMER_INT_REQ_1}: J?.7 (Pin_7)
Other:
- note added: "TIMERS CONN"
- note removed: "Should this cause an interrupt? Or should it be 100% hardware?"
- moved on the sheet: J21, SW1, U2B, U2C, U4, U5, U6, U7, U8
