File: PCB-Modules/99_IN PROGRESS/Latest-Full-Backplane/Latest-Full-Backplane.kicad_pcb (KiCad board)
At the start: 2 copper layers, 328.1 x 234.2 mm, 112 parts, among them J1 Conn_01x08, J10 Conn_01x13, J11 Conn_01x08, J12 Conn_01x04, J13 Conn_01x16, J14 Conn_01x08, J15 Conn_01x16, J16 Conn_01x11, J17 Conn_01x08, J18 Barrel_Jack_MountingPin, J19 Conn_01x07, J2 Conn_01x08, J20 Conn_01x12, J21 Conn_01x11, J22 Conn_01x08, J23 Conn_01x08, J24 Conn_01x08, J25 Conn_01x08, J26 Conn_01x09, J27 Conn_01x08, J28 Conn_01x16, J29 Conn_01x11, J3 Conn_01x13, J30 Conn_01x16, J31 Conn_01x16, J32 Conn_01x08, J33 Conn_01x11, J34 Conn_01x16, J35 Conn_01x16, J36 Conn_01x08, J37 Conn_01x09, J38 Conn_01x12, J39 Conn_01x08, J4 Conn_01x14, J40 Conn_01x11, J41 Conn_01x06, J42 Conn_01x12, J43 Conn_01x08, J44 Conn_01x10, J45 Conn_01x03, J46 Conn_01x03, J47 Conn_01x08, J48 Conn_01x07, J49 Conn_01x15, J5 Conn_01x08, J50 Conn_01x08, J51 Conn_01x16, J52 Conn_01x25, J53 Conn_01x06, J54 Conn_01x25, J55 Conn_01x02, J6 Conn_01x08, J7 Conn_01x08, J8 Conn_01x08, J9 Conn_01x16, SW1 SW_DPDT_x2

Commit message: saving
Parts:
- added J1: Conn_01x08, Connector_PinHeader_2.54mm:PinHeader_1x08_P2.54mm_Vertical, B.Cu at (490.2, 511.0)
- added J2: Conn_01x09, Connector_PinHeader_2.54mm:PinHeader_1x09_P2.54mm_Vertical, B.Cu at (529.6, 481.6)
- added REF**: trilobyte-logo-tiny, Stephenv6:trilobyte-logo-tiny, F.Cu at (490.2, 475.9)
- moved J27 371.0 mm to (8.78, 707.4)
- moved J28 371.0 mm to (-0.42, 707.4)
- moved J29 371.0 mm to (4.18, 707.4)
- moved J1 371.0 mm to (134.3, 694.5)
- moved J10 371.0 mm to (120.5, 694.5)
- moved J11 371.0 mm to (115.9, 732.1)
- moved J12 371.0 mm to (106.7, 737.2)
- moved J13 371.0 mm to (111.3, 694.5)
- moved J14 371.0 mm to (143.5, 694.5)
- moved J15 371.0 mm to (102.1, 694.5)
- moved J16 371.0 mm to (129.7, 694.5)
- moved J17 371.0 mm to (120.5, 729.6)
- moved J19 371.0 mm to (102.1, 737.2)
- moved J2 371.0 mm to (152.7, 694.5)
- moved J20 371.0 mm to (173.6, 694.5)
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- renumbered RN1 to RN'
Routing:
- net (no net): track 50.9 -> 0.00 mm
Other:
- board size 328.1 x 234.2 mm -> 353.3 x 375.7 mm
- board text added: "Timer Array"
- board text removed: "CPU"
- board text removed: "MEMORY"
- board text removed: "MR"
- board text removed: "TRILOBYTE"
