File: PCB-Modules/99_IN PROGRESS/READY-TO-PRINT/Minified-Gpr/Minified-Gpr.kicad_sch (KiCad schematic)
At the start: 33 parts, among them J1 Conn_01x08, J2 Conn_01x16, J3 Conn_01x11, U1 74LS574, U10 74LS245, U11 74LS245, U12 74LS574, U13 74LS574, U14 74LS574, U15 74LS245, U16 74LS245, U17 74LS245, U18 74LS245, U19 74LS138, U2 74LS138, U20 74LS00, U21 74LS00, U3 74LS138, U4 74LS574, U5 74LS574, U6 74LS574, U7 74LS574, U8 74LS245, U9 74LS245

Commit message: saving
Changed lines of the file:
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@@
   )
   (text "To just ASSERT or LOAD a value to the data \nbus to be used with external modules, just\nselect a single value from either READ or WRITE\n\nTo do a GPR to GPR transfer just select a \nREAD and WRITE control word and then OR \nthem together.\n\nTo do a RESET, ~{CONTROL7} is set LOW\nand all data buses are set to 0x0,\nwhich causes each register to load the \nvalue presented on their data bus."
-    (at 189.738 336.296 0)
+    (at 171.45 282.194 0)
     (effects (font (size 2 2)) (justify left bottom))
   )
-  (text "Control Word Truth Table" (at 188.976 295.91 0)
+  (text "Control Word Truth Table" (at 170.688 241.808 0)
     (effects (font (size 4 4)) (justify left bottom))
   )
