File: PCB-Modules/scratch-pad/Arithmetic.kicad_pcb (KiCad board)
At the start: 4 copper layers, 126.9 x 116.3 mm, 131 parts, among them J1 Conn_01x08, J1 Conn_01x13, J1 Conn_01x16, J2 Conn_01x08, J2 Conn_01x14, J3 Conn_01x07, J3 Conn_01x08, J3 Conn_01x11, J4 Conn_01x04, J4 Conn_01x08, J5 Conn_01x12, J6 Conn_01x08, U1 74LS04, U1 74LS08, U1 74LS157, U1 74LS173, U1 74LS245, U10 74LS21, U10 CD4072, U11 74LS245, U11 CD4072, U12 74LS04, U12 74LS32, U13 74LS154, U14 74LS08, U2 74LS02, U2 74LS04, U2 74LS08, U2 74LS157, U2 74LS245, U2 74LS574, U3 74LS08, U3 74LS154, U3 74LS32, U3 74LS86, U32 74LS04, U33 74LS08, U34 74LS32, U35 74LS32, U36 74LS02, U37 74LS08, U38 74LS157, U39 74LS86, U4 74LS04, U4 74LS08, U4 74LS32, U4 74LS574, U4 74LS86, U5 74LS02, U5 74LS245, U5 74LS283, U5 74LS32, U6 74HC640, U6 74LS08, U6 74LS245, U6 74LS283, U7 74LS00, U7 74LS245, U7 74LS32, U7 74LS86, U8 74LS00, U8 74LS86, U9 74LS02, U9 74LS08, U9 74LS245

Commit message: saving
Routing:
- net (no net): track 8024.2 -> 8022.3 mm
- net GND: track 440.5 -> 442.5 mm
Changed lines of the file:
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@@
   (segment (start 133.555 124.981069) (end 133.593901 124.942167) (width 0.2) (layer "F.Cu") (net 0))
   (segment (start 84.45 57.994) (end 84.45 56.488008) (width 0.25) (layer "F.Cu") (net 0))
-  (segment (start 43.572 146.9945) (end 43.572 145.0345) (width 0.25) (layer "F.Cu") (net 0))
   (segment (start 147.345006 117.74) (end 146.23 117.74) (width 0.2) (layer "F.Cu") (net 0))
   (segment (start 133.059989 61.042) (end 132.964 60.946011) (width 0.25) (layer "F.Cu") (net 0))
@@
   (segment (start 54.494 122.278) (end 54.494 122.024) (width 0.25) (layer "F.Cu") (net 26))
   (segment (start 113.515 97.9305) (end 113.515 95.961) (width 0.2) (layer "F.Cu") (net 26))
+  (segment (start 43.572 146.9945) (end 43.572 145.0345) (width 0.25) (layer "F.Cu") (net 26))
   (segment (start 130.03 136.815) (end 128.555 136.815) (width 0.2) (layer "F.Cu") (net 26))
   (segment (start 140.836 84.278) (end 137.656 84.278) (width 0.2) (layer "F.Cu") (net 26))
