File: PCBs/99_IN PROGRESS/FUTURE-WORK/ADC-Backplane/ADC-Backplane.kicad_sch (KiCad schematic)
At the start: 15 parts, among them J1 Conn_01x11, J10 Conn_01x03, J11 Conn_01x16, J12 Conn_01x08, J13 Screw_Terminal_01x02, J2 Conn_01x09, J3 Conn_01x03, J4 Conn_01x09, J5 Conn_01x03, J6 Conn_01x09, J7 Conn_01x03, J8 Conn_01x09, J9 Conn_01x03

Commit message: saving
Parts:
- added J1: Conn_01x02, Connector_PinHeader_2.54mm:PinHeader_1x02_P2.54mm_Horizontal, symbol Connector_Generic:Conn_01x02
- added J15: PCIE-Edge-Connect-036-02-X-D-RA_1, Connector_PCBEdge:BUS_PCIexpress_x1, symbol LIBRARY-8-bit-computer:PCIE-Edge-Connect-036-02-X-D-RA_1
- J5: renamed from J1; value Conn_01x11 -> Conn_01x12; footprint Connector_PinHeader_2.54mm:PinHeader_1x11_P2.54mm_Horizontal -> Connector_PinHeader_2.54mm:PinHeader_1x12_P2.54mm_Horizontal; symbol Connector_Generic:Conn_01x11 -> Connector_Generic:Conn_01x12
- renumbered J9 to J10, J10 to J11, J11 to J12, J12 to J13, J13 to J14, J5 to J6, J6 to J7, J7 to J8, J8 to J9
Connections:
- net +12V: now also J10.2 (Pin_2), J3.2 (Pin_2), J5.1 (Pin_1), J6.2 (Pin_2), J8.2 (Pin_2), J15.A1 (A01)
- net +5V: now also J10.3 (Pin_3), J11.3 (Pin_3), J3.3 (Pin_3), J5.2 (Pin_2), J6.3 (Pin_3), J8.3 (Pin_3), J15.B18; no longer J5.1 (Pin_1)
- net BUS0: now also J5.5 (Pin_5), J15.B1 (B01); no longer J5.4 (Pin_4)
- net BUS1: now also J5.6 (Pin_6), J15.B2 (B02); no longer J5.5 (Pin_5)
- net BUS2: now also J5.7 (Pin_7), J15.B3 (B03); no longer J5.6 (Pin_6)
- net BUS3: now also J5.8 (Pin_8), J15.B4 (B04); no longer J5.7 (Pin_7)
- net BUS4: now also J5.9 (Pin_9), J15.B5 (B05); no longer J5.8 (Pin_8)
- net BUS5: now also J5.10 (Pin_10), J15.B6 (B06); no longer J5.9 (Pin_9)
- net BUS6: now also J5.11 (Pin_11), J15.B7 (B07); no longer J5.10 (Pin_10)
- net BUS7: now also J5.12 (Pin_12), J15.B8 (B08); no longer J5.11 (Pin_11)
- net GND: now also J11.2 (Pin_2), J5.3 (Pin_3), J15.B17; no longer J5.2 (Pin_2)
- net ~{OE}: now also J11.1 (Pin_1), J5.4 (Pin_4), J15.A2 (A02); no longer J5.3 (Pin_3)
- net ~{EOx}: now reaches J2.2 (Pin_2)
- net ~{EOx}: now also J1.1 (Pin_1), J15.A3 (A03)
- net Vrefox: now reaches J2.6 (Pin_6)
- net Vrefox: now also J1.2 (Pin_2), J15.A4 (A04)
- no-connect marks 2 -> 22
