File: PCBs/99_IN PROGRESS/LEFT-TO-DO-MVP/SPR-DisplacementRegister/DisplacementRegister/powerful-register-2022.kicad_pcb (KiCad board)
At the start: 4 copper layers, 92.5 x 45 mm, 17 parts, among them J1 Conn_01x06, J2 Conn_01x16, J3 Conn_01x08, J4 Conn_01x16, J5 Conn_01x16, U1 74LS283, U2 74LS283, U3 74LS283, U4 74LS283, U5 74LS245, U6 74LS245, U7 74LS245, U8 74LS245

Commit message: saving
Parts:
- removed C3, C4: C, Capacitor_SMD:C_0805_2012Metric
- removed the J3 at (161.3, 91.2)
- removed U5, U6, U7, U8: 74LS245, Package_SO:SOIC-20W_7.5x12.8mm_P1.27mm
- added R1: R_Small_US, Resistor_SMD:R_0805_2012Metric, F.Cu at (149.4, 79.2)
- added R10: R_Small_US, Resistor_SMD:R_0805_2012Metric, F.Cu at (144.9, 76.3)
- added R11: R_Small_US, Resistor_SMD:R_0805_2012Metric, F.Cu at (149.4, 73.3)
- added R12: R_Small_US, Resistor_SMD:R_0805_2012Metric, F.Cu at (140.5, 76.3)
- added R13: R_Small_US, Resistor_SMD:R_0805_2012Metric, F.Cu at (149.4, 76.3)
- added R14: R_Small_US, Resistor_SMD:R_0805_2012Metric, F.Cu at (140.5, 79.2)
- added R15: R_Small_US, Resistor_SMD:R_0805_2012Metric, F.Cu at (136.1, 82.2)
- added R16: R_Small_US, Resistor_SMD:R_0805_2012Metric, F.Cu at (153.8, 76.3)
- added R17: R_Small_US, Resistor_SMD:R_0805_2012Metric, F.Cu at (140.5, 82.2)
- added R2: R_Small_US, Resistor_SMD:R_0805_2012Metric, F.Cu at (136.1, 79.2)
- added R3: R_Small_US, Resistor_SMD:R_0805_2012Metric, F.Cu at (144.9, 79.2)
- added R4: R_Small_US, Resistor_SMD:R_0805_2012Metric, F.Cu at (144.9, 82.2)
- added R5: R_Small_US, Resistor_SMD:R_0805_2012Metric, F.Cu at (136.1, 73.3)
- added R6: R_Small_US, Resistor_SMD:R_0805_2012Metric, F.Cu at (140.5, 73.3)
- added R7: R_Small_US, Resistor_SMD:R_0805_2012Metric, F.Cu at (136.1, 76.3)
- added R8: R_Small_US, Resistor_SMD:R_0805_2012Metric, F.Cu at (144.9, 73.3)
- added R9: R_Small_US, Resistor_SMD:R_0805_2012Metric, F.Cu at (153.8, 73.3)
- added REF**: trilobyte-logo-tiny, Stephenv6:trilobyte-logo-tiny, F.Cu at (163.1, 119.0)
- J1: footprint Connector_PinHeader_2.54mm:PinHeader_1x06_P2.54mm_Vertical -> Connector_PinHeader_2.54mm:PinHeader_1x04_P2.54mm_Vertical
- moved U4 46.7 mm to (152.4, 124.5)
- moved C2 44.1 mm to (146.7, 116.1), turned to 0 degrees
- moved C1 41.5 mm to (142.2, 116.1), turned to 0 degrees
- moved U1 30.0 mm to (101.3, 124.5)
- moved J1 19.3 mm to (169.4, 110.5)
- moved J4 19.3 mm to (97.5, 110.5)
- moved U2 18.8 mm to (135.4, 124.5)
- moved U3 9.88 mm to (118.4, 124.5)
- moved J2 6.35 mm to (135.6, 138.7)
- moved J3 6.35 mm to (144.0, 138.7)
- renumbered J4 to J3, J5 to J4
Connections:
- J1 pad 3: ~{DISP_MSB_OUT} -> CARRY_OUT
- J1 pad 4: ~{DISP_LSB_OUT} -> CARRY_IN
- J3 pad 1: ADDR15 -> Q15
- J3 pad 10: ADDR6 -> Q6
- J3 pad 11: ADDR5 -> Q5
- J3 pad 12: ADDR4 -> Q4
- J3 pad 13: ADDR3 -> Q3
- J3 pad 14: ADDR2 -> Q2
- J3 pad 15: ADDR1 -> Q1
- J3 pad 16: ADDR0 -> Q0
- J3 pad 2: ADDR14 -> Q14
- J3 pad 3: ADDR13 -> Q13
- J3 pad 4: ADDR12 -> Q12
- J3 pad 5: ADDR11 -> Q11
- J3 pad 6: ADDR10 -> Q10
- J3 pad 7: ADDR9 -> Q9
- J3 pad 8: ADDR8 -> Q8
- J3 pad 9: ADDR7 -> Q7
- U1 pad 1: /Q1 -> Q1
- U1 pad 10: /Q3 -> Q3
- U1 pad 13: /Q2 -> Q2
- U1 pad 4: /Q0 -> Q0
- U1 pad 7: GND -> CARRY_IN
- U2 pad 1: /Q9 -> Q9
- U2 pad 10: /Q11 -> Q11
- U2 pad 13: /Q10 -> Q10
- U2 pad 4: /Q8 -> Q8
- U3 pad 1: /Q5 -> Q5
- U3 pad 10: /Q7 -> Q7
- U3 pad 13: /Q6 -> Q6
- U3 pad 4: /Q4 -> Q4
- U4 pad 1: /Q13 -> Q13
- U4 pad 10: /Q15 -> Q15
- U4 pad 13: /Q14 -> Q14
- U4 pad 4: /Q12 -> Q12
Routing:
- net CARRY_OUT: track 96.0 -> 0.00 mm, vias 1 -> 0
- net /Q13: track 90.2 -> 0.00 mm, vias 4 -> 0
- net /Q12: track 89.4 -> 0.00 mm, vias 4 -> 0
- net /Q5: track 82.3 -> 0.00 mm, vias 4 -> 0
- net /Q6: track 81.9 -> 0.00 mm, vias 4 -> 0
- net /Q4: track 79.8 -> 0.00 mm, vias 4 -> 0
- net /Q14: track 78.0 -> 0.00 mm, vias 4 -> 0
- net /Q7: track 74.8 -> 0.00 mm, vias 2 -> 0
- net /Q15: track 73.3 -> 0.00 mm, vias 4 -> 0
- net /Q1: track 66.2 -> 0.00 mm, vias 4 -> 0
- net /Q9: track 65.9 -> 0.00 mm, vias 2 -> 0
- net /Q8: track 61.7 -> 0.00 mm, vias 2 -> 0
- net /Q0: track 60.4 -> 0.00 mm, vias 4 -> 0
- net /Q2: track 59.3 -> 0.00 mm, vias 4 -> 0
- net /Q10: track 58.8 -> 0.00 mm, vias 4 -> 0
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Other:
- board size 92.5 x 45 mm -> 92.5 x 32 mm
- board text added: "CI"
- board text removed: "~{LSBO}"
- board text removed: "~{MSBO}"
- board text removed: "~{OUT}"
