File: PCBs/99_IN PROGRESS/LEFT-TO-DO-MVP/SPR-DisplacementRegister/DisplacementRegister/powerful-register-2022.kicad_sch (KiCad schematic)
At the start: 17 parts, among them J1 Conn_01x06, J2 Conn_01x16, J3 Conn_01x08, J4 Conn_01x16, J5 Conn_01x16, U1 74LS283, U2 74LS283, U3 74LS283, U4 74LS283, U5 74LS245, U6 74LS245, U7 74LS245, U8 74LS245

Commit message: saving
Parts:
- removed C3, C4: C, Capacitor_SMD:C_0805_2012Metric, symbol Device:C
- removed J3: Conn_01x08, Connector_PinHeader_2.54mm:PinHeader_1x08_P2.54mm_Vertical, symbol Connector_Generic:Conn_01x08
- removed U5, U6, U7, U8: 74LS245, Package_SO:SOIC-20W_7.5x12.8mm_P1.27mm, symbol 74xx:74LS245
- added R1, R10, R11, R12, R13, R14, R15, R16, R17, R2, R3, R4, R5, R6, R7, R8, R9: R_Small_US, Resistor_SMD:R_0805_2012Metric, symbol Device:R_Small_US
- J1: footprint Connector_PinHeader_2.54mm:PinHeader_1x06_P2.54mm_Vertical -> Connector_PinHeader_2.54mm:PinHeader_1x04_P2.54mm_Vertical; symbol Connector_Generic:Conn_01x06 -> Connector_Generic:Conn_01x04
- J3: renamed from J4; Field5 Address Bus -> Result
- renumbered J5 to J4
Connections:
- net ADDR0 is gone; now on net Q0: J3.16 (Pin_16)
- net ADDR1 is gone; now on net Q1: J3.15 (Pin_15)
- net ADDR10 is gone; now on net Q10: J3.6 (Pin_6)
- net ADDR11 is gone; now on net Q11: J3.5 (Pin_5)
- net ADDR12 is gone; now on net Q12: J3.4 (Pin_4)
- net ADDR13 is gone; now on net Q13: J3.3 (Pin_3)
- net ADDR14 is gone; now on net Q14: J3.2 (Pin_2)
- net ADDR15 is gone; now on net Q15: J3.1 (Pin_1)
- net ADDR2 is gone; now on net Q2: J3.14 (Pin_14)
- net ADDR3 is gone; now on net Q3: J3.13 (Pin_13)
- net ADDR4 is gone; now on net Q4: J3.12 (Pin_12)
- net ADDR5 is gone; now on net Q5: J3.11 (Pin_11)
- net ADDR6 is gone; now on net Q6: J3.10 (Pin_10)
- net ADDR7 is gone; now on net Q7: J3.9 (Pin_9)
- net ADDR8 is gone; now on net Q8: J3.8 (Pin_8)
- net ADDR9 is gone; now on net Q9: J3.7 (Pin_7)
- net ~{DISP_MSB_OUT} is gone; now on net CARRY_OUT: J1.3 (Pin_3)
- net B0: now also R17.1
- net B1: now also R16.1
- net B10: now also R7.1
- net B11: now also R6.1
- net B12: now also R5.1
- net B13: now also R4.1
- net B14: now also R2.1
- net B15: now also R1.1
- net B2: now also R15.1
- net B3: now also R14.1
- net B4: now also R13.1
- net B5: now also R12.1
- net B6: now also R11.1
- net B7: now also R10.1
- net B8: now also R9.1
- net B9: now also R8.1
- net CARRY_OUT: no longer J1.6 (Pin_6)
- net GND: now also R1.2, R10.2, R11.2, R12.2, R13.2, R14.2, R15.2, R16.2, R17.2, R2.2, R3.2, R4.2, R5.2, R6.2, R7.2, R8.2, R9.2; no longer U1.7 (C0)
- removed net ~{DISPLACE_OUT}: J1.5 (Pin_5)
- net ~{DISP_LSB_OUT} renamed CARRY_IN
- net CARRY_IN: now also U1.7 (C0), R3.1
Other:
- note added: "BASE DATA"
- note added: "OFFSET DATA"
- note added: "RESULT"
