File: PCBs/03_MODULES/MEMORY-2022/memory.kicad_sch (KiCad schematic)
At the start: 20 parts, among them J1 Conn_01x07, J2 Conn_01x08, J3 Conn_01x16, J4 Conn_01x09, U1 74LS00, U2 4072, U3 74LS139

Commit message: cray cray save
Parts:
- added D34: LED, LED_SMD:LED_0805_2012Metric, symbol Device:LED
- added R35: R_Small_US, Resistor_SMD:R_0805_2012Metric, symbol Device:R_Small_US
- added U11: PLCC32_28_28C256, Stephenv6:PLCC-32-SOCKET-Microchip-32J-10_2001-B-IPC_A, symbol Stephen:PLCC32_28_28C256
- U1: value 74LS00 -> 74HC00
- U3: value 74LS139 -> 74HC139
Connections:
- net ADDR0: now also U11.11 (A0)
- net ADDR1: now also U11.10 (A1)
- net ADDR10: now also U11.24 (A10)
- net ADDR11: now also U11.27 (A11)
- net ADDR12: now also U11.3 (A12)
- net ADDR13: now also U11.30 (A13)
- net ADDR14: now also U11.2 (A14)
- net ADDR2: now also U11.9 (A2)
- net ADDR3: now also U11.8 (A3)
- net ADDR4: now also U11.7 (A4)
- net ADDR5: now also U11.6 (A5)
- net ADDR6: now also U11.5 (A6)
- net ADDR7: now also U11.4 (A7)
- net ADDR8: now also U11.29 (A8)
- net ADDR9: now also U11.28 (A9)
- net BUS0: now also U11.13 (I/O0)
- net BUS1: now also U11.14 (I/O1)
- net BUS2: now also U11.15 (I/O2)
- net BUS3: now also U11.18 (I/O3)
- net BUS4: now also U11.19 (I/O4)
- net BUS5: now also U11.20 (I/O5)
- net BUS6: now also U11.21 (I/O6)
- net BUS7: now also U11.22 (I/O7)
- net GND: now also R35.1, U11.16 (Gnd)
- net VCC: now also U11.31 (~{WE}), U11.32 (Vcc)
- net ~{EEPROM_EN}: now also D34.2 (A), U11.23 (~{CE})
- net ~{READ}: now also U11.25 (~{OE})
- new net: D34.1 (K), R35.2
Other:
- removed sheet EEPROM
