File: PCBs/03_MODULES/Minified-Gpr/Minified-Gpr.kicad_sch (KiCad schematic)
At the start: 33 parts, among them J1 Conn_01x08, J2 Conn_01x16, J3 Conn_01x11, U1 74LS574, U10 74LS245, U11 74LS245, U12 74LS574, U13 74LS574, U14 74LS574, U15 74LS245, U16 74LS245, U17 74LS245, U18 74LS245, U19 74LS138, U2 74LS138, U20 74LS00, U21 74LS00, U3 74LS138, U4 74LS574, U5 74LS574, U6 74LS574, U7 74LS574, U8 74LS245, U9 74LS245

Commit message: cray cray save
Parts:
- U1, U12, U13, U14, U4, U5, U6, U7: value 74LS574 -> 74HC574
- U10, U11, U15, U16, U17, U18, U8, U9: value 74LS245 -> 74HC245
- U19, U2, U3: value 74LS138 -> 74HC138
- U20, U21: value 74LS00 -> 74HC00
Other:
- note added: "CPU CONNECTIONS"
- note removed: "CONNECTIONS"
