File: PCBs/99_IN PROGRESS/LEFT-TO-DO-MVP/CPU-Control-Unit/CONTROL_UNIT.kicad_sch (KiCad schematic)
At the start: 24 parts, among them J1 Conn_01x08, J2 Conn_01x29, J3 Conn_01x24, J4 Conn_01x12, J5 Conn_01x07, J6 Conn_01x08, J7 Conn_01x07, J8 Conn_01x11, U1 PLCC32_28_28C256, U10 74LS08, U11 74LS08, U12 74LS139, U13 74LS154, U14 74LS08, U15 74HC245, U16 74HC245, U2 74HC245, U3 74HC245, U4 PLCC32_28_28C256, U5 74LS139, U6 74LS154, U7 74LS154, U8 74LS04, U9 74LS08

Commit message: saving
Parts:
- removed J1, J6: Conn_01x08, Connector_PinHeader_2.54mm:PinHeader_1x08_P2.54mm_Vertical, symbol Connector_Generic:Conn_01x08
- removed J2: Conn_01x29, Connector_PinHeader_2.54mm:PinHeader_1x29_P2.54mm_Vertical, symbol Connector_Generic:Conn_01x29
- removed J3: Conn_01x24, Connector_PinHeader_2.54mm:PinHeader_1x24_P2.54mm_Vertical, symbol Connector_Generic:Conn_01x24
- removed J4: Conn_01x12, Connector_PinSocket_2.54mm:PinSocket_1x12_P2.54mm_Vertical, symbol Connector_Generic:Conn_01x12
- removed J5: Conn_01x07, Connector_PinSocket_2.54mm:PinSocket_1x07_P2.54mm_Vertical, symbol Connector_Generic:Conn_01x07
- removed J7: Conn_01x07, Connector_PinHeader_2.54mm:PinHeader_1x07_P2.54mm_Vertical, symbol Connector_Generic:Conn_01x07
- removed U1, U4: PLCC32_28_28C256, Stephenv6:PLCC-32-SOCKET-Microchip-32J-10_2001-B-IPC_A, symbol Stephen:PLCC32_28_28C256
- removed U10, U14, U9: 74LS08, Package_SO:SOIC-14_3.9x8.7mm_P1.27mm, symbol 74xx:74LS08
- removed U12: 74LS139, Package_SO:SOIC-16_3.9x9.9mm_P1.27mm, symbol 74xx:74LS139
- removed U13, U6, U7: 74LS154, Package_SO:SOIC-24W_7.5x15.4mm_P1.27mm, symbol 74xx:74LS154
- removed U15, U16, U3: 74HC245, Package_SO:SOIC-20W_7.5x12.8mm_P1.27mm, symbol 74xx:74HC245
- removed U8: 74LS04, Package_SO:SOIC-14_3.9x8.7mm_P1.27mm, symbol 74xx:74LS04
- added J1, J4: Conn_01x05, Connector_PinHeader_2.54mm:PinHeader_1x05_P2.54mm_Vertical, symbol Connector_Generic:Conn_01x05
- added J2: Conn_01x13, Connector_PinHeader_2.54mm:PinHeader_1x13_P2.54mm_Vertical, symbol Connector_Generic:Conn_01x13
- added J3: Conn_01x03, Connector_PinHeader_2.54mm:PinHeader_1x03_P2.54mm_Vertical, symbol Connector_Generic:Conn_01x03
- added J5: Conn_01x25, Connector_PinHeader_2.54mm:PinHeader_1x25_P2.54mm_Vertical, symbol Connector_Generic:Conn_01x25
- added J6: Conn_01x20, Connector_PinHeader_2.54mm:PinHeader_1x20_P2.54mm_Vertical, symbol Connector_Generic:Conn_01x20
- added J7: Conn_01x04, Connector_PinHeader_2.54mm:PinHeader_1x04_P2.54mm_Vertical, symbol Connector_Generic:Conn_01x04
- added U1, U14, U4, U7: 74HC245, Package_SO:SOIC-20W_7.5x12.8mm_P1.27mm, symbol 74xx:74HC245
- added U10, U8, U9: 74LS154, Package_SO:SOIC-24W_7.5x15.4mm_P1.27mm, symbol 74xx:74LS154
- added U12, U13, U3: 74LS08, Package_SO:SOIC-14_3.9x8.7mm_P1.27mm, symbol 74xx:74LS08
- added U6: 74LS138, Package_SO:SOIC-16_3.9x9.9mm_P1.27mm, symbol 74xx:74LS138
- added U? (x7): 74LS04, symbol 74xx:74LS04
- J8: value Conn_01x11 -> Conn_01x10; Field4 Unused Control Lines -> (none)
- U2: Field4 Writes: 0bxx_00_xxxx -> (none); Field5 General Purpose Registers -> (none)
- U5: Field4 Write Enable Decoder -> (none); Field5 0bxx11xxxx -> (none)
- U5: Field4 Special Write Decoder -> (none); Field5 0b11xxxxxx -> (none)
- U5: Field4 Read Decoder -> (none)
Connections:
- net ~{IRQ_WRITE} is gone; now on net ~{WRITE_DATA}: U11.10
- net ~{MEM_REQUEST} is gone; now on net ~{MEM_READ}: U11.6
- net ALU_FUNC_0: now also J5.6 (Pin_6), U7.18 (B0)
- net ALU_FUNC_1: now also J5.5 (Pin_5), U7.17 (B1)
- net ALU_FUNC_2: now also J5.4 (Pin_4), U7.16 (B2)
- net ALU_FUNC_3: now also J5.3 (Pin_3), U7.15 (B3)
- net ALU_FUNC_4: now also J5.2 (Pin_2), U7.14 (B4)
- net ALU_FUNC_5: now also J5.1 (Pin_1), U7.13 (B5)
- net CLOCK: now also J1.5 (Pin_5)
- net GND: now also J1.2 (Pin_2), U1.10 (GND), U1.5 (A3), U1.6 (A4), U1.7 (A5), U1.8 (A6), U1.9 (A7), U10.12 (GND), U12.7 (GND), U13.7 (GND), U14.10 (GND), U14.6 (A4), U14.7 (A5), U14.8 (A6), U14.9 (A7), U3.7 (GND), U4.10 (GND), U4.6 (A4), U4.7 (A5), U4.8 (A6), U4.9 (A7), U6.4 (E1), U6.5 (E2), U6.8 (GND), U7.10 (GND), U7.8 (A6), U7.9 (A7), U8.12 (GND), U9.12 (GND); no longer U2.5 (A3)
- net GPR0: now also J6.13 (Pin_13), U1.18 (B0); no longer U2.18 (B0)
- net GPR1: now also J6.14 (Pin_14), U1.17 (B1); no longer U2.17 (B1)
- net GPR2: now also J6.15 (Pin_15), U1.16 (B2); no longer U2.16 (B2)
- net GPR3: now also U2.18 (B0), J6.16 (Pin_16)
- net GPR4: now also U2.17 (B1), J6.17 (Pin_17)
- net GPR5: now also U2.16 (B2), J6.18 (Pin_18)
- net GPR6: now also U2.15 (B3), J6.19 (Pin_19)
- net INSTRUCTION0: now also J2.6 (Pin_6)
- net INSTRUCTION1: now also J2.7 (Pin_7)
- net INSTRUCTION2: now also J2.8 (Pin_8)
- net INSTRUCTION3: now also J2.9 (Pin_9)
- net INSTRUCTION4: now also J2.10 (Pin_10)
- net INSTRUCTION5: now also J2.11 (Pin_11)
- net INSTRUCTION6: now also J2.12 (Pin_12)
- net INSTRUCTION7: now also J2.13 (Pin_13)
- net JCC_ADR0: now also J5.9 (Pin_9), U4.18 (B0)
- net JCC_ADR1: now also J5.10 (Pin_10), U4.17 (B1)
- net JCC_ADR2: now also J5.11 (Pin_11), U4.16 (B2)
- net JCC_ADR3: now also J5.12 (Pin_12), U4.15 (B3)
- net RESET: now also J1.3 (Pin_3)
- net STEP0: now also J2.1 (Pin_1)
- net STEP1: now also J2.2 (Pin_2)
- net STEP2: now also J2.3 (Pin_3)
- net STEP3: now also J2.4 (Pin_4)
- net VCC: now also J1.1 (Pin_1), U1.1 (A->B), U1.20 (VCC), U10.24 (VCC), U12.14 (VCC), U13.14 (VCC), U14.1 (A->B), U14.20 (VCC), U3.14 (VCC), U4.1 (A->B), U4.20 (VCC), U6.16 (VCC), U6.6 (E3), U7.1 (A->B), U7.20 (VCC), U7.7 (A5), U8.24 (VCC), U9.24 (VCC)
- net ~{IO_READ}: now also J7.4 (Pin_4), U12.6; no longer U11.11
- net ~{IO_REQUEST}: now also J7.2 (Pin_2), U12.8; no longer U11.3
- net ~{IO_WRITE}: now also J7.3 (Pin_3), U12.3
- net ~{MEM_LATCH_MAR}: now also J6.1 (Pin_1), U8.4 (S3)
- net ~{MEM_READ}: now also J6.2 (Pin_2)
- net ~{MEM_WRITE}: now also U11.11, J6.3 (Pin_3)
- net ~{PC_DEC}: now also J5.21 (Pin_21), U8.8 (S7)
- net ~{PC_INC}: now also J5.20 (Pin_20)
- net ~{READ_IO_MEM}: now also U12.12, U12.5, U9.13 (S11); no longer U11.13, U11.4
- net ~{READ_IO}: now also U12.4, U12.9, U9.11 (S10); no longer U11.1, U11.12
- net ~{RESET}: now also J1.4 (Pin_4); no longer U5.9 (O3)
- net ~{SP_DEC}: now also U5.9 (O3), J5.25 (Pin_25)
- net ~{SP_INC}: now also J5.24 (Pin_24), U?.2
- net ~{SP_LOAD}: now also J5.23 (Pin_23), U8.9 (S8)
- net ~{WRITE_DATA}: now also U3.10, U8.2 (S1)
- net ~{WRITE_IO_MEM}: now also U10.10 (S9), U12.1, U12.13; no longer U11.5
- net ~{WRITE_IO}: now also U10.9 (S8), U12.10, U12.2; no longer U11.2
- net ~{WRITE_STACK}: now also U11.13, U3.13, U8.3 (S2)
- net ~{RESET_STEP}: now reaches U5.10 (O2)
- net ~{RESET_STEP}: now also J3.3 (Pin_3)
- net WRITE0 renamed μ1_0
- net μ1_0: now also U7.2 (A0), U9.23 (A0)
- net WRITE1 renamed μ1_1
- net μ1_1: now also U7.3 (A1), U9.22 (A1)
- net WRITE2 renamed μ1_2
- net μ1_2: now also U7.4 (A2), U9.21 (A2)
- net WRITE4 renamed μ1_5
- net WRITE5 renamed μ1_4
- net WRITE6 renamed μ1_6
- net WRITE7 renamed μ1_7
- net ~{EN_WRITE_0} renamed ~{EN_READ_GPR}
- net ~{EN_WRITE_1} renamed ~{EN_ALU}
- net ~{EN_ALU}: now also U3.1, U7.6 (A4)
- net ~{EN_WRITE_2} renamed ~{EN_ALU_INVERT}
- net ~{EN_ALU_INVERT}: now also U3.2
- net ~{EN_WRITE_3} renamed ~{EN_READ_GENERAL_CONTROL}
- net ~{EN_READ_GENERAL_CONTROL}: now also U9.18 (E0), U9.19 (E1)
- net ~{IRQ_EN}: no longer names the net of U11.8
- net ~{IRQ_EN}: now also U11.12
- net ~{IRQ_READ} renamed ~{WRITE_CODE}
- net ~{WRITE_CODE}: now also U3.5, U8.1 (S0)
- net ~{NC_READ1_15} renamed ~{OFFSET_OUT}
- net ~{OFFSET_OUT}: now also U14.16 (B2)
- net ~{NC_WRITE1_14} renamed ~{OFFSET_LATCH}
- net ~{OFFSET_LATCH}: now also U10.1 (S0)
- net ~{NC_WRITE1_15} renamed ~{INDEX_DEC}
- net ~{INDEX_DEC}: now also U10.3 (S2)
- net ~{NC_WRITE2_10} renamed ~{INDEX_C0}
- net ~{INDEX_C0}: now also U14.18 (B0)
- net ~{NC_WRITE2_11} renamed ~{INDEX_C1}
- net ~{INDEX_C1}: now also U14.17 (B1)
- net ~{NC_WRITE2_12} renamed ~{INDEX_OUT}
- net ~{INDEX_OUT}: now also U14.15 (B3)
- net ~{NC_WRITE2_13} renamed ~{DISPLACEMENT_INC}
- net ~{DISPLACEMENT_INC}: now also U10.5 (S4)
- net ~{NC_WRITE2_14} renamed ~{DISPLACEMENT_LATCH}
- net ~{DISPLACEMENT_LATCH}: now also U13.11
- net ~{NC_WRITE2_15} renamed ~{DISPLACEMENT_OUT}
- net ~{DISPLACEMENT_OUT}: now also U9.14 (S12)
- net ~{NC_WRITE2_8} renamed ~{INDEX_INC}
- net ~{INDEX_INC}: now also U10.4 (S3)
- net ~{NC_WRITE2_9} renamed ~{INDEX_LOAD}
- net ~{INDEX_LOAD}: now also U10.2 (S1)
- new net: J5.14 (Pin_14), J5.19 (Pin_19)
- new net: U11.3, U11.4
- new net: U3.3, U7.19 (CE)
- new net: J3.2 (Pin_2), J4.1 (Pin_1)
- new net FLAGS_RESTORE: J5.16 (Pin_16), U13.1, U8.10 (S9)
- new net INT_REG_SEL: J4.4 (Pin_4), U10.8 (S7), U13.4
- new net Microcode EEPROM 2/Q7: U?.1
- new net STEP4: J2.5 (Pin_5)
- new net ~{A_IN}: J5.8 (Pin_8), U8.14 (S12)
- new net ~{B_IN}: J5.7 (Pin_7), U8.15 (S13)
- new net ~{CODE_SEG_EN}: J6.5 (Pin_5), U3.6
- new net ~{CODE_SEG_IN}: J6.4 (Pin_4), U8.5 (S4)
- new net ~{CODE_SEG_OUT}: J6.6 (Pin_6), U9.6 (S5)
- new net ~{DATA_SEG_EN}: J6.8 (Pin_8), U3.8
- new net ~{DATA_SEG_IN}: J6.7 (Pin_7), U8.6 (S5)
- new net ~{DATA_SEG_OUT}: J6.9 (Pin_9), U9.5 (S4)
- new net ~{DISPLACEMENT_IN_BASED}: U10.6 (S5), U13.13
- new net ~{ENABLE_INDEX_OFFSET}: U13.12, U14.19 (CE), U6.11 (O4)
- new net ~{EN_JCC}: J5.13 (Pin_13), U4.19 (CE), U6.14 (O1)
- new net ~{EN_WRITE_GENERAL_1}: U6.13 (O2), U8.18 (E0), U8.19 (E1)
- new net ~{EN_WRITE_GENERAL_2}: U10.18 (E0), U10.19 (E1), U6.12 (O3)
- new net ~{EN_WRITE_GENERAL_3}: U6.10 (O5)
- new net ~{EN_WRITE_GENERAL_4}: U6.9 (O6)
- new net ~{EN_WRITE_GENERAL_5}: U6.7 (O7)
- new net ~{EN_WRITE_GPR}: U1.19 (CE), U6.15 (O0)
- new net ~{FLAGS_IN}: J5.15 (Pin_15), U13.3
- new net ~{FLAGS_OUT}: J5.17 (Pin_17), U9.8 (S7)
- new net ~{INT_EN}: J4.5 (Pin_5), U13.8
- new net ~{INT_READ}: J4.3 (Pin_3), U13.10, U9.7 (S6)
- new net ~{INT_WRITE}: J4.2 (Pin_2), U13.6, U13.9
- new net ~{IO_MEM_REQUEST}: J7.1 (Pin_1), U12.11
- new net ~{IR_IN}: J3.1 (Pin_1), U8.13 (S11)
- new net ~{PC_OUT}: J5.18 (Pin_18), U9.9 (S8)
- new net ~{READ_CODE}: U11.1, U3.4, U9.1 (S0)
- new net ~{READ_DATA}: U11.2, U3.9, U9.2 (S1)
- new net ~{READ_STACK}: U11.5, U3.12, U9.3 (S2)
- new net ~{RESET_GPR}: J6.20 (Pin_20), U8.17 (S15)
- new net ~{RESTORE_FLAGS}: U13.2, U8.11 (S10)
- new net ~{SP_OUT}: J5.22 (Pin_22), U9.10 (S9)
- new net ~{STACK_SEG_EN}: J6.11 (Pin_11), U3.11
- new net ~{STACK_SEG_IN}: J6.10 (Pin_10), U8.7 (S6)
- new net ~{STACK_SEG_OUT}: J6.12 (Pin_12), U9.4 (S3)
- new net ~{WRITE_IPR}: U10.7 (S6), U13.5
- new net μ1_3: U2.5 (A3), U7.5 (A3), U9.20 (A3)
- new net μ2_0: U1.2 (A0), U10.23 (A0), U14.2 (A0), U4.2 (A0), U8.23 (A0)
- new net μ2_1: U1.3 (A1), U10.22 (A1), U14.3 (A1), U4.3 (A1), U8.22 (A1)
- new net μ2_2: U1.4 (A2), U10.21 (A2), U14.4 (A2), U4.4 (A2), U8.21 (A2)
- new net μ2_3: U10.20 (A3), U14.5 (A3), U4.5 (A3), U8.20 (A3)
- new net μ2_4: U6.1 (A0)
- new net μ2_5: U6.2 (A1)
- new net μ2_6: U6.3 (A2)
Other:
- added sheet Microcode EEPROM 1 (eeprom.kicad_sch)
- added sheet Microcode EEPROM 2 (eeprom.kicad_sch)
- note added: "& Step Counter"
- note added: "0x0: NOP"
- note added: "0x0: NOP 0x1: ASSERT C 0x2: ASSERT D 0x3: ASSERT S1 0x4: ASSERT S2 0x5: ASSERT S1S2 0x6: ASSERT F 0x7: ASSERT S3 0x8: ASSERT S3L 0x9: ASSERT S3H 0xa: nc 0xb: nc 0xc: nc 0xd: nc 0xe: nc 0xf: nc"
- note added: "0x10: A 0x11: ADD 0x12: ADC 0x13: SUB 0x14: SBB 0x15: INC 0x16: DEC 0x17: AND 0x18: OR 0x19: XOR 0x1a: SHL 0x1b: SHR 0x1c: ASL 0x1d: ASR 0x1e: ROR 0x1f: ROL"
- note added: "0x10: JUMP"
- note added: "0x11: JLE, JNG"
- note added: "0x12: JG, JNLE"
- note added: "0x13: JGE, JNL"
- note added: "0x14: JL, JNGE"
- note added: "0x15: JA, JNBE"
- note added: "0x16: JBE, JNA"
- note added: "0x17: JNB, JAE, JNC"
- note added: "0x18: JB, JNAE, JC"
- note added: "0x19: JNE, JNZ"
- note added: "0x1: Load C"
- note added: "0x1a: JE, JZ"
- note added: "0x1b: JNS"
- note added: "0x1c: JS"
- note added: "0x1d: JNO"
- note added: "0x1e: JO"
- note added: "0x1f: NOP"
- note added: "0x20: NOT A 0x21: **NOT ADD 0x22: **NOT ADC 0x23: **NOT SUB 0x24: **NOT SBB 0x25: **NOT INC 0x26: **NOT DEC 0x27: NAND 0x28: NOR 0x29: XNOR 0x2a: **NOT SHL 0x2b: **NOT SHR 0x2c: **NOT ASL 0x2d: **NOT ASR 0x2e: **NOT ROR 0x2f: **NOT ROL ** Strange, but maybe there is a use?"
- note added: "0x20: WRITE CODE"
- note added: "0x21: WRITE DATA"
- note added: "0x22: WRITE STACK"
- note added: "0x23: LATCH MAR"
- note added: "0x24: LATCH CODE SEGMENT"
- note added: "0x25: LATCH DATA SEGMENT"
- note added: "0x26: LATCH STACK SEGMENT"
- note added: "0x27: DECREMENT PROGRAM COUNTER"
- note added: "0x28: INCREMENT STACK POINTER"
- note added: "0x29: DECREMENT STACK POINTER"
- note added: "0x2: Load D"
- note added: "0x2a: LATCH STACK POINTER"
- note added: "0x2b: LATCH FLAGS"
- note added: "0x2c: RESTORE FLAGS"
- note added: "0x2d: LATCH INSTRUCTION REGISTER"
- note added: "0x2e: LATCH ACCUMULATOR"
- note added: "0x2f: LATCH B REGISTER"
- note added: "0x30: Latch Offset Register"
- note added: "0x30: READ CODE MEMORY 0x31: READ DATA MEMORY 0x32: READ STACK MEMORY 0x33: READ CODE SEGMENT 0x34: READ DATA SEGMENT 0x35: READ STACK SEGMENT 0x36: READ INTERRUPT PORT 0x37: READ FLAGS 0x38: READ PROGRAM COUNTER 0x39: READ STACK POINTER 0x3a: READ I/O 0x3b: READ I/O MEMORY 0x3c: READ DISPLACEMENT 0x3d: n.c. 0x3e: n.c. 0x3f: n.c."
- note added: "0x31: Latch Index Register"
- note added: "0x32: Decrement Index Register"
- note added: "0x33: Increment Index Register"
- note added: "0x34: Write Interrupt Priority Register"
- note added: "0x35: Write Interrupt Mask Register"
- note added: "0x36: Write I/O"
- note added: "0x37: Write I/O Mem"
- note added: "0x38: n.c."
- note added: "0x39: n.c."
- note added: "0x3: Load Scratch 1"
- note added: "0x3a: n.c."
- note added: "0x3b: n.c."
- note added: "0x3c: n.c."
- note added: "0x3d: n.c."
- note added: "0x3e: n.c."
- note added: "0x3f: n.c."
- note added: "0x40"
- note added: "0x40: Indexed * 1 + Displacement"
- note added: "0x41: Indexed * 2 + Displacement"
- note added: "0x42: Indexed * 4 + Displacement"
- note added: "0x43: Indexed * 8 + Displacement"
- note added: "0x44: Indexed * 1"
- note added: "0x45: Indexed * 2"
- note added: "0x46: Indexed * 4"
- note added: "0x47: Indexed * 8"
- note added: "0x48: Displacement"
- note added: "0x49: NOP"
- note added: "0x4: Load Scratch 2"
- note added: "0x4a: NOP"
- note added: "0x4b: NOP"
- note added: "0x4c: NOP"
- note added: "0x4d: NOP"
- note added: "0x4e: NOP"
- note added: "0x4f: NOP"
- note added: "0x5: Load F"
- note added: "0x6: Load Scratch 3"
- note added: "0x7: NOP"
- note added: "0x80"
- note added: "0x8: NOP"
- note added: "0x9: NOP"
- note added: "0xC0"
- note added: "0xa: NOP"
- note added: "0xb: NOP"
- note added: "0xc: NOP"
- note added: "0xd: NOP"
- note added: "0xe: NOP"
- note added: "0xf: NOP"
- note added: "Additional Decode Logic"
- note added: "Displacement"
- note added: "General"
- note added: "General Purpose Registers & Memory"
- note added: "I/O"
- note added: "Instruction Register"
- note added: "Interrupts"
- note added: "Program Counter / Stack Pointer / ALU"
- note added: "READS"
- note added: "Unused"
- note added: "WRITES"
- note added: "[0x0..0xF]"
- note added: "[0x00..0x0f]"
- note added: "[0x00..0xf]"
- note added: "[0x10..0x1F]"
- note added: "[0x10..0x1f]"
- note added: "[0x20..0x2F]"
- note added: "[0x20..0x2f]"
- note added: "[0x30..0x3F]"
- note added: "[0x30..0x3f]"
- note added: "[0x40..0x4F]"
- note added: "[0x40..0x4f]"
- note added: "[0x50..0x5f]"
- note added: "[0x60..0x6f]"
- note added: "[0x70..0x7f]"
- note added: "~{INT_REQUEST}"
- note added: "~{IREQ}"
- note added: "~{JCC_LD_PC_COND}"
- note removed: "0b00xxxxxx - 0x00 NOP"
- note removed: "0b01xxxxxx - 0x40 Enable Offset"
- note removed: "0b01xxxxxx - 0x40 Increment PC"
- note removed: "0b10xxxxxx - 0x80 Reset Op Counter"
- note removed: "0b10xxxxxx - 0x80 n.c."
- note removed: "0b11xxxxxx - 0xC0 Reset CPU"
- note removed: "0b11xxxxxx - 0xC0 n.c."
- note removed: "0bxx000000: (0x0 | 0x0) 0x0 NOP 0bxx000001: (0x0 | 0x1) 0x1 ASSERT C 0bxx000010: (0x0 | 0x2) 0x2 ASSERT D 0bxx000011: (0x0 | 0x3) 0x3 ASSERT S1 0bxx000100: (0x0 | 0x4) 0x4 ASSERT S2 0bxx000101: (0x0 | 0x5) 0x5 ASSERT S1S2 0bxx000110: (0x0 | 0x6) 0x6 ASSERT F 0bxx000111: (0x0 | 0x7) 0x7 ASSERT S3 0bxx001000: (0x0 | 0x8) 0x8 ASSERT S3L 0bxx001001: (0x0 | 0x9) 0x9 ASSERT S3H 0bxx001010: (0x0 | 0xA) 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"
- note removed: "0bxx00x000: (0x0 | 0x0) 0x0 NOP 0bxx00x001: (0x0 | 0x1) 0x1 LDC 0bxx00x010: (0x0 | 0x2) 0x2 LDD 0bxx00x011: (0x0 | 0x3) 0x3 LDS1 0bxx00x100: (0x0 | 0x4) 0x4 LDS2 0bxx00x101: (0x0 | 0x5) 0x5 LDF 0bxx00x110: (0x0 | 0x6) 0x6 LDS3 0bxx00x111: (0x0 | 0x7) 0x7 NOP"
- note removed: "0bxx00xxxx"
- note removed: "0bxx010000: (0x10 | 0x0) 0x10 LDA 0bxx010001: (0x10 | 0x1) 0x11 LDB 0bxx010010: (0x10 | 0x2) 0x12 LDMAR 0bxx010011: (0x10 | 0x3) 0x13 LDCS 0bxx010100: (0x10 | 0x4) 0x14 LDDS 0bxx010101: (0x10 | 0x5) 0x15 LDSS 0bxx010110: (0x10 | 0x6) 0x16 MEM WRITE DATA 0bxx010111: (0x10 | 0x7) 0x17 MEM WRITE STACK 0bxx011000: (0x10 | 0x8) 0x18 LDFLAGS 0bxx011001: (0x10 | 0x9) 0x19 RESTORE FLAGS 0bxx011010: (0x10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"
- note removed: "0bxx010000: (0x10 | 0x0) 0x10 READ CODE 0bxx010001: (0x10 | 0x1) 0x11 READ DATA 0bxx010010: (0x10 | 0x2) 0x12 READ STACK 0bxx010011: (0x10 | 0x3) 0x13 CS OUT 0bxx010100: (0x10 | 0x4) 0x14 DS OUT 0bxx010101: (0x10 | 0x5) 0x15 SS OUT 0bxx010110: (0x10 | 0x6) 0x16 PC OUT 0bxx010111: (0x10 | 0x7) 0x17 SP OUT 0bxx011000: (0x10 | 0x8) 0x18 FLAGS OUT 0bxx011001: (0x10 | 0x9) 0x19 READ IO 0bxx011010: (0x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"
- note removed: "0bxx01xxxx"
- note removed: "0bxx100000: (0x20 | 0x0) 0x20 A 0bxx100001: (0x20 | 0x1) 0x21 ADD 0bxx100010: (0x20 | 0x2) 0x22 ADC 0bxx100011: (0x20 | 0x3) 0x23 SUB 0bxx100100: (0x20 | 0x4) 0x24 SBB 0bxx100101: (0x20 | 0x5) 0x25 INC 0bxx100110: (0x20 | 0x6) 0x26 DEC 0bxx100111: (0x20 | 0x7) 0x27 AND 0bxx101000: (0x20 | 0x8) 0x28 OR 0bxx101001: (0x20 | 0x9) 0x29 XOR 0bxx101010: (0x20 | 0xA) 0x2A SHL 0bxx101011: (0x20 | 0xB) 0x2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"
- note removed: "0bxx100000: (0x20 | 0x0) 0x20 LDIR 0bxx100001: (0x20 | 0x1) 0x21 LDPC 0bxx100010: (0x20 | 0x2) 0x22 DEC PC 0bxx100011: (0x20 | 0x3) 0x23 LDSP 0bxx100100: (0x20 | 0x4) 0x24 DEC SP 0bxx100101: (0x20 | 0x5) 0x25 INC SP 0bxx100110: (0x20 | 0x6) 0x26 LDS4 0bxx100111: (0x20 | 0x7) 0x27 LD OFFSET 0bxx101000: (0x20 | 0x8) 0x28 n.c. 0bxx101001: (0x20 | 0x9) 0x29 n.c. 0bxx101010: (0x20 | 0xA) 0x2A n.c. 0bx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"
- note removed: "0bxx10xxxx"
- note removed: "0bxx110000: (0x30 | 0x0) 0x30 Jump 0bxx110001: (0x30 | 0x1) 0x31 JLE, JNG 0bxx110010: (0x30 | 0x2) 0x32 JG, JNLE 0bxx110011: (0x30 | 0x3) 0x33 JGE, JNL 0bxx110100: (0x30 | 0x4) 0x34 JL, JNGE 0bxx110101: (0x30 | 0x5) 0x35 JA, JNBE 0bxx110110: (0x30 | 0x6) 0x36 JBE, JNA 0bxx110111: (0x30 | 0x7) 0x37 JNB, JAE, JNC 0bxx111000: (0x30 | 0x8) 0x38 JB, JNAE, JC 0bxx111001: (0x30 | 0x9) 0x39 JNE, JNZ 0bxx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"
- note removed: "0bxx110000: (0x30 | 0x0) 0x30 NOT A 0bxx110001: (0x30 | 0x1) 0x31 **NOT ADD 0bxx110010: (0x30 | 0x2) 0x32 **NOT ADC 0bxx110011: (0x30 | 0x3) 0x33 **NOT SUB 0bxx110100: (0x30 | 0x4) 0x34 **NOT SBB 0bxx110101: (0x30 | 0x5) 0x35 **NOT INC 0bxx110110: (0x30 | 0x6) 0x36 **NOT DEC 0bxx110111: (0x30 | 0x7) 0x37 NAND 0bxx111000: (0x30 | 0x8) 0x38 NOR 0bxx111001: (0x30 | 0x9) 0x39 XNOR 0bxx111010: (0x30 |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"
- note removed: "0bxx11xxxx"
- note removed: "CLOCK SOURCE"
- note removed: "Control Unit - Microcode Instruction Decoding"
- note removed: "From JCC Module: Active Conditional Jump"
- note removed: "I should get HALT in here somewhere. I think perhaps it should just be part of the Instruction Register Module with a control line here. But need to figure out how to "un halt" Perhaps "halt" is just an instruction that does not increment the PC, just loops itself"
- note removed: "If I add additional counter/address registers, I would be able to add new instructions, as well as perform some instructions more quickly, such as: "MOV SP, (F)" (could be added)"
- note removed: "NOP"
- note removed: "Read Enable Decoder is in charge of enabling other decoders which use READ[0..3] - They are all the control lines that perform any "read" operation"
- note removed: "Special Read Decoder is able to add an additional active control line at the same time as another Read operation. For example, this allows the CPU to ....[todo]..."
- note removed: "Special Write Decoder is able to add an additional active control line at the same time as another Write operation. For example, this allows the CPU to Increment the PC at the same time as latching the instrution register."
- note removed: "WHY DO I NEED PC_LOAD HERE? WHY NOT JUST USE 0b0000 with the JCC Module?"
- note removed: "Write Enable Decoder is in charge of enabling other decoders which use WRITE[0..3] - They are all the control lines that perform any "write" operation"
- note removed: "~{CLOCK}"
- note removed: "~{FLAGS_IN}"
- note removed: "~{JCC_EN}"
- note removed: "~{READ_CODE}"
- note removed: "~{READ_DATA}"
- note removed: "~{READ_STACK}"
- note removed: "~{RESTORE_FLAGS}"
- note removed: "~{WRITE_IRQ_MASK}"
- note removed: "~{WRITE_IRQ_PRIORITY}"

Commit message: cray cray save
Parts:
- added J9: Conn_01x03, Connector_PinHeader_2.54mm:PinHeader_1x03_P2.54mm_Vertical, symbol Connector_Generic:Conn_01x03
- added U15, U16: PLCC32_28_28C256, LIBRARY-8-bit-computer:Socket-PLCC-32, symbol LIBRARY-8-bit-computer:PLCC32_28_28C256
- gave numbers to parts that had none: 1
Connections:
- net GND: now also U15.16 (Gnd), U15.2 (A14), U15.23 (~{CE}), U15.25 (~{OE}), U16.16 (Gnd), U16.2 (A14), U16.23 (~{CE}), U16.25 (~{OE}), U16.30 (A13)
- net INSTRUCTION0: now also U15.6 (A5), U16.6 (A5)
- net INSTRUCTION1: now also U15.5 (A6), U16.5 (A6)
- net INSTRUCTION2: now also U15.4 (A7), U16.4 (A7)
- net INSTRUCTION3: now also U15.29 (A8), U16.29 (A8)
- net INSTRUCTION4: now also U15.28 (A9), U16.28 (A9)
- net INSTRUCTION5: now also U15.24 (A10), U16.24 (A10)
- net INSTRUCTION6: now also U15.27 (A11), U16.27 (A11)
- net INSTRUCTION7: now also U15.3 (A12), U16.3 (A12)
- net STEP0: now also U15.11 (A0), U16.11 (A0)
- net STEP1: now also U15.10 (A1), U16.10 (A1)
- net STEP2: now also U15.9 (A2), U16.9 (A2)
- net STEP3: now also U15.8 (A3), U16.8 (A3)
- net STEP4: now also U15.7 (A4), U16.7 (A4)
- net VCC: now also U15.30 (A13), U15.31 (~{WE}), U15.32 (Vcc), U16.31 (~{WE}), U16.32 (Vcc)
- net ~{EN_WRITE_GENERAL_3}: now also J9.1 (Pin_1)
- net ~{EN_WRITE_GENERAL_4}: now also J9.2 (Pin_2)
- net ~{EN_WRITE_GENERAL_5}: now also J9.3 (Pin_3)
- net μ1_0: now also U16.13 (I/O0)
- net μ1_1: now also U16.14 (I/O1)
- net μ1_2: now also U16.15 (I/O2)
- net μ1_3: now also U16.18 (I/O3)
- net μ1_4: now also U16.19 (I/O4)
- net μ1_5: now also U16.20 (I/O5)
- net μ1_6: now also U16.21 (I/O6)
- net μ1_7: now also U16.22 (I/O7)
- net μ2_0: now also U15.13 (I/O0)
- net μ2_1: now also U15.14 (I/O1)
- net μ2_2: now also U15.15 (I/O2)
- net μ2_3: now also U15.18 (I/O3)
- net μ2_4: now also U15.19 (I/O4)
- net μ2_5: now also U15.20 (I/O5)
- net μ2_6: now also U15.21 (I/O6)
- net Microcode EEPROM 2/Q7: no longer names the net of U17.1
- net Microcode EEPROM 2/Q7: now also U15.22 (I/O7)
Other:
- removed sheet Microcode EEPROM 1
- removed sheet Microcode EEPROM 2
- note added: "Extra NC"
- moved on the sheet: U1, U10, U13D, U14, U17A, U4, U6, U8
