File: PCBs/99_IN PROGRESS/LEFT-TO-DO-MVP/CPU-Control-Unit/eeprom.kicad_sch (KiCad schematic)
At the start: 1 part, among them U16 PLCC32_28_28C256

Commit message: cray cray save
Parts:
- removed U16: PLCC32_28_28C256, LIBRARY-8-bit-computer:Socket-PLCC-32, symbol LIBRARY-8-bit-computer:PLCC32_28_28C256
Changed lines of the file:
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@@
 (kicad_sch (version 20211123) (generator eeschema)
   (paper "A4")
-  (hierarchical_label "STEP2" (shape input) (at 102.108 100.838 180)
-    (effects (font (size 1.27 1.27)) (justify right))
-  )
-  (hierarchical_label "INSTRUCTION5" (shape input) (at 133.858 103.378 0)
-    (effects (font (size 1.27 1.27)) (justify left))
-  )
-  (hierarchical_label "INSTRUCTION3" (shape input) (at 133.858 90.678 0)
-    (effects (font (size 1.27 1.27)) (justify left))
-  )
-  (hierarchical_label "STEP0" (shape input) (at 102.108 105.918 180)
-    (effects (font (size 1.27 1.27)) (justify right))
-  )
-  (hierarchical_label "Q2" (shape output) (at 112.268 121.158 270)
-    (effects (font (size 1.27 1.27)) (justify right))
-  )
-  (hierarchical_label "INSTRUCTION0" (shape input) (at 102.108 93.218 180)
-    (effects (font (size 1.27 1.27)) (justify right))
-  )
-  (hierarchical_label "STEP1" (shape input) (at 102.108 103.378 180)
-    (effects (font (size 1.27 1.27)) (justify right))
-  )
-  (hierarchical_label "Q1" (shape output) (at 109.728 121.158 270)
-    (effects (font (size 1.27 1.27)) (justify right))
-  )
-  (hierarchical_label "Q7" (shape output) (at 133.858 108.458 0)
-    (effects (font (size 1.27 1.27)) (justify left))
-  )
-  (hierarchical_label "Q3" (shape output) (at 119.888 121.158 270)
-    (effects (font (size 1.27 1.27)) (justify right))
-  )
-  (hierarchical_label "INSTRUCTION7" (shape input) (at 113.538 83.058 90)
-    (effects (font (size 1.27 1.27)) (justify left))
-  )
-  (hierarchical_label "Q0" (shape output) (at 102.108 110.998 180)
-    (effects (font (size 1.27 1.27)) (justify right))
-  )
-  (hierarchical_label "INSTRUCTION4" (shape input) (at 133.858 93.218 0)
-    (effects (font (size 1.27 1.27)) (justify left))
-  )
-  (hierarchical_label "Q4" (shape output) (at 122.428 121.158 270)
-    (effects (font (size 1.27 1.27)) (justify right))
-  )
-  (hierarchical_label "INSTRUCTION2" (shape input) (at 110.998 83.058 90)
-    (effects (font (size 1.27 1.27)) (justify left))
-  )
-  (hierarchical_label "Q5" (shape output) (at 124.968 121.158 270)
-    (effects (font (size 1.27 1.27)) (justify right))
-  )
-  (hierarchical_label "A14_ID" (shape input) (at 126.238 83.058 90)
-    (effects (font (size 1.27 1.27)) (justify left))
-  )
-  (hierarchical_label "INSTRUCTION1" (shape input) (at 102.108 90.678 180)
-    (effects (font (size 1.27 1.27)) (justify right))
-  )
-  (hierarchical_label "STEP4" (shape input) (at 102.108 95.758 180)
-    (effects (font (size 1.27 1.27)) (justify right))
-  )
-  (hierarchical_label "STEP3" (shape input) (at 102.108 98.298 180)
-    (effects (font (size 1.27 1.27)) (justify right))
-  )
-  (hierarchical_label "Q6" (shape output) (at 133.858 110.998 0)
-    (effects (font (size 1.27 1.27)) (justify left))
-  )
-  (hierarchical_label "INSTRUCTION6" (shape input) (at 133.858 95.758 0)
-    (effects (font (size 1.27 1.27)) (justify left))
-  )
-  (symbol (lib_id "power:GND") (at 133.858 100.838 90)
-    (in_bom yes) (on_board yes)
-    (property "Reference" "#PWR061" (id 0) (at 140.208 100.838 0)
-      (effects (font (size 1.27 1.27)) hide)
-    )
-    (property "Value" "GND" (id 1) (at 138.684 100.838 90))
-    (property "Footprint" "" (id 2) (at 133.858 100.838 0)
-      (effects (font (size 1.27 1.27)) hide)
-    )
-    (property "Datasheet" "" (id 3) (at 133.858 100.838 0)
-      (effects (font (size 1.27 1.27)) hide)
-    )
-    (pin "1")
-  )
-  (symbol (lib_id "power:GND") (at 114.808 121.158 0)
-    (in_bom yes) (on_board yes)
-    (property "Reference" "#PWR056" (id 0) (at 114.808 127.508 0)
-      (effects (font (size 1.27 1.27)) hide)
-    )
-    (property "Value" "GND" (id 1) (at 114.808 125.984 90))
-    (property "Footprint" "" (id 2) (at 114.808 121.158 0)
-      (effects (font (size 1.27 1.27)) hide)
-    )
-    (property "Datasheet" "" (id 3) (at 114.808 121.158 0)
-      (effects (font (size 1.27 1.27)) hide)
-    )
-    (pin "1")
-  )
-  (symbol (lib_id "LIBRARY-8-bit-computer:PLCC32_28_28C256") (at 117.348 100.838 0)
-    (in_bom yes) (on_board yes)
-    (property "Reference" "U16" (id 0) (at 116.586 97.79 0)
-      (effects (font (size 1.27 1.27)) (justify left))
-    )
-    (property "Value" "PLCC32_28_28C256" (id 1) (at 108.712 100.838 0)
-      (effects (font (size 1.27 1.27)) (justify left) hide)
-    )
-    (property "Footprint" "LIBRARY-8-bit-computer:Socket-PLCC-32" (id 2) (at 127.508 105.918 0)
-      (effects (font (size 1.27 1.27)) hide)
-    )
-    (property "Datasheet" "http://ww1.microchip.com/downloads/en/DeviceDoc/doc0006.pdf" (id 3) (at 118.618 142.748 0)
-      (effects (font (size 1.27 1.27)) hide)
-    )
-    (property "Field4" "Write Microcode EEPROM" (id 4) (at 117.348 61.468 0)
-      (effects (font (size 3 3)) hide)
-    )
-    (pin "1")
-    (pin "10")
-    (pin "11")
-    (pin "12")
-    (pin "13")
-    (pin "14")
-    (pin "15")
-    (pin "16")
-    (pin "17")
-    (pin "18")
-    (pin "19")
-    (pin "2")
-    (pin "20")
-    (pin "21")
-    (pin "22")
-    (pin "23")
-    (pin "24")
-    (pin "25")
-    (pin "26")
-    (pin "27")
-    (pin "28")
-    (pin "29")
-    (pin "3")
-    (pin "30")
-    (pin "31")
-    (pin "32")
-    (pin "4")
-    (pin "5")
-    (pin "6")
-    (pin "7")
-    (pin "8")
-    (pin "9")
-  )
-  (symbol (lib_id "power:GND") (at 116.078 83.058 180)
-    (in_bom yes) (on_board yes)
-    (property "Reference" "#PWR?" (id 0) (at 116.078 76.708 0)
-      (effects (font (size 1.27 1.27)) hide)
-    )
-    (property "Value" "GND" (id 1) (at 116.078 78.232 90))
-    (property "Footprint" "" (id 2) (at 116.078 83.058 0)
-      (effects (font (size 1.27 1.27)) hide)
-    )
-    (property "Datasheet" "" (id 3) (at 116.078 83.058 0)
-      (effects (font (size 1.27 1.27)) hide)
-    )
-    (pin "1")
-  )
-  (symbol (lib_id "power:VCC") (at 121.158 83.058 0)
-    (in_bom yes) (on_board yes)
-    (property "Reference" "#PWR058" (id 0) (at 121.158 86.868 0)
-      (effects (font (size 1.27 1.27)) hide)
-    )
-    (property "Value" "VCC" (id 1) (at 121.158 78.232 90))
-    (property "Footprint" "" (id 2) (at 121.158 83.058 0)
-      (effects (font (size 1.27 1.27)) hide)
-    )
-    (property "Datasheet" "" (id 3) (at 121.158 83.058 0)
-      (effects (font (size 1.27 1.27)) hide)
-    )
-    (pin "1")
-  )
-  (symbol (lib_id "power:VCC") (at 123.698 83.058 0)
-    (in_bom yes) (on_board yes)
-    (property "Reference" "#PWR059" (id 0) (at 123.698 86.868 0)
-      (effects (font (size 1.27 1.27)) hide)
-    )
-    (property "Value" "VCC" (id 1) (at 123.698 78.232 90))
-    (property "Footprint" "" (id 2) (at 123.698 83.058 0)
-      (effects (font (size 1.27 1.27)) hide)
-    )
-    (property "Datasheet" "" (id 3) (at 123.698 83.058 0)
-      (effects (font (size 1.27 1.27)) hide)
-    )
-    (pin "1")
-  )
-  (symbol (lib_id "power:GND") (at 133.858 105.918 90)
-    (in_bom yes) (on_board yes)
-    (property "Reference" "#PWR062" (id 0) (at 140.208 105.918 0)
-      (effects (font (size 1.27 1.27)) hide)
-    )
-    (property "Value" "GND" (id 1) (at 138.684 105.918 90))
-    (property "Footprint" "" (id 2) (at 133.858 105.918 0)
-      (effects (font (size 1.27 1.27)) hide)
-    )
-    (property "Datasheet" "" (id 3) (at 133.858 105.918 0)
-      (effects (font (size 1.27 1.27)) hide)
-    )
-    (pin "1")
-  )
 )
