File: PCBs/99_IN PROGRESS/LEFT-TO-DO-MVP/__CHECKED__/Backplane-IO-Controller/cpu-input-output-control.kicad_sch (KiCad schematic)
At the start: 73 parts, among them J1 Conn_01x26, J10 Conn_01x28, J11 Conn_02x20_Odd_Even, J12 Conn_01x26, J13 Conn_01x28, J14 Conn_01x26, J15 Conn_01x28, J16 Conn_01x26, J17 Conn_01x28, J2 Conn_01x28, J3 Conn_01x39, J4 Conn_01x26, J5 Conn_01x28, J6 Conn_01x26, J7 Conn_01x28, J8 Conn_01x26, J9 PCIE-036-02-X-D-RA, U1 74LS08, U2 74LS154

Commit message: cray cray save
Parts:
- J1: Field4 (none) -> Port 0x14
- J12: Field4 (none) -> Port 0x10
- J14: Field4 (none) -> Port 0x9
- J16: Field4 (none) -> Port 0x8
- J4: Field4 (none) -> Port 0x13
- J6: Field4 (none) -> Port 0x12
- J8: Field4 (none) -> Port 0x11
Other:
- note added: "CPU Connections"
- note added: "I/O Port Connections"
- note added: "Input / Output Controller (I/O) & Backplane"
- note added: "LED Indicators"
- note removed: "AUDIO VIDEO DAC ADC"
- note removed: "Connections"
- note removed: "Input / Output Controller (I/O)"
- note removed: "UART/SERIAL Timer0 Timer1 KEYBOARD GAME CONTROLLER 1 GAME CONTROLLER 2"
- moved on the sheet: J9, U1A, U1B, U1C, U1D, U1E, U2
