File: PCBs/99_IN PROGRESS/LEFT-TO-DO-MVP/__CHECKED__/IO-Timer-2022/interrupts.kicad_sch (KiCad schematic)
At the start: 53 parts, among them J1 Conn_01x28, U1 74LS32, U2 74LS169, U3 74LS169, U4 74LS00, U5 74LS169, U6 74LS169, U7 74LS138, U8 74LS138

Commit message: cray cray save
Other:
- note added: "DOUBLE CHECK ~{PE} LINE - I THINK IT SHOULD ONLY COME FROM LAST COUNTER"
